File: ele/MainBoard.brd (EAGLE design)
At the start: 94 x 54.6 mm, 53 parts, among them X1 M8, X2 M8, X4 POWER_IN

Commit message: better
Parts:
- moved IM3 1.80 mm to (78.0, 3.81)
Routing:
- net GND: track 125.1 -> 144.0 mm, vias 7 -> 9
- net VCC: track 118.2 -> 120.7 mm
- net SLEEP: track 105.5 -> 103.0 mm
- net PWM2: track 122.3 -> 124.1 mm
- net GPIO26: track 66.2 -> 65.6 mm

Commit message: popisky
Parts:
- moved IM3 2.54 mm to (75.4, 3.81)
- moved JP8 2.17 mm to (93.0, 26.9)
- moved C5 1.27 mm to (39.4, 49.5)
- moved SW0 0.90 mm to (39.4, 49.5)
- moved JP11 0.25 mm to (87.0, 26.9)
- moved JP5 0.25 mm to (83.2, 26.9)
Routing:
- net GPIO13: track 95.4 -> 98.3 mm
- net VCC: track 120.7 -> 118.2 mm
- net GND: track 144.0 -> 141.5 mm
- net +5V: track 145.1 -> 142.5 mm
- net GPIO23: track 113.6 -> 116.1 mm
- net GPIO25: track 63.9 -> 66.3 mm
- net GPIO34: track 46.9 -> 49.1 mm
- net GPIO33: track 49.8 -> 52.1 mm
- net GPIO27: track 77.7 -> 79.9 mm
- net GPIO26: track 65.6 -> 67.9 mm
- net GPIO32: track 55.7 -> 57.9 mm
- net GPIO39: track 60.4 -> 62.4 mm
- net GPIO36: track 50.8 -> 52.9 mm
- net GPIO14: track 88.9 -> 90.9 mm
- net TX: track 60.5 -> 62.4 mm
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Other:
- board size 94 x 54.6 mm -> 99.3 x 54.6 mm
- board text added: "+"
- board text added: "-"
- board text added: "3.3V"
- board text added: "3V"
- board text added: "5V"
- board text added: "BLUE"
- board text added: "Batteri"
- board text added: "EN"
- board text added: "ENC_A1"
- board text added: "ENC_A2"
- board text added: "ENC_B1"
- board text added: "ENC_B2"
- board text added: "GND"
- board text added: "GREEN"
- board text added: "IN"
- board text added: "IO13"
- board text added: "IO14"
- board text added: "IO15"
- board text added: "IO16"
- board text added: "IO17"
- board text added: "IO21"
- board text added: "IO22"
- board text added: "IO23"
- board text added: "IO25"
- board text added: "IO26"
- board text added: "IO27"
- board text added: "IO32"
- board text added: "IO33"
- board text added: "IO34"
- board text added: "IO35"
- board text added: "IO36"
- board text added: "IO39"
- board text added: "M1"
- board text added: "M2"
- board text added: "MA1"
- board text added: "MA2"
- board text added: "MB1"
- board text added: "MB2"
- board text added: "OUT1"
- board text added: "OUT2"
- board text added: "OUT3"
- board text added: "OUT4"
- board text added: "P-LED"
- board text added: "PWM0"
- board text added: "PWM1"
- board text added: "PWM2"
- board text added: "PWM3"
- board text added: "RED"
- board text added: "RX"
- board text added: "S-leds"
- board text added: "S-servo"
- board text added: "SLEEP"
- board text added: "SW0"
- board text added: "SW1"
- board text added: "SW2"
- board text added: "SW3"
- board text added: "ServoS-5V"
- board text added: "TX"
- board text added: "ULT"
- board text added: "V5"
- board text added: "VCC"

Commit message: DRC
Parts:
- moved JP8 1.27 mm to (91.7, 26.9)
- moved R1 0.90 mm to (42.8, 10.0)
- moved C2 0.89 mm to (42.8, 10.2)
- moved JP6 0.76 mm to (40.1, 10.2)
- moved C1 0.13 mm to (34.2, 10.2)
- moved R4 0.13 mm to (34.2, 10.2)
Routing:
- net GND: track 141.5 -> 131.8 mm, vias 9 -> 13
- net OFF: track 32.7 -> 39.0 mm
- net ENC_B1: track 109.9 -> 113.4 mm
- net GPIO13: track 98.3 -> 96.0 mm
- net M1B: track 27.3 -> 29.1 mm
- net GPIO35: track 65.1 -> 66.8 mm
- net M2A: track 25.0 -> 26.3 mm
- net TX: track 62.4 -> 61.1 mm
- net RX: track 58.7 -> 57.5 mm
- net GPIO33: track 52.1 -> 50.8 mm
- net GPIO14: track 90.9 -> 89.6 mm
- net GPIO36: track 52.9 -> 51.7 mm
- net GPIO32: track 57.9 -> 56.7 mm
- net GPIO22: track 78.5 -> 77.3 mm
- net GPIO21: track 77.8 -> 78.9 mm
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Other:
- board size 99.3 x 54.6 mm -> 99.5 x 56.7 mm
