File: ele/SchoolBot/v1.0/SchoolBot.sch (EAGLE design)
At the start: 64 parts, among them X1 M8, X2 M8, X4 POWER_IN

Commit message: nove rozlozeni
konecne zaroutovano
Parts:
- removed R10: 1k, resistor:R-EU_M0805
- removed R11: 3k9, resistor:R-EU_M0805
- removed R9: 10k, resistor:R-EU_M0805
- added R5: (no value), pot:TRIM_US-SM-42/43X
Connections:
- removed net N$2: JP2.1, R10.2
- removed net N$4: R10.1, R11.2, R9.2
- new net BAT-REF: JP2.1, R5.S
- net GND: now also R5.E; no longer R11.1
- net GPIO23: no longer JP42.3, JP47.3, JP48.3
- net GPIO33: no longer JP2.2
- net GPIO34: now also JP2.2
- net GPIO35: now also JP42.3, JP47.3, JP48.3
- net PWM0: now also IM6.IO5; no longer IM6.IO0
- net PWM2: now also IM6.IO16; no longer IM6.IO5
- net PWM3: now also IM6.IO0; no longer IM6.IO16
- net VCC: now also R5.A; no longer R9.1
Other:
- note added: "THIS SIGNAL MUST BE HERE!"
- moved on the sheet: JP2
Changed lines of the file:
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@@
 <part name="JP4" library="pinhead" library_urn="urn:adsk.eagle:library:325" deviceset="PINHD-2X3" device="" package3d_urn="urn:adsk.eagle:package:22462/2"/>
 <part name="NC7" library="NC" deviceset="NC" device=""/>
-<part name="R9" library="resistor" library_urn="urn:adsk.eagle:library:348" deviceset="R-EU_" device="M0805" package3d_urn="urn:adsk.eagle:package:26079/1" value="10k"/>
-<part name="R10" library="resistor" library_urn="urn:adsk.eagle:library:348" deviceset="R-EU_" device="M0805" package3d_urn="urn:adsk.eagle:package:26079/1" value="1k"/>
-<part name="R11" library="resistor" library_urn="urn:adsk.eagle:library:348" deviceset="R-EU_" device="M0805" package3d_urn="urn:adsk.eagle:package:26079/1" value="3k9"/>
-<part name="P+1" library="supply1" library_urn="urn:adsk.eagle:library:371" deviceset="VCC" device=""/>
-<part name="GND17" library="supply1" library_urn="urn:adsk.eagle:library:371" deviceset="GND" device=""/>
 <part name="JP2" library="jumper" library_urn="urn:adsk.eagle:library:252" deviceset="JP1Q" device="" package3d_urn="urn:adsk.eagle:package:15455/1"/>
 <part name="SW4" library="switch-omron" library_urn="urn:adsk.eagle:library:377" deviceset="10-XX" device="" package3d_urn="urn:adsk.eagle:package:27496/1"/>
@@
 <part name="GND56" library="supply1" library_urn="urn:adsk.eagle:library:371" deviceset="GND" device=""/>
 <part name="JP6" library="pinhead" library_urn="urn:adsk.eagle:library:325" deviceset="PINHD-2X4" device="" package3d_urn="urn:adsk.eagle:package:22461/2"/>
+<part name="R5" library="pot" library_urn="urn:adsk.eagle:library:331" deviceset="TRIM_US-" device="SM-42/43X" package3d_urn="urn:adsk.eagle:package:22720/1"/>
+<part name="P+2" library="supply1" library_urn="urn:adsk.eagle:library:371" deviceset="VCC" device=""/>
+<part name="GND25" library="supply1" library_urn="urn:adsk.eagle:library:371" deviceset="GND" device=""/>
 </parts>
 <sheets>
@@
 RobotikaBrno.cz
 Robotarna</text>
+<text x="116.84" y="180.34" size="1.778" layer="94">THIS SIGNAL MUST BE HERE!</text>
+<text x="116.84" y="182.88" size="1.778" layer="94">THIS SIGNAL MUST BE HERE!</text>
+<text x="55.88" y="180.34" size="1.778" layer="94" rot="R180">THIS SIGNAL MUST BE HERE!</text>
 </plain>
 <instances>
@@
 <attribute name="VALUE" x="209.55" y="231.14" size="1.778" layer="96"/>
 </instance>
-<instance part="R9" gate="G$1" x="236.22" y="91.44" smashed="yes">
-<attribute name="NAME" x="232.41" y="92.9386" size="1.778" layer="95"/>
-<attribute name="VALUE" x="232.41" y="88.138" size="1.778" layer="96"/>
-</instance>
-<instance part="R10" gate="G$1" x="251.46" y="91.44" smashed="yes">
-<attribute name="NAME" x="247.65" y="92.9386" size="1.778" layer="95"/>
-<attribute name="VALUE" x="247.65" y="88.138" size="1.778" layer="96"/>
-</instance>
-<instance part="R11" gate="G$1" x="243.84" y="83.82" smashed="yes" rot="R90">
-<attribute name="NAME" x="242.3414" y="80.01" size="1.778" layer="95" rot="R90"/>
-<attribute name="VALUE" x="247.142" y="80.01" size="1.778" layer="96" rot="R90"/>
-</instance>
-<instance part="P+1" gate="VCC" x="226.06" y="91.44" smashed="yes" rot="R90">
-<attribute name="VALUE" x="228.6" y="88.9" size="1.778" layer="96" rot="R180"/>
-</instance>
-<instance part="GND17" gate="1" x="243.84" y="73.66" smashed="yes">
-<attribute name="VALUE" x="241.3" y="71.12" size="1.778" layer="96"/>
-</instance>
-<instance part="JP2" gate="A" x="269.24" y="91.44" smashed="yes" rot="R270">
-<attribute name="NAME" x="264.16" y="93.98" size="1.778" layer="95"/>
-<attribute name="VALUE" x="264.16" y="86.995" size="1.778" layer="96"/>
+<instance part="JP2" gate="A" x="243.84" y="78.74" smashed="yes" rot="R270">
+<attribute name="NAME" x="238.76" y="81.28" size="1.778" layer="95"/>
+<attribute name="VALUE" x="238.76" y="74.295" size="1.778" layer="96"/>
 </instance>
 <instance part="RN2" gate="A" x="193.04" y="205.74" smashed="yes">
@@
 <instance part="JP3" gate="A" x="292.1" y="116.84"/>
 <instance part="JP6" gate="A" x="60.96" y="99.06"/>
+<instance part="R5" gate="G$1" x="220.98" y="78.74" rot="MR180"/>
+<instance part="P+2" gate="VCC" x="220.98" y="96.52" smashed="yes" rot="MR0">
+<attribute name="VALUE" x="223.52" y="93.98" size="1.778" layer="96" rot="MR90"/>
+</instance>
+<instance part="GND25" gate="1" x="220.98" y="63.5" smashed="yes" rot="MR0">
+<attribute name="VALUE" x="223.52" y="60.96" size="1.778" layer="96" rot="MR0"/>
+</instance>
 </instances>
 <busses>
@@
 </segment>
 <segment>
-<pinref part="GND17" gate="1" pin="GND"/>
-<pinref part="R11" gate="G$1" pin="1"/>
-<wire x1="243.84" y1="76.2" x2="243.84" y2="78.74" width="0.1524" layer="91"/>
-</segment>
-<segment>
 <wire x1="322.58" y1="129.54" x2="312.42" y2="129.54" width="0.1524" layer="91"/>
 <wire x1="312.42" y1="129.54" x2="312.42" y2="132.08" width="0.1524" layer="91"/>
@@
 <wire x1="335.28" y1="200.66" x2="335.28" y2="205.74" width="0.1524" layer="91"/>
 </segment>
+<segment>
+<pinref part="R5" gate="G$1" pin="E"/>
+<wire x1="220.98" y1="71.12" x2="220.98" y2="66.04" width="0.1524" layer="91"/>
+<pinref part="GND25" gate="1" pin="GND"/>
+</segment>
 </net>
 <net name="+5V" class="0">
@@
 <wire x1="66.04" y1="203.2" x2="55.88" y2="203.2" width="0.1524" layer="91"/>
 <label x="55.88" y="203.2" size="1.778" layer="95"/>
+<junction x="55.88" y="203.2"/>
 </segment>
 <segment>
@@
 <pinref part="JP11" gate="A" pin="14"/>
 </segment>
+<segment>
+<pinref part="JP2" gate="A" pin="2"/>
+<wire x1="251.46" y1="78.74" x2="261.62" y2="78.74" width="0.1524" layer="91"/>
+<label x="254" y="78.74" size="1.778" layer="95"/>
+</segment>
 </net>
 <net name="GPIO35" class="0">
@@
 <wire x1="66.04" y1="200.66" x2="55.88" y2="200.66" width="0.1524" layer="91"/>
 <label x="55.88" y="200.66" size="1.778" layer="95"/>
+<junction x="55.88" y="200.66"/>
 </segment>
 <segment>
@@
 </segment>
 <segment>
-<pinref part="JP2" gate="A" pin="2"/>
-<wire x1="276.86" y1="91.44" x2="287.02" y2="91.44" width="0.1524" layer="91"/>
-<label x="279.4" y="91.44" size="1.778" layer="95"/>
-</segment>
-<segment>
 <label x="147.32" y="96.52" size="1.778" layer="95"/>
 <wire x1="142.24" y1="96.52" x2="154.94" y2="96.52" width="0.1524" layer="91"/>
@@
 </segment>
 </net>
-<net name="PWM1" class="0">
-<segment>
-<pinref part="IM6" gate="G$1" pin="IO17"/>
-<wire x1="106.68" y1="190.5" x2="116.84" y2="190.5" width="0.1524" layer="91"/>
-<label x="106.68" y="190.5" size="1.778" layer="95"/>
-<junction x="116.84" y="190.5"/>
-</segment>
-</net>
 <net name="PWM0" class="0">
 <segment>
-<pinref part="IM6" gate="G$1" pin="IO0"/>
-<wire x1="106.68" y1="182.88" x2="116.84" y2="182.88" width="0.1524" layer="91"/>
-<label x="106.68" y="182.88" size="1.778" layer="95"/>
-<junction x="116.84" y="182.88"/>
+<pinref part="IM6" gate="G$1" pin="IO5"/>
+<wire x1="106.68" y1="193.04" x2="116.84" y2="193.04" width="0.1524" layer="91"/>
+<label x="106.68" y="193.04" size="1.778" layer="95"/>
+<junction x="116.84" y="193.04"/>
 </segment>
 </net>
@@
 </segment>
 </net>
-<net name="PWM2" class="0">
-<segment>
-<pinref part="IM6" gate="G$1" pin="IO5"/>
-<wire x1="106.68" y1="193.04" x2="116.84" y2="193.04" width="0.1524" layer="91"/>
-<label x="106.68" y="193.04" size="1.778" layer="95"/>
-<junction x="116.84" y="193.04"/>
-</segment>
-</net>
-<net name="N$4" class="0">
-<segment>
-<pinref part="R9" gate="G$1" pin="2"/>
-<pinref part="R11" gate="G$1" pin="2"/>
-<wire x1="241.3" y1="91.44" x2="243.84" y2="91.44" width="0.1524" layer="91"/>
-<pinref part="R10" gate="G$1" pin="1"/>
-<wire x1="243.84" y1="91.44" x2="243.84" y2="88.9" width="0.1524" layer="91"/>
-<wire x1="243.84" y1="91.44" x2="246.38" y2="91.44" width="0.1524" layer="91"/>
-<junction x="243.84" y="91.44"/>
-</segment>
-</net>
 <net name="VCC" class="0">
 <segment>
-<pinref part="R9" gate="G$1" pin="1"/>
-<wire x1="228.6" y1="91.44" x2="231.14" y2="91.44" width="0.1524" layer="91"/>
-<pinref part="P+1" gate="VCC" pin="VCC"/>
-</segment>
-</net>
-<net name="N$2" class="0">
-<segment>
-<pinref part="R10" gate="G$1" pin="2"/>
-<wire x1="256.54" y1="91.44" x2="261.62" y2="91.44" width="0.1524" layer="91"/>
-<pinref part="JP2" gate="A" pin="1"/>
+<pinref part="R5" gate="G$1" pin="A"/>
+<wire x1="220.98" y1="93.98" x2="220.98" y2="86.36" width="0.1524" layer="91"/>
+<pinref part="P+2" gate="VCC" pin="VCC"/>
 </segment>
 </net>
@@
 </segment>
 </net>
-<net name="PWM3" class="0">
-<segment>
-<pinref part="IM6" gate="G$1" pin="IO16"/>
-<wire x1="106.68" y1="187.96" x2="116.84" y2="187.96" width="0.1524" layer="91"/>
-<label x="106.68" y="187.96" size="1.778" layer="95"/>
-<junction x="116.84" y="187.96"/>
-</segment>
-</net>
 <net name="GPIO33_5V" class="0">
 <segment>
@@
 </segment>
 </net>
+<net name="BAT-REF" class="0">
+<segment>
+<pinref part="R5" gate="G$1" pin="S"/>
+<wire x1="226.06" y1="78.74" x2="236.22" y2="78.74" width="0.1524" layer="91"/>
+<label x="236.22" y="78.74" size="1.778" layer="95" rot="MR0"/>
+<pinref part="JP2" gate="A" pin="1"/>
+</segment>
+</net>
+<net name="PWM1" class="0">
+<segment>
+<pinref part="IM6" gate="G$1" pin="IO17"/>
+<wire x1="106.68" y1="190.5" x2="116.84" y2="190.5" width="0.1524" layer="91"/>
+<label x="106.68" y="190.5" size="1.778" layer="95"/>
+<junction x="116.84" y="190.5"/>
+</segment>
+</net>
+<net name="PWM3" class="0">
+<segment>
+<pinref part="IM6" gate="G$1" pin="IO0"/>
+<wire x1="106.68" y1="182.88" x2="116.84" y2="182.88" width="0.1524" layer="91"/>
+<label x="106.68" y="182.88" size="1.778" layer="95"/>
+<junction x="116.84" y="182.88"/>
+</segment>
+</net>
+<net name="PWM2" class="0">
+<segment>
+<pinref part="IM6" gate="G$1" pin="IO16"/>
+<wire x1="106.68" y1="187.96" x2="116.84" y2="187.96" width="0.1524" layer="91"/>
+<label x="106.68" y="187.96" size="1.778" layer="95"/>
+<junction x="116.84" y="187.96"/>
+</segment>
+</net>
 </nets>
 </sheet>
@@
 </segment>
 </net>
-<net name="GPIO23" class="0">
+<net name="GPIO35" class="0">
 <segment>
 <pinref part="JP42" gate="G$1" pin="3"/>
