File: ele/SchoolBot/v1.0/SchoolBoard.brd (EAGLE design)
At the start: 95 x 60 mm, 55 parts, among them X1 M8, X2 M8, X4 POWER_IN

Commit message: drobnosti
Parts:
- moved LED0 0.76 mm to (12.7, 48.3)
- moved LED1 0.76 mm to (20.3, 48.3)
- moved LED2 0.76 mm to (27.9, 48.3)
- moved LED3 0.76 mm to (35.6, 48.3)
Routing:
- net LED3: track 44.6 -> 46.1 mm
- net LED1: track 30.3 -> 31.2 mm
- net LED0: track 28.8 -> 29.6 mm
- net SW1: track 36.1 -> 35.4 mm, vias 2 -> 1
- net LED2: track 34.3 -> 33.7 mm

Commit message: RB3202_jednotny_konektor_na_motory
Parts:
- removed C7: (no value), rcl:E5-10,5
- added JP12: (no value), pinhead:1X06
- JP6: device pinhead:2X04 -> pinhead:1X06
- moved JP10 86.9 mm to (6.10, 43.2), turned to 180 degrees
- moved C8 86.0 mm to (82.5, 5.13), turned to 90 degrees
- moved SW3 86.0 mm to (82.5, 5.13), turned to 180 degrees
- moved JP1 83.7 mm to (13.8, 55.8), turned to 0 degrees
- moved JP7 83.6 mm to (13.8, 51.9), turned to 180 degrees
- moved X1 83.5 mm to (81.0, 54.9), turned to 180 degrees
- moved JP9 81.9 mm to (86.6, 17.8), turned to 0 degrees
- moved IM11 80.8 mm to (8.13, 20.9), turned to 0 degrees
- moved LED0 78.6 mm to (82.3, 11.7), turned to 0 degrees
- moved JP3 78.1 mm to (13.7, 49.4), turned to 0 degrees
- moved C4 71.8 mm to (73.4, 5.13), turned to 90 degrees
- moved SW2 71.8 mm to (73.4, 5.13), turned to 180 degrees
- moved IM10 68.7 mm to (77.5, 44.2), turned to 270 degrees
- moved JP47 68.4 mm to (24.6, 54.7), turned to 90 degrees
- moved X2 68.3 mm to (70.9, 54.9), turned to 180 degrees
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Connections:
- net +5V: now also JP12.5; no longer JP6.1
- net ENC_A1: now also JP12.3; no longer JP6.6
- net ENC_A2: now also IM6.31, JP6.4; no longer IM6.30, JP6.3
- net ENC_B1: now also IM6.23, JP12.4; no longer IM6.31, JP6.4
- net ENC_B2: now also IM6.30, JP6.3; no longer IM6.23, JP6.5
- net GND: now also JP12.2, JP6.5; no longer C7.-, JP6.7, JP6.8
- net M1A: now also JP12.6
- net M1B: now also JP12.1
- net M2A: now also JP6.1
- net M2B: now also JP6.6
- net PWM0: now also IM6.25; no longer IM6.29
- net PWM1: now also IM6.27; no longer IM6.28
- net PWM2: now also IM6.28; no longer IM6.27
- net PWM3: now also IM6.29; no longer IM6.25
- net VCC: no longer C7.+
Routing:
- net +5V: track 93.3 -> 172.9 mm, vias 2 -> 4
- net VCC: track 13.5 -> 71.4 mm, vias 1 -> 6
- net M2B: track 0.00 -> 30.5 mm
- net ENC_A2: track 70.4 -> 46.0 mm, vias 1 -> 0
- net GND: track 22.2 -> 0.00 mm, vias 23 -> 25
- net ENC_B1: track 69.8 -> 48.9 mm, vias 1 -> 0
- net SLEEP: track 71.1 -> 51.1 mm
- net ON: track 74.3 -> 57.5 mm
- net PWM0: track 59.2 -> 43.9 mm
- net GPIO35: track 80.7 -> 90.7 mm
- net ENC_B2: track 52.8 -> 44.9 mm, vias 1 -> 0
- net BAT1: track 0.00 -> 7.67 mm
- net PWM3: track 60.1 -> 67.4 mm
- net PWM1: track 57.8 -> 51.7 mm
- net GPIO33_5V: track 37.8 -> 42.7 mm
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- added copper zone on layer 1, net M1B
- added copper zone on layer 1, net VCC
- removed copper zone on layer 1, net +5V
- removed copper zone on layer 1, net BAT1
- removed copper zone on layer 16, net M1B
- removed copper zone on layer 16, net M2B
- removed copper zone on layer 16, net VCC
Other:
- board text added: "!12"
- board text added: "!14"
- board text added: "!21"
- board text added: "!22"
- board text added: "!23"
- board text added: "!25"
- board text added: "!26"
- board text added: "!27"
- board text added: "!32"
- board text added: "!33"
- board text added: "!34"
- board text added: "!35"
- board text added: "+"
- board text added: "+3V"
- board text added: "+5V"
- board text added: "+5V pinhed"
- board text added: "-"
- board text added: "13"
- board text added: "14"
- board text added: "32"
- board text added: "33"
- board text added: "36"
- board text added: "39"
- board text added: "6-11V"
- board text added: "A"
- board text added: "B"
- board text added: "BAT_REF"
- board text added: "EN"
- board text added: "GND"
- board text added: "GPIO"
- board text added: "GPIO_34"
- board text added: "I-SERVO"
- board text added: "IO1"
- board text added: "IO3"
- board text added: "LED0"
- board text added: "LED1"
- board text added: "LED2"
- board text added: "LED3"
- board text added: "OFF"
- board text added: "ON"
- board text added: "OUT1"
- board text added: "OUT2"
- board text added: "OUT3"
- board text added: "OUT4"
- board text added: "POWER"
- board text added: "PWM0"
- board text added: "PWM1"
- board text added: "PWM2"
- board text added: "PWM3"
- board text added: "RB3202 SCHOOL-BOARD V1"
- board text added: "RB3202_SCHOOL-BOARD_V1"
- board text added: "SLP"
- board text added: "SW0"
- board text added: "SW1"
- board text added: "SW2"
- board text added: "SW3"
- board text added: "ULT"
- board text added: "VCC"

Commit message: DRV8833_jen_svab
Other:
- board text added: "7-11V"
- board text removed: "6-11V"
Changed lines of the file:
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@@
 <text x="57.0484" y="8.6868" size="1.2" layer="25" rot="R90">POWER</text>
 <text x="53.1368" y="57.658" size="2.54" layer="25">+</text>
-<text x="65.5828" y="51.2572" size="2.54" layer="26" rot="MR0">6-11V</text>
+<text x="65.5828" y="51.2572" size="2.54" layer="26" rot="MR0">7-11V</text>
 <text x="59.182" y="57.15" size="2.54" layer="26" rot="MR0">+</text>
 <text x="63.8048" y="57.3024" size="2.54" layer="26" rot="MR0">-</text>

Commit message: ir led pro encodery
Changed lines of the file:
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@@
 <layer number="47" name="Measures" color="7" fill="1" visible="no" active="yes"/>
 <layer number="48" name="Document" color="7" fill="1" visible="yes" active="yes"/>
-<layer number="49" name="Reference" color="7" fill="1" visible="no" active="yes"/>
+<layer number="49" name="Reference" color="7" fill="1" visible="yes" active="yes"/>
 <layer number="50" name="dxf" color="7" fill="1" visible="no" active="no"/>
 <layer number="51" name="tDocu" color="7" fill="1" visible="yes" active="yes"/>
@@
 <circle x="82.296" y="11.7348" radius="3" width="0.1524" layer="25"/>
 <rectangle x1="55.996" y1="21.9948" x2="75.996" y2="31.9948" layer="49" rot="R180"/>
-<dimension x1="0" y1="0" x2="94.996" y2="0" x3="47.498" y3="-12.7" textsize="1.778" layer="1"/>
-<dimension x1="93.98" y1="0" x2="94.0308" y2="59.8932" x3="121.9109125" y3="29.92293125" textsize="1.778" layer="1"/>
+<dimension x1="0" y1="0" x2="94.996" y2="0" x3="47.498" y3="-7.62" textsize="1.778" layer="49"/>
+<dimension x1="93.98" y1="0" x2="94.0308" y2="59.8932" x3="102.15661875" y3="29.939684375" textsize="1.778" layer="49"/>
 <text x="15.0368" y="23.622" size="1.2" layer="25" rot="R90">+3V</text>
 <text x="8.2296" y="12.3952" size="2" layer="25" rot="R180">GND</text>
@@
 <contactref element="X1" pad="2"/>
 <contactref element="JP12" pad="1"/>
-<polygon width="0.2" layer="1" thermals="no">
-<vertex x="87.796" y="41.7948"/>
-<vertex x="87.796" y="47.5948"/>
-<vertex x="80.796" y="54.5948"/>
-<vertex x="80.796" y="62.5348"/>
-<vertex x="76.096" y="62.5348"/>
-<vertex x="76.096" y="53.1948"/>
-<vertex x="77.396" y="51.8948"/>
-<vertex x="77.396" y="47.8948"/>
-<vertex x="79.196" y="46.0948"/>
-<vertex x="83.596" y="46.0948"/>
-<vertex x="85.596" y="44.0948"/>
-<vertex x="85.596" y="41.4948"/>
+<polygon width="0.5" layer="1">
+<vertex x="87.6436" y="41.6424"/>
+<vertex x="87.6436" y="47.544"/>
+<vertex x="80.5928" y="54.5948"/>
+<vertex x="80.5928" y="62.5348"/>
+<vertex x="76.2484" y="62.5348"/>
+<vertex x="76.2484" y="53.3472"/>
+<vertex x="77.5484" y="52.0472"/>
+<vertex x="77.5484" y="48.0472"/>
+<vertex x="79.3992" y="46.1964"/>
+<vertex x="83.6976" y="46.1964"/>
+<vertex x="85.6976" y="44.1964"/>
+<vertex x="85.6976" y="41.3932"/>
 <vertex x="85.996" y="41.0948"/>
 <vertex x="87.096" y="41.0948"/>

Commit message: eagle_librarys
Parts:
- turned JP1 to 180 degrees
Connections:
- removed net GPIO13-5V: IM11.11, JP1.3, JP3.2
- removed net GPIO14-5V: IM11.12, JP1.1, JP3.1
- removed net GPIO32_5V: IM11.7, JP1.7, JP3.4
- removed net GPIO33_5V: IM11.8, JP1.5, JP3.3
- new net GPIO12_5V: IM11.7, JP1.1, JP3.4
- new net GPIO14_5V: IM11.8, JP1.3, JP3.3
- new net GPIO32-5V: IM11.12, JP1.7, JP3.1
- new net GPIO33-5V: IM11.11, JP1.5, JP3.2
Routing:
- net GPIO12_5V: track 0.00 -> 48.6 mm
- net GPIO32_5V: track 46.4 -> 0.00 mm
- net GPIO14_5V: track 0.00 -> 44.8 mm
- net GPIO33_5V: track 42.7 -> 0.00 mm
- net GPIO33-5V: track 0.00 -> 35.9 mm
- net GPIO13-5V: track 33.8 -> 0.00 mm
- net GPIO32-5V: track 0.00 -> 32.7 mm
- net GPIO14-5V: track 30.5 -> 0.00 mm
- net SERVO_STEPDOWN_5V: track 23.2 -> 20.3 mm

Commit message: 2.KSK
Other:
- board text added: "12"
- board text removed: "13"
Changed lines of the file:
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@@
 <text x="19.05" y="51.4096" size="1.2" layer="25">GND</text>
 <text x="18.9992" y="53.8988" size="1.2" layer="25">+5V</text>
-<text x="9.0932" y="58.5216" size="1.2" layer="25">14</text>
-<text x="11.6332" y="58.5216" size="1.2" layer="25">13</text>
-<text x="14.1732" y="58.5216" size="1.2" layer="25">33</text>
-<text x="16.7132" y="58.5216" size="1.2" layer="25">32</text>
+<text x="16.7132" y="58.5216" size="1.2" layer="25">12</text>
+<text x="11.6332" y="58.5216" size="1.2" layer="25">33</text>
+<text x="14.1732" y="58.5216" size="1.2" layer="25">14</text>
+<text x="9.0932" y="58.5216" size="1.2" layer="25">32</text>
 <text x="57.0484" y="8.6868" size="1.2" layer="25" rot="R90">POWER</text>
 <text x="53.1368" y="57.658" size="2.54" layer="25">+</text>

Commit message: dokumentace ke SchoolBoardu
Routing:
- net GPIO22: track 80.8 -> 81.9 mm
- net OFF: track 94.7 -> 95.2 mm
Changed lines of the file:
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@@
 <wire x1="55.3688" y1="13.620825" x2="55.3688" y2="17.0656" width="0.3048" layer="1"/>
 <wire x1="47.9044" y1="2.8448" x2="47.9044" y2="6.1468" width="0.3048" layer="1"/>
-<wire x1="10.546" y1="39.6948" x2="10.546" y2="37.6378" width="0.3048" layer="16"/>
-<wire x1="10.546" y1="37.6378" x2="10.9252" y2="37.2586" width="0.3048" layer="16"/>
+<wire x1="10.546" y1="39.6948" x2="10.546" y2="37.714" width="0.3048" layer="16"/>
+<wire x1="10.546" y1="37.714" x2="13.5414" y2="34.7186" width="0.3048" layer="16"/>
 <via x="24.0751125" y="22.2209125" extent="1-16" drill="0.35"/>
-<wire x1="19.324425" y1="37.2586" x2="24.0751125" y2="32.5079125" width="0.3048" layer="16"/>
-<wire x1="10.9252" y1="37.2586" x2="19.324425" y2="37.2586" width="0.3048" layer="16"/>
+<wire x1="21.864425" y1="34.7186" x2="24.0751125" y2="32.5079125" width="0.3048" layer="16"/>
+<wire x1="13.5414" y1="34.7186" x2="21.864425" y2="34.7186" width="0.3048" layer="16"/>
 <wire x1="24.0751125" y1="32.5079125" x2="24.0751125" y2="22.2209125" width="0.3048" layer="16"/>
 <via x="44.831" y="13.3858" extent="1-16" drill="0.35"/>
@@
 <wire x1="45.3644" y1="6.1468" x2="45.3644" y2="2.8448" width="0.3048" layer="1"/>
 <via x="24.845725" y="21.467525" extent="1-16" drill="0.35"/>
-<wire x1="13.086" y1="39.6948" x2="15.0174" y2="37.7634" width="0.3048" layer="16"/>
-<wire x1="15.0174" y1="37.7634" x2="19.533525" y2="37.7634" width="0.3048" layer="16"/>
-<wire x1="19.533525" y1="37.7634" x2="24.845725" y2="32.4512" width="0.3048" layer="16"/>
+<wire x1="15.5766" y1="35.2234" x2="13.086" y2="37.714" width="0.3048" layer="16"/>
+<wire x1="13.086" y1="39.6948" x2="13.086" y2="37.714" width="0.3048" layer="16"/>
+<wire x1="15.5766" y1="35.2234" x2="22.073525" y2="35.2234" width="0.3048" layer="16"/>
+<wire x1="22.073525" y1="35.2234" x2="24.845725" y2="32.4512" width="0.3048" layer="16"/>
 <wire x1="24.845725" y1="32.4512" x2="24.845725" y2="21.467525" width="0.3048" layer="16"/>
 <wire x1="24.845725" y1="19.308525" x2="27.21165" y2="16.9426" width="0.3048" layer="1"/>
@@
 <wire x1="4.7276" y1="43.3864" x2="4.699" y2="43.3578" width="0.3048" layer="16"/>
 <wire x1="4.699" y1="43.3578" x2="4.699" y2="40.2082" width="0.3048" layer="16"/>
-<wire x1="4.699" y1="40.2082" x2="8.1534" y2="36.7538" width="0.3048" layer="16"/>
-<wire x1="17.653" y1="36.7538" x2="22.098" y2="32.3088" width="0.3048" layer="16"/>
-<wire x1="8.1534" y1="36.7538" x2="17.653" y2="36.7538" width="0.3048" layer="16"/>
+<wire x1="4.699" y1="40.2082" x2="10.6934" y2="34.2138" width="0.3048" layer="16"/>
+<wire x1="20.193" y1="34.2138" x2="22.098" y2="32.3088" width="0.3048" layer="16"/>
+<wire x1="10.6934" y1="34.2138" x2="20.193" y2="34.2138" width="0.3048" layer="16"/>
 <wire x1="4.7276" y1="43.87200625" x2="5.76279375" y2="44.9072" width="0.3048" layer="16"/>
 <wire x1="5.76279375" y1="44.9072" x2="13.8684" y2="44.9072" width="0.3048" layer="16"/>
@@
 <contactref element="SW5" pad="4"/>
 <contactref element="JP16" pad="8"/>
-<wire x1="67.546" y1="35.1028" x2="67.142" y2="34.6988" width="0.3048" layer="1"/>
-<wire x1="67.142" y1="34.6988" x2="67.142" y2="33.3858" width="0.3048" layer="1"/>
 <via x="64.516" y="33.7058" extent="1-16" drill="0.35"/>
 <wire x1="64.516" y1="33.7058" x2="64.836" y2="33.3858" width="0.3048" layer="1"/>
@@
 <wire x1="58.76960625" y1="40.0884" x2="65.2804" y2="40.0884" width="0.2032" layer="1"/>
 <wire x1="41.9096" y1="48.653" x2="50.20500625" y2="48.653" width="0.2032" layer="1"/>
+<wire x1="64.516" y1="33.7058" x2="64.516" y2="33.8588" width="0.2" layer="1"/>
+<wire x1="64.516" y1="33.8588" x2="66.103" y2="35.4458" width="0.2" layer="1"/>
 </signal>
 <signal name="SW2">
@@
 <signal name="GPIO14_5V">
 <contactref element="IM11" pad="8"/>
-<wire x1="19.558" y1="32.3088" x2="15.6178" y2="36.249" width="0.3048" layer="16"/>
-<wire x1="15.6178" y1="36.249" x2="7.9443" y2="36.249" width="0.3048" layer="16"/>
-<wire x1="7.9443" y1="36.249" x2="4.1942" y2="39.9991" width="0.3048" layer="16"/>
+<wire x1="19.558" y1="32.3088" x2="18.1578" y2="33.709" width="0.3048" layer="16"/>
+<wire x1="18.1578" y1="33.709" x2="10.4843" y2="33.709" width="0.3048" layer="16"/>
+<wire x1="10.4843" y1="33.709" x2="4.1942" y2="39.9991" width="0.3048" layer="16"/>
 <wire x1="4.1942" y1="44.05250625" x2="4.1942" y2="39.9991" width="0.3048" layer="16"/>
 <wire x1="11.8332" y1="45.412" x2="5.55369375" y2="45.412" width="0.3048" layer="16"/>
