File: ele/SchoolBot/v1.0/SchoolBoard.brd (EAGLE design)
At the start: 95 x 60 mm, 55 parts, among them X1 M8, X2 M8, X4 POWER_IN

Commit message: dalsi_text_a_firstbot
Routing:
- net VCC: track 71.4 -> 68.4 mm

Commit message: trochu v tom delam bordel
proste to neumim delat poredne tak tet delam tenhle bordel commit bych mel vse na gitu a budu se snazit to dal delat poradne
Routing:
- net EN: track 72.7 -> 71.8 mm
- net BAT-REF: track 36.0 -> 36.7 mm
Other:
- board text added: "RB3202 SCHOOL-BOARD V1.0.1"
- board text added: "RB3202_SCHOOL-BOARD_V1.0.1"
- board text removed: "RB3202 SCHOOL-BOARD V1"
- board text removed: "RB3202_SCHOOL-BOARD_V1"
