File: ele/SchoolBot/v1.0/SchoolBoard.sch (EAGLE design)
At the start: 62 parts, among them X1 M8, X2 M8, X4 POWER_IN

Commit message: RB3202_jednotny_konektor_na_motory
Parts:
- removed C7: (no value), rcl:CPOL-EUE5-10.5
- added JP12: (no value), pinhead:PINHD-1X6
- JP6: device pinhead:PINHD-2X4 -> pinhead:PINHD-1X6
Connections:
- net +5V: now also JP12.5; no longer JP6.1
- net ENC_A1: now also JP12.3; no longer JP6.6
- net ENC_A2: now also IM6.IO19, JP6.4; no longer IM6.IO18, JP6.3
- net ENC_B1: now also IM6.IO15, JP12.4; no longer IM6.IO19, JP6.4
- net ENC_B2: now also IM6.IO18, JP6.3; no longer IM6.IO15, JP6.5
- net GND: now also JP12.2, JP6.5; no longer C7.-, JP6.7, JP6.8
- net M1A: now also JP12.6
- net M1B: now also JP12.1
- net M2A: now also JP6.1
- net M2B: now also JP6.6
- net PWM0: now also IM6.IO0; no longer IM6.IO5
- net PWM1: now also IM6.IO16; no longer IM6.IO17
- net PWM2: now also IM6.IO17; no longer IM6.IO16
- net PWM3: now also IM6.IO5; no longer IM6.IO0
- net VCC: no longer C7.+

Commit message: eagle_librarys
Connections:
- removed net GPIO13-5V: IM11.HIGH2, JP1.3, JP3.2
- removed net GPIO14-5V: IM11.HIGH1, JP1.1, JP3.1
- removed net GPIO32_5V: IM11.HIGH4, JP1.7, JP3.4
- removed net GPIO33_5V: IM11.HIGH3, JP1.5, JP3.3
- new net GPIO12_5V: IM11.HIGH4, JP1.1, JP3.4
- new net GPIO14_5V: IM11.HIGH3, JP1.3, JP3.3
- new net GPIO32-5V: IM11.HIGH1, JP1.7, JP3.1
- new net GPIO33-5V: IM11.HIGH2, JP1.5, JP3.2
Other:
- moved on the sheet: JP1
Changed lines of the file:
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@@
 <attribute name="NAME" x="187.96" y="167.132" size="1.778" layer="95"/>
 </instance>
-<instance part="JP1" gate="A" x="292.1" y="132.08" smashed="yes">
-<attribute name="NAME" x="285.75" y="140.335" size="1.778" layer="95"/>
-<attribute name="VALUE" x="285.75" y="124.46" size="1.778" layer="96"/>
+<instance part="JP1" gate="A" x="292.1" y="134.62" smashed="yes" rot="MR180">
+<attribute name="NAME" x="285.75" y="141.605" size="1.778" layer="95" rot="MR180"/>
+<attribute name="VALUE" x="285.75" y="142.24" size="1.778" layer="96" rot="MR180"/>
 </instance>
 <instance part="JP7" gate="A" x="325.12" y="132.08" smashed="yes">
@@
 </segment>
 </net>
-<net name="GPIO32_5V" class="0">
+<net name="GPIO12_5V" class="0">
 <segment>
 <pinref part="IM11" gate="G$1" pin="HIGH4"/>
-<wire x1="264.16" y1="129.54" x2="274.32" y2="129.54" width="0.1524" layer="91"/>
-<label x="271.78" y="129.54" size="1.778" layer="95"/>
+<label x="266.7" y="129.54" size="1.778" layer="95"/>
+<pinref part="JP1" gate="A" pin="1"/>
+<wire x1="289.56" y1="129.54" x2="276.86" y2="129.54" width="0.1524" layer="91"/>
+<pinref part="JP3" gate="A" pin="4"/>
+<wire x1="276.86" y1="129.54" x2="264.16" y2="129.54" width="0.1524" layer="91"/>
+<wire x1="276.86" y1="129.54" x2="276.86" y2="114.3" width="0.1524" layer="91"/>
+<wire x1="276.86" y1="114.3" x2="289.56" y2="114.3" width="0.1524" layer="91"/>
+<junction x="276.86" y="129.54"/>
+</segment>
+</net>
+<net name="GPIO33-5V" class="0">
+<segment>
+<pinref part="IM11" gate="G$1" pin="HIGH2"/>
+<wire x1="264.16" y1="134.62" x2="281.94" y2="134.62" width="0.1524" layer="91"/>
+<label x="266.7" y="134.62" size="1.778" layer="95"/>
+<pinref part="JP1" gate="A" pin="5"/>
+<pinref part="JP3" gate="A" pin="2"/>
+<wire x1="281.94" y1="134.62" x2="289.56" y2="134.62" width="0.1524" layer="91"/>
+<wire x1="281.94" y1="134.62" x2="281.94" y2="119.38" width="0.1524" layer="91"/>
+<wire x1="281.94" y1="119.38" x2="289.56" y2="119.38" width="0.1524" layer="91"/>
+<junction x="281.94" y="134.62"/>
+</segment>
+</net>
+<net name="GPIO32-5V" class="0">
+<segment>
+<pinref part="IM11" gate="G$1" pin="HIGH1"/>
+<wire x1="264.16" y1="137.16" x2="284.48" y2="137.16" width="0.1524" layer="91"/>
+<label x="266.7" y="137.16" size="1.778" layer="95"/>
 <pinref part="JP1" gate="A" pin="7"/>
-<pinref part="JP3" gate="A" pin="4"/>
-<wire x1="274.32" y1="129.54" x2="289.56" y2="129.54" width="0.1524" layer="91"/>
-<wire x1="274.32" y1="129.54" x2="274.32" y2="114.3" width="0.1524" layer="91"/>
-<wire x1="274.32" y1="114.3" x2="289.56" y2="114.3" width="0.1524" layer="91"/>
-<junction x="274.32" y="129.54"/>
-</segment>
-</net>
-<net name="GPIO13-5V" class="0">
-<segment>
-<pinref part="IM11" gate="G$1" pin="HIGH2"/>
-<wire x1="264.16" y1="134.62" x2="279.4" y2="134.62" width="0.1524" layer="91"/>
-<label x="271.78" y="134.62" size="1.778" layer="95"/>
-<pinref part="JP1" gate="A" pin="3"/>
-<pinref part="JP3" gate="A" pin="2"/>
-<wire x1="279.4" y1="134.62" x2="289.56" y2="134.62" width="0.1524" layer="91"/>
-<wire x1="279.4" y1="134.62" x2="279.4" y2="119.38" width="0.1524" layer="91"/>
-<wire x1="279.4" y1="119.38" x2="289.56" y2="119.38" width="0.1524" layer="91"/>
-<junction x="279.4" y="134.62"/>
-</segment>
-</net>
-<net name="GPIO14-5V" class="0">
-<segment>
-<pinref part="IM11" gate="G$1" pin="HIGH1"/>
-<wire x1="264.16" y1="137.16" x2="281.94" y2="137.16" width="0.1524" layer="91"/>
-<label x="271.78" y="137.16" size="1.778" layer="95"/>
-<pinref part="JP1" gate="A" pin="1"/>
 <pinref part="JP3" gate="A" pin="1"/>
-<wire x1="281.94" y1="137.16" x2="289.56" y2="137.16" width="0.1524" layer="91"/>
-<wire x1="289.56" y1="121.92" x2="281.94" y2="121.92" width="0.1524" layer="91"/>
-<wire x1="281.94" y1="121.92" x2="281.94" y2="137.16" width="0.1524" layer="91"/>
-<junction x="281.94" y="137.16"/>
+<wire x1="284.48" y1="137.16" x2="289.56" y2="137.16" width="0.1524" layer="91"/>
+<wire x1="289.56" y1="121.92" x2="284.48" y2="121.92" width="0.1524" layer="91"/>
+<wire x1="284.48" y1="121.92" x2="284.48" y2="137.16" width="0.1524" layer="91"/>
+<junction x="284.48" y="137.16"/>
 </segment>
 </net>
@@
 </segment>
 </net>
-<net name="GPIO33_5V" class="0">
+<net name="GPIO14_5V" class="0">
 <segment>
 <pinref part="IM11" gate="G$1" pin="HIGH3"/>
-<wire x1="264.16" y1="132.08" x2="276.86" y2="132.08" width="0.1524" layer="91"/>
-<label x="271.78" y="132.08" size="1.778" layer="95"/>
-<pinref part="JP1" gate="A" pin="5"/>
+<label x="266.7" y="132.08" size="1.778" layer="95"/>
+<pinref part="JP1" gate="A" pin="3"/>
+<wire x1="264.16" y1="132.08" x2="279.4" y2="132.08" width="0.1524" layer="91"/>
 <pinref part="JP3" gate="A" pin="3"/>
-<wire x1="276.86" y1="132.08" x2="289.56" y2="132.08" width="0.1524" layer="91"/>
-<wire x1="289.56" y1="116.84" x2="276.86" y2="116.84" width="0.1524" layer="91"/>
-<wire x1="276.86" y1="116.84" x2="276.86" y2="132.08" width="0.1524" layer="91"/>
-<junction x="276.86" y="132.08"/>
+<wire x1="279.4" y1="132.08" x2="289.56" y2="132.08" width="0.1524" layer="91"/>
+<wire x1="289.56" y1="116.84" x2="279.4" y2="116.84" width="0.1524" layer="91"/>
+<wire x1="279.4" y1="116.84" x2="279.4" y2="132.08" width="0.1524" layer="91"/>
+<junction x="279.4" y="132.08"/>
 </segment>
 </net>
@@
 <net name="SERVO_STEPDOWN_5V" class="0">
 <segment>
+<wire x1="304.8" y1="129.54" x2="304.8" y2="132.08" width="0.1524" layer="91"/>
+<label x="292.1" y="144.78" size="1.778" layer="95"/>
 <pinref part="JP1" gate="A" pin="2"/>
-<wire x1="297.18" y1="137.16" x2="304.8" y2="137.16" width="0.1524" layer="91"/>
-<wire x1="304.8" y1="137.16" x2="304.8" y2="134.62" width="0.1524" layer="91"/>
+<wire x1="304.8" y1="132.08" x2="304.8" y2="134.62" width="0.1524" layer="91"/>
+<wire x1="304.8" y1="134.62" x2="304.8" y2="137.16" width="0.1524" layer="91"/>
+<wire x1="304.8" y1="137.16" x2="304.8" y2="144.78" width="0.1524" layer="91"/>
+<wire x1="297.18" y1="129.54" x2="304.8" y2="129.54" width="0.1524" layer="91"/>
 <pinref part="JP1" gate="A" pin="4"/>
-<wire x1="304.8" y1="134.62" x2="304.8" y2="132.08" width="0.1524" layer="91"/>
-<wire x1="304.8" y1="132.08" x2="304.8" y2="129.54" width="0.1524" layer="91"/>
-<wire x1="297.18" y1="134.62" x2="304.8" y2="134.62" width="0.1524" layer="91"/>
-<junction x="304.8" y="134.62"/>
-<pinref part="JP1" gate="A" pin="6"/>
 <wire x1="297.18" y1="132.08" x2="304.8" y2="132.08" width="0.1524" layer="91"/>
 <junction x="304.8" y="132.08"/>
+<pinref part="JP1" gate="A" pin="6"/>
+<wire x1="304.8" y1="134.62" x2="297.18" y2="134.62" width="0.1524" layer="91"/>
+<junction x="304.8" y="134.62"/>
 <pinref part="JP1" gate="A" pin="8"/>
-<wire x1="297.18" y1="129.54" x2="304.8" y2="129.54" width="0.1524" layer="91"/>
-<wire x1="304.8" y1="137.16" x2="304.8" y2="144.78" width="0.1524" layer="91"/>
+<wire x1="297.18" y1="137.16" x2="304.8" y2="137.16" width="0.1524" layer="91"/>
 <junction x="304.8" y="137.16"/>
-<label x="292.1" y="144.78" size="1.778" layer="95"/>
-</segment>
-</net>
+</segment>
+</net>

Commit message: postup_pajeni_a_nejake_datadhity
Changed lines of the file:
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@@
 <grid distance="0.1" unitdist="inch" unit="inch" style="lines" multiple="1" display="no" altdistance="0.01" altunitdist="inch" altunit="inch"/>
 <layers>
-<layer number="1" name="Top" color="4" fill="1" visible="no" active="no"/>
-<layer number="2" name="Route2" color="16" fill="1" visible="no" active="no"/>
-<layer number="3" name="Route3" color="17" fill="1" visible="no" active="no"/>
-<layer number="4" name="Route4" color="18" fill="1" visible="no" active="no"/>
-<layer number="5" name="Route5" color="19" fill="1" visible="no" active="no"/>
-<layer number="6" name="Route6" color="25" fill="1" visible="no" active="no"/>
-<layer number="7" name="Route7" color="26" fill="1" visible="no" active="no"/>
-<layer number="8" name="Route8" color="27" fill="1" visible="no" active="no"/>
-<layer number="9" name="Route9" color="28" fill="1" visible="no" active="no"/>
-<layer number="10" name="Route10" color="29" fill="1" visible="no" active="no"/>
-<layer number="11" name="Route11" color="30" fill="1" visible="no" active="no"/>
-<layer number="12" name="Route12" color="20" fill="1" visible="no" active="no"/>
-<layer number="13" name="Route13" color="21" fill="1" visible="no" active="no"/>
-<layer number="14" name="Route14" color="22" fill="1" visible="no" active="no"/>
-<layer number="15" name="Route15" color="23" fill="1" visible="no" active="no"/>
-<layer number="16" name="Bottom" color="1" fill="1" visible="no" active="no"/>
-<layer number="17" name="Pads" color="2" fill="1" visible="no" active="no"/>
-<layer number="18" name="Vias" color="2" fill="1" visible="no" active="no"/>
-<layer number="19" name="Unrouted" color="6" fill="1" visible="no" active="no"/>
-<layer number="20" name="Dimension" color="24" fill="1" visible="no" active="no"/>
-<layer number="21" name="tPlace" color="7" fill="1" visible="no" active="no"/>
-<layer number="22" name="bPlace" color="7" fill="1" visible="no" active="no"/>
-<layer number="23" name="tOrigins" color="15" fill="1" visible="no" active="no"/>
-<layer number="24" name="bOrigins" color="15" fill="1" visible="no" active="no"/>
-<layer number="25" name="tNames" color="7" fill="1" visible="no" active="no"/>
-<layer number="26" name="bNames" color="7" fill="1" visible="no" active="no"/>
-<layer number="27" name="tValues" color="7" fill="1" visible="no" active="no"/>
-<layer number="28" name="bValues" color="7" fill="1" visible="no" active="no"/>
+<layer number="1" name="Top" color="4" fill="1" visible="yes" active="no"/>
+<layer number="2" name="Route2" color="16" fill="1" visible="yes" active="no"/>
+<layer number="3" name="Route3" color="17" fill="1" visible="yes" active="no"/>
+<layer number="4" name="Route4" color="18" fill="1" visible="yes" active="no"/>
+<layer number="5" name="Route5" color="19" fill="1" visible="yes" active="no"/>
+<layer number="6" name="Route6" color="25" fill="1" visible="yes" active="no"/>
+<layer number="7" name="Route7" color="26" fill="1" visible="yes" active="no"/>
+<layer number="8" name="Route8" color="27" fill="1" visible="yes" active="no"/>
+<layer number="9" name="Route9" color="28" fill="1" visible="yes" active="no"/>
+<layer number="10" name="Route10" color="29" fill="1" visible="yes" active="no"/>
+<layer number="11" name="Route11" color="30" fill="1" visible="yes" active="no"/>
+<layer number="12" name="Route12" color="20" fill="1" visible="yes" active="no"/>
+<layer number="13" name="Route13" color="21" fill="1" visible="yes" active="no"/>
+<layer number="14" name="Route14" color="22" fill="1" visible="yes" active="no"/>
+<layer number="15" name="Route15" color="23" fill="1" visible="yes" active="no"/>
+<layer number="16" name="Bottom" color="1" fill="1" visible="yes" active="no"/>
+<layer number="17" name="Pads" color="2" fill="1" visible="yes" active="no"/>
+<layer number="18" name="Vias" color="2" fill="1" visible="yes" active="no"/>
+<layer number="19" name="Unrouted" color="6" fill="1" visible="yes" active="no"/>
+<layer number="20" name="Dimension" color="24" fill="1" visible="yes" active="no"/>
+<layer number="21" name="tPlace" color="7" fill="1" visible="yes" active="no"/>
+<layer number="22" name="bPlace" color="7" fill="1" visible="yes" active="no"/>
+<layer number="23" name="tOrigins" color="15" fill="1" visible="yes" active="no"/>
+<layer number="24" name="bOrigins" color="15" fill="1" visible="yes" active="no"/>
+<layer number="25" name="tNames" color="7" fill="1" visible="yes" active="no"/>
+<layer number="26" name="bNames" color="7" fill="1" visible="yes" active="no"/>
+<layer number="27" name="tValues" color="7" fill="1" visible="yes" active="no"/>
+<layer number="28" name="bValues" color="7" fill="1" visible="yes" active="no"/>
 <layer number="29" name="tStop" color="7" fill="3" visible="no" active="no"/>
 <layer number="30" name="bStop" color="7" fill="6" visible="no" active="no"/>
@@
 <layer number="35" name="tGlue" color="7" fill="4" visible="no" active="no"/>
 <layer number="36" name="bGlue" color="7" fill="5" visible="no" active="no"/>
-<layer number="37" name="tTest" color="7" fill="1" visible="no" active="no"/>
-<layer number="38" name="bTest" color="7" fill="1" visible="no" active="no"/>
+<layer number="37" name="tTest" color="7" fill="1" visible="yes" active="no"/>
+<layer number="38" name="bTest" color="7" fill="1" visible="yes" active="no"/>
 <layer number="39" name="tKeepout" color="4" fill="11" visible="no" active="no"/>
 <layer number="40" name="bKeepout" color="1" fill="11" visible="no" active="no"/>
@@
 <layer number="44" name="Drills" color="7" fill="1" visible="no" active="no"/>
 <layer number="45" name="Holes" color="7" fill="1" visible="no" active="no"/>
-<layer number="46" name="Milling" color="3" fill="1" visible="no" active="no"/>
-<layer number="47" name="Measures" color="7" fill="1" visible="no" active="no"/>
-<layer number="48" name="Document" color="7" fill="1" visible="no" active="no"/>
-<layer number="49" name="Reference" color="7" fill="1" visible="no" active="no"/>
-<layer number="50" name="dxf" color="7" fill="1" visible="no" active="no"/>
-<layer number="51" name="tDocu" color="7" fill="1" visible="no" active="no"/>
-<layer number="52" name="bDocu" color="7" fill="1" visible="no" active="no"/>
-<layer number="53" name="tGND_GNDA" color="7" fill="9" visible="no" active="no"/>
-<layer number="54" name="bGND_GNDA" color="1" fill="9" visible="no" active="no"/>
-<layer number="55" name="tPotisk" color="7" fill="1" visible="no" active="no"/>
-<layer number="56" name="wert" color="7" fill="1" visible="no" active="no"/>
-<layer number="57" name="tCAD" color="7" fill="1" visible="no" active="no"/>
-<layer number="58" name="bNC" color="7" fill="1" visible="no" active="no"/>
-<layer number="59" name="tCarbon" color="7" fill="1" visible="no" active="no"/>
-<layer number="60" name="bCarbon" color="7" fill="1" visible="no" active="no"/>
-<layer number="61" name="stand" color="7" fill="1" visible="no" active="no"/>
+<layer number="46" name="Milling" color="3" fill="1" visible="yes" active="no"/>
+<layer number="47" name="Measures" color="7" fill="1" visible="yes" active="no"/>
+<layer number="48" name="Document" color="7" fill="1" visible="yes" active="no"/>
+<layer number="49" name="Reference" color="7" fill="1" visible="yes" active="no"/>
+<layer number="50" name="dxf" color="7" fill="1" visible="yes" active="no"/>
+<layer number="51" name="tDocu" color="7" fill="1" visible="yes" active="no"/>
+<layer number="52" name="bDocu" color="7" fill="1" visible="yes" active="no"/>
+<layer number="53" name="tGND_GNDA" color="7" fill="9" visible="yes" active="no"/>
+<layer number="54" name="bGND_GNDA" color="1" fill="9" visible="yes" active="no"/>
+<layer number="55" name="tPotisk" color="7" fill="1" visible="yes" active="no"/>
+<layer number="56" name="wert" color="7" fill="1" visible="yes" active="no"/>
+<layer number="57" name="tCAD" color="7" fill="1" visible="yes" active="no"/>
+<layer number="58" name="bNC" color="7" fill="1" visible="yes" active="no"/>
+<layer number="59" name="tCarbon" color="7" fill="1" visible="yes" active="no"/>
+<layer number="60" name="bCarbon" color="7" fill="1" visible="yes" active="no"/>
+<layer number="61" name="stand" color="7" fill="1" visible="yes" active="no"/>
 <layer number="88" name="SimResults" color="9" fill="1" visible="no" active="yes"/>
 <layer number="89" name="SimProbes" color="9" fill="1" visible="yes" active="yes"/>
@@
 <part name="GND27" library="supply1" library_urn="urn:adsk.eagle:library:371" deviceset="GND" device=""/>
 <part name="P+8" library="supply1" library_urn="urn:adsk.eagle:library:371" deviceset="VCC" device=""/>
-<part name="C6" library="rcl" library_urn="urn:adsk.eagle:library:334" deviceset="CPOL-EU" device="E5-10.5" package3d_urn="urn:adsk.eagle:package:23372/1"/>
-<part name="RN2" library="resistor-dil" library_urn="urn:adsk.eagle:library:342" deviceset="4R-N" device="EXBS8V" package3d_urn="urn:adsk.eagle:package:24925/1"/>
-<part name="RN3" library="resistor-dil" library_urn="urn:adsk.eagle:library:342" deviceset="4R-N" device="EXBS8V" package3d_urn="urn:adsk.eagle:package:24925/1"/>
+<part name="C6" library="rcl" library_urn="urn:adsk.eagle:library:334" deviceset="CPOL-EU" device="E5-10.5" package3d_urn="urn:adsk.eagle:package:23372/2"/>
+<part name="RN2" library="resistor-dil" deviceset="4R-N" device="EXBS8V" package3d_urn="urn:adsk.eagle:package:24925/1"/>
+<part name="RN3" library="resistor-dil" deviceset="4R-N" device="EXBS8V" package3d_urn="urn:adsk.eagle:package:24925/1"/>
 <part name="JP1" library="pinhead" library_urn="urn:adsk.eagle:library:325" deviceset="PINHD-2X4" device="" package3d_urn="urn:adsk.eagle:package:22461/2"/>
 <part name="JP7" library="pinhead" library_urn="urn:adsk.eagle:library:325" deviceset="PINHD-1X4" device="" package3d_urn="urn:adsk.eagle:package:22407/2"/>
