File: ele/FirstTableBot/untitled.sch (EAGLE design)
At the start: 49 parts, among them Q1 FDN360P, X4 POWER_IN

Commit message: FirstTableBot
schema desky
Parts:
- removed Q1: FDN360P, transistor-power:FDN360P
- added Q3: (no value), transistors:N-MOSFET-SOT23-DIST
Connections:
- net +3V3: now also Q3.G; no longer Q1.G
- net GPIO21: now also Q3.S; no longer Q1.S
- net N$6: now also Q3.D; no longer Q1.D
Other:
- moved on the sheet: R7
Changed lines of the file:
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@@
 <layer number="112" name="tSilk" color="7" fill="1" visible="yes" active="yes"/>
 <layer number="113" name="ReferenceLS" color="7" fill="1" visible="no" active="no"/>
+<layer number="114" name="Senzor_teploty" color="7" fill="1" visible="yes" active="yes"/>
+<layer number="115" name="podporaDPS" color="7" fill="1" visible="yes" active="yes"/>
 <layer number="116" name="Patch_BOT" color="9" fill="4" visible="yes" active="yes"/>
+<layer number="117" name="stredy" color="7" fill="1" visible="yes" active="yes"/>
 <layer number="118" name="Rect_Pads" color="7" fill="1" visible="no" active="no"/>
+<layer number="119" name="osy" color="7" fill="1" visible="yes" active="yes"/>
+<layer number="120" name="_velikost1/2AA" color="7" fill="1" visible="yes" active="yes"/>
 <layer number="121" name="_tsilk" color="7" fill="1" visible="yes" active="yes"/>
 <layer number="122" name="_bsilk" color="7" fill="1" visible="yes" active="yes"/>
@@
 <layer number="128" name="_bValues" color="7" fill="1" visible="yes" active="yes"/>
 <layer number="129" name="Mask" color="7" fill="1" visible="yes" active="yes"/>
+<layer number="130" name="SMDSTROOK" color="7" fill="1" visible="yes" active="yes"/>
 <layer number="131" name="tAdjust" color="7" fill="1" visible="yes" active="yes"/>
 <layer number="132" name="bAdjust" color="7" fill="1" visible="yes" active="yes"/>
+<layer number="133" name="bottom_silk" color="7" fill="1" visible="yes" active="yes"/>
 <layer number="144" name="Drill_legend" color="7" fill="1" visible="yes" active="yes"/>
 <layer number="150" name="Notes" color="7" fill="1" visible="yes" active="yes"/>
@@
 <part name="GND13" library="supply1" library_urn="urn:adsk.eagle:library:371" deviceset="GND" device=""/>
 <part name="JP6" library="pinhead" library_urn="urn:adsk.eagle:library:325" deviceset="PINHD-1X3" device="" package3d_urn="urn:adsk.eagle:package:22458/2"/>
-<part name="Q1" library="transistor-power" library_urn="urn:adsk.eagle:library:400" deviceset="FDN360P" device="" package3d_urn="urn:adsk.eagle:package:29529/2"/>
 <part name="R6" library="resistor" library_urn="urn:adsk.eagle:library:348" deviceset="R-EU_" device="R0402" package3d_urn="urn:adsk.eagle:package:26058/2" value="5k"/>
 <part name="+3V1" library="supply1" library_urn="urn:adsk.eagle:library:371" deviceset="+3V3" device=""/>
@@
 <part name="R7" library="resistor" library_urn="urn:adsk.eagle:library:348" deviceset="R-EU_" device="R0402" package3d_urn="urn:adsk.eagle:package:26058/2" value="5k"/>
 <part name="GND14" library="supply1" library_urn="urn:adsk.eagle:library:371" deviceset="GND" device=""/>
+<part name="Q3" library="transistors" deviceset="N-MOSFET" device="-SOT23-DIST"/>
 </parts>
 <sheets>
@@
 </instance>
 <instance part="JP6" gate="A" x="233.68" y="78.74"/>
-<instance part="Q1" gate="G$1" x="213.36" y="78.74" rot="R90"/>
 <instance part="R6" gate="G$1" x="220.98" y="88.9" rot="R90"/>
 <instance part="+3V1" gate="G$1" x="205.74" y="101.6" smashed="yes">
@@
 <attribute name="VALUE" x="223.52" y="96.52" size="1.778" layer="96" rot="MR90"/>
 </instance>
-<instance part="R7" gate="G$1" x="200.66" y="73.66" rot="R90"/>
-<instance part="GND14" gate="1" x="220.98" y="63.5" smashed="yes">
-<attribute name="VALUE" x="218.44" y="60.96" size="1.778" layer="96"/>
+<instance part="R7" gate="G$1" x="200.66" y="88.9" rot="R270"/>
+<instance part="GND14" gate="1" x="220.98" y="66.04" smashed="yes">
+<attribute name="VALUE" x="218.44" y="63.5" size="1.778" layer="96"/>
+</instance>
+<instance part="Q3" gate="G$1" x="213.36" y="78.74" smashed="yes" rot="MR90">
+<attribute name="VALUE" x="213.36" y="67.31" size="1.778" layer="96" rot="MR90"/>
+<attribute name="NAME" x="209.55" y="86.36" size="1.778" layer="95" rot="MR180"/>
 </instance>
 </instances>
@@
 <pinref part="JP6" gate="A" pin="3"/>
 <wire x1="231.14" y1="76.2" x2="220.98" y2="76.2" width="0.1524" layer="91"/>
-<wire x1="220.98" y1="76.2" x2="220.98" y2="66.04" width="0.1524" layer="91"/>
+<wire x1="220.98" y1="76.2" x2="220.98" y2="68.58" width="0.1524" layer="91"/>
 <pinref part="GND14" gate="1" pin="GND"/>
 </segment>
@@
 <segment>
 <pinref part="+3V1" gate="G$1" pin="+3V3"/>
-<wire x1="205.74" y1="99.06" x2="205.74" y2="66.04" width="0.1524" layer="91"/>
-<wire x1="205.74" y1="66.04" x2="210.82" y2="66.04" width="0.1524" layer="91"/>
-<pinref part="Q1" gate="G$1" pin="G"/>
-<wire x1="210.82" y1="66.04" x2="210.82" y2="76.2" width="0.1524" layer="91"/>
+<wire x1="205.74" y1="99.06" x2="205.74" y2="96.52" width="0.1524" layer="91"/>
+<wire x1="205.74" y1="96.52" x2="205.74" y2="73.66" width="0.1524" layer="91"/>
+<wire x1="205.74" y1="73.66" x2="210.82" y2="73.66" width="0.1524" layer="91"/>
+<wire x1="210.82" y1="73.66" x2="210.82" y2="76.2" width="0.1524" layer="91"/>
 <pinref part="R7" gate="G$1" pin="1"/>
-<wire x1="200.66" y1="68.58" x2="200.66" y2="66.04" width="0.1524" layer="91"/>
-<wire x1="200.66" y1="66.04" x2="205.74" y2="66.04" width="0.1524" layer="91"/>
-<junction x="205.74" y="66.04"/>
+<wire x1="200.66" y1="93.98" x2="200.66" y2="96.52" width="0.1524" layer="91"/>
+<wire x1="200.66" y1="96.52" x2="205.74" y2="96.52" width="0.1524" layer="91"/>
+<junction x="205.74" y="96.52"/>
+<pinref part="Q3" gate="G$1" pin="G"/>
 </segment>
 </net>
@@
 </segment>
 <segment>
-<pinref part="Q1" gate="G$1" pin="S"/>
 <wire x1="208.28" y1="81.28" x2="200.66" y2="81.28" width="0.1524" layer="91"/>
 <label x="193.04" y="81.28" size="1.778" layer="95"/>
@@
 <pinref part="R7" gate="G$1" pin="2"/>
 <wire x1="200.66" y1="81.28" x2="193.04" y2="81.28" width="0.1524" layer="91"/>
-<wire x1="200.66" y1="78.74" x2="200.66" y2="81.28" width="0.1524" layer="91"/>
+<wire x1="200.66" y1="83.82" x2="200.66" y2="81.28" width="0.1524" layer="91"/>
 <junction x="200.66" y="81.28"/>
+<pinref part="Q3" gate="G$1" pin="S"/>
 </segment>
 </net>
@@
 <wire x1="55.88" y1="127" x2="66.04" y2="127" width="0.1524" layer="91"/>
 <label x="66.04" y="127" size="1.778" layer="95" rot="MR0"/>
+<junction x="66.04" y="127"/>
 </segment>
 </net>
@@
 <net name="N$6" class="0">
 <segment>
-<pinref part="Q1" gate="G$1" pin="D"/>
 <pinref part="JP6" gate="A" pin="1"/>
 <wire x1="218.44" y1="81.28" x2="220.98" y2="81.28" width="0.1524" layer="91"/>
@@
 <junction x="220.98" y="81.28"/>
 <pinref part="R6" gate="G$1" pin="1"/>
-</segment>
-</net>
+<pinref part="Q3" gate="G$1" pin="D"/>
+</segment>
+</net>
