File: ele/FirstTableBot/main_board.brd (EAGLE design)
At the start: 140 x 140 mm, 89 parts, among them X4 POWER_IN

Commit message: upravi elektra
Parts:
- removed JP2: (no value), pinhead:1X06
- removed LED0: BLUE, led:CHIPLED_1206
- removed RN2: (no value), resistor-dil:EXBS8V
- removed U$11: BA10358F-E2SOIC, Rohm:SOIC
- added JP1: (no value), pinhead:1X03
- added R29, R39, R42, R45, R48: (no value), resistor:R0805
- added R30, R31, R50, R51, R52, R53: (no value), resistor:R0603
- added R38, R41, R44, R47: 620, resistor:R0805
- added R40, R43, R46, R49: 10k, resistor:R0805
- added U$15: MCP6022-E/ST, MCP6022-E_ST:SOP65P640X120-8N
- LED4: value RED -> BLUE
- LED5: value GREEN -> BLUE; device led:LED3MM -> led:CHIPLED_1206
- R19, R62: value (none) -> 22m
- R21, R22: value 5k -> 10k
- R23: value (none) -> 10k
- R24: value (none) -> 620; device resistor:R0603 -> resistor:R0805
- moved LED5 293.2 mm to (-66.0, -279.4)
- moved C9 284.2 mm to (-58.4, -279.4), flipped to the top, turned to 0 degrees
- moved SW6 277.7 mm to (-63.5, -271.8), turned to 0 degrees
- moved LED4 255.4 mm to (-66.0, -251.5)
- moved C8 253.5 mm to (-58.4, -251.5), flipped to the top, turned to 0 degrees
- moved SW3 246.6 mm to (-63.5, -243.8), turned to 0 degrees
- moved LED2 237.6 mm to (-66.0, -223.5)
- moved C4 217.4 mm to (-58.4, -223.5), flipped to the top, turned to 0 degrees
- moved SW2 211.0 mm to (-63.5, -215.9)
- moved C3 210.0 mm to (-58.4, -195.6), flipped to the top, turned to 0 degrees
- moved SW1 203.6 mm to (-63.5, -188.0)
- moved LED1 190.4 mm to (-66.0, -195.6)
- moved R23 177.4 mm to (-68.6, -180.3)
- moved R24 166.1 mm to (-38.1, -147.3)
- moved C5 142.3 mm to (-43.2, -139.7), flipped to the top, turned to 0 degrees
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Connections:
- removed net MISO: JP2.5, U$8.PA2
- removed net MOSI: JP2.6, U$8.PA1
- removed net SW1: C3.2, JP4.8, LED2.A, RN2.7, SW1.3, SW1.4
- new net IR-LED-POWER: R1.1, R11.1, R13.1, R3.1, R5.1, R7.1, R9.1, U$8.PB2
- new net N$24: LED2.A, R41.2
- new net N$26: LED1.A, R38.2
- new net N$27: LED4.A, R44.2
- new net N$28: LED5.A, R47.2
- new net N$29: R51.2, R53.1, U$15.2
- new net N$30: R50.2, R52.1, U$15.6
- new net PC7: R47.1, R48.1, R49.1
- new net SW5: C3.2, JP4.8, R39.2, SW1.3, SW1.4
- net +3V3: now also R30.1, R31.1
- net +5V: now also JP1.2, R23.2, R40.2, R43.2, R46.2, R49.2; no longer JP2.2, R1.1, R11.1, R13.1, R3.1, R5.1, R7.1, R9.1
- net AMPLIFIED_I-MOT_A: now also R53.2, U$15.1; no longer U$11.OUT2
- net AMPLIFIED_I-MOT_B: now also R52.2, U$15.7; no longer U$11.OUT1
- net BAT_POL+: no longer R24.2
- net CDA: now also IM6.36, R30.2, U$8.PA2; no longer IM6.24, U$8.PB2
- net GND: now also JP1.3, LED5.C, R50.1, R51.1, U$15.4; no longer JP2.3, LED0.C, LED5.K, U$11.-IN2, U$11.-INT1, U$11.VEE
- net I-MOT_A: now also U$15.3; no longer U$11.+INT1
- net I-MOT_B: now also U$15.5; no longer U$11.+IN2
- net N$10: now also LED3.A, R24.2; no longer LED5.A, R24.1
- net PB3: now also R44.1, R45.1, R46.1; no longer R23.1
- net PC0: now also R23.1, R24.1, R29.1; no longer RN2.1
- net PC1: now also R38.1, R39.1, R40.1; no longer RN2.2
- net PC2: now also R41.1, R42.1, R43.1; no longer RN2.3
- net PC3: no longer RN2.4
- net RESET: now also JP1.1; no longer JP2.1
- net SCK: now also IM6.37, R31.2; no longer IM6.25, JP2.4
- net SW0: now also R29.2; no longer LED3.A, RN2.8
- net SW2: now also R42.2; no longer LED1.A, RN2.6
- net SW3: now also C9.2, R45.2, R48.2, SW6.3, SW6.4; no longer LED0.A, RN2.5
- net SW4: no longer C9.2, LED4.A, R23.2, SW6.3, SW6.4
- net VCC: now also U$15.8; no longer U$11.VCC

Commit message: schematická obměna OZ
Parts:
- removed U$15: MCP6022-E/ST, MCP6022-E_ST:SOP65P640X120-8N
- added IC1: MCP602ST, linear:TSSOP8
Connections:
- net RESET renamed !RESET
- net SCK renamed SCL
- net AMPLIFIED_I-MOT_A: now also IC1.1; no longer U$15.1
- net AMPLIFIED_I-MOT_B: now also IC1.7; no longer U$15.7
- net GND: now also IC1.4; no longer U$15.4
- net I-MOT_A: now also IC1.3; no longer U$15.3
- net I-MOT_B: now also IC1.5; no longer U$15.5
- net N$29: now also IC1.2; no longer U$15.2
- net N$30: now also IC1.6; no longer U$15.6
- net VCC: now also IC1.8; no longer U$15.8
Changed lines of the file:
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@@
 <attribute name="VALUE" x="-69.215" y="-294.64" size="1.27" layer="27"/>
-</element>
-<element name="U$15" library="MCP6022-E_ST" package="SOP65P640X120-8N" value="MCP6022-E/ST" x="-63.5" y="-302.26" smashed="yes">
-<attribute name="AVAILABILITY" value="Unavailable" x="-63.5" y="-302.26" size="1.778" layer="27" display="off"/>
-<attribute name="DESCRIPTION" value=" MCP6022 Series 5.5 V 10 MHz Rail-to-Rail I/O Operational Amplifier - TSSOP-8 " x="-63.5" y="-302.26" size="1.778" layer="27" display="off"/>
-<attribute name="MF" value="Microchip" x="-63.5" y="-302.26" size="1.778" layer="27" display="off"/>
-<attribute name="MP" value="MCP6022-E/ST" x="-63.5" y="-302.26" size="1.778" layer="27" display="off"/>
-<attribute name="NAME" x="-68.00353125" y="-300.35171875" size="2.08638125" layer="25" ratio="10" rot="SR0"/>
-<attribute name="PACKAGE" value="TSSOP-8 Microchip" x="-63.5" y="-302.26" size="1.778" layer="27" display="off"/>
-<attribute name="PRICE" value="None" x="-63.5" y="-302.26" size="1.778" layer="27" display="off"/>
-<attribute name="VALUE" x="-69.072490625" y="-306.07676875" size="2.0865" layer="27" ratio="10" rot="SR0"/>
 </element>
 <element name="R50" library="resistor" library_urn="urn:adsk.eagle:library:348" package="R0603" package3d_urn="urn:adsk.eagle:package:23555/3" value="" x="-68.58" y="-309.88" smashed="yes">
@@
 <attribute name="NAME" x="-69.215" y="-334.645" size="1.27" layer="25"/>
 <attribute name="VALUE" x="-69.215" y="-337.185" size="1.27" layer="27"/>
+</element>
+<element name="IC1" library="linear" library_urn="urn:adsk.eagle:library:262" package="TSSOP8" package3d_urn="urn:adsk.eagle:package:20813/2" value="MCP602ST" x="-76.2" y="-330.2" smashed="yes">
+<attribute name="NAME" x="-77.825" y="-333.125" size="1.27" layer="25" rot="R90"/>
+<attribute name="POPULARITY" value="0" x="-76.2" y="-330.2" size="1.778" layer="27" display="off"/>
+<attribute name="VALUE" x="-73.275" y="-333.45" size="1.27" layer="27" rot="R90"/>
 </element>
 </elements>
@@
 <contactref element="C9" pad="1"/>
 <contactref element="LED5" pad="C"/>
-<contactref element="U$15" pad="4"/>
 <contactref element="R50" pad="1"/>
 <contactref element="R51" pad="1"/>
+<contactref element="IC1" pad="4"/>
 <wire x1="-60.2488" y1="-185.6994" x2="-66.7512" y2="-185.6994" width="0" layer="19" extent="1-1"/>
 <wire x1="-66.04" y1="-193.83" x2="-66.7512" y2="-185.6994" width="0" layer="19" extent="1-1"/>
@@
 <wire x1="-66.04" y1="-277.65" x2="-66.7512" y2="-269.5194" width="0" layer="19" extent="1-1"/>
 <wire x1="-59.82" y1="-279.4" x2="-66.04" y2="-277.65" width="0" layer="19" extent="1-1"/>
-<wire x1="-66.3194" y1="-303.2252" x2="-59.82" y2="-279.4" width="0" layer="19" extent="1-1"/>
-<wire x1="-69.43" y1="-309.88" x2="-66.3194" y2="-303.2252" width="0" layer="19" extent="1-1"/>
+<wire x1="-69.43" y1="-309.88" x2="-59.82" y2="-279.4" width="0" layer="19" extent="1-1"/>
 <wire x1="-69.43" y1="-314.96" x2="-69.43" y2="-309.88" width="0" layer="19" extent="1-1"/>
+<wire x1="-75.225" y1="-333.125" x2="-69.43" y2="-314.96" width="0" layer="19" extent="1-1"/>
 <wire x1="-44.58" y1="-139.7" x2="-60.2488" y2="-185.6994" width="0" layer="19" extent="1-1"/>
 <wire x1="-43.18" y1="-130.33" x2="-44.58" y2="-139.7" width="0" layer="19" extent="1-1"/>
@@
 <wire x1="32.6" y1="-38.1" x2="44.45" y2="-47.41" width="0" layer="19" extent="1-1"/>
 </signal>
-<signal name="RESET">
-<contactref element="U$8" pad="PA0"/>
-<contactref element="JP1" pad="1"/>
-<wire x1="-45.295" y1="-0.635" x2="-68.58" y2="-106.68" width="0" layer="19" extent="1-1"/>
-</signal>
-<signal name="SCK">
-<contactref element="U$8" pad="PA3"/>
-<contactref element="IM6" pad="37"/>
-<contactref element="R31" pad="2"/>
-<wire x1="-45.295" y1="-4.445" x2="-67.73" y2="-335.28" width="0" layer="19" extent="1-1"/>
-<wire x1="57.15" y1="-12.7" x2="-45.295" y2="-4.445" width="0" layer="19" extent="1-1"/>
-</signal>
 <signal name="+3V3">
 <contactref element="R22" pad="1"/>
@@
 <contactref element="Q2" pad="7"/>
 <contactref element="Q2" pad="8"/>
-<contactref element="U$15" pad="8"/>
-<wire x1="49.53" y1="-27.94" x2="-60.6806" y2="-301.2948" width="0" layer="19" extent="1-1"/>
-<wire x1="66.04" y1="-10.15" x2="49.53" y2="-27.94" width="0" layer="19" extent="1-1"/>
-<wire x1="26.24" y1="-3.515" x2="49.53" y2="-27.94" width="0" layer="19" extent="1-1"/>
+<contactref element="IC1" pad="8"/>
+<wire x1="16.51" y1="-16.51" x2="-77.175" y2="-327.275" width="0" layer="19" extent="1-1"/>
+<wire x1="21.59" y1="-7.62" x2="16.51" y2="-16.51" width="0" layer="19" extent="1-1"/>
+<wire x1="26.24" y1="-3.515" x2="21.59" y2="-7.62" width="0" layer="19" extent="1-1"/>
 <wire x1="26.24" y1="-2.865" x2="26.24" y2="-3.515" width="0" layer="19" extent="1-1"/>
 <wire x1="26.24" y1="-2.215" x2="26.24" y2="-2.865" width="0" layer="19" extent="1-1"/>
 <wire x1="26.24" y1="-1.565" x2="26.24" y2="-2.215" width="0" layer="19" extent="1-1"/>
-<wire x1="21.59" y1="-7.62" x2="26.24" y2="-3.515" width="0" layer="19" extent="1-1"/>
 <wire x1="17.78" y1="-2.54" x2="21.59" y2="-7.62" width="0" layer="19" extent="1-1"/>
 <wire x1="8.38" y1="-0.284375" x2="17.78" y2="-2.54" width="0" layer="19" extent="1-1"/>
 <wire x1="6.77" y1="-3.81" x2="8.38" y2="-0.284375" width="0" layer="19" extent="1-1"/>
-<wire x1="16.51" y1="-16.51" x2="21.59" y2="-7.62" width="0" layer="19" extent="1-1"/>
 <wire x1="16.51" y1="16.51" x2="8.38" y2="-0.284375" width="0" layer="19" extent="1-1"/>
+<wire x1="49.53" y1="-27.94" x2="26.24" y2="-3.515" width="0" layer="19" extent="1-1"/>
+<wire x1="66.04" y1="-10.15" x2="49.53" y2="-27.94" width="0" layer="19" extent="1-1"/>
 </signal>
 <signal name="N$11">
@@
 <contactref element="U$9" pad="BISEN"/>
 <contactref element="R62" pad="2"/>
-<contactref element="U$15" pad="5"/>
-<wire x1="3.39" y1="-3.81" x2="-60.6806" y2="-303.2252" width="0" layer="19" extent="1-1"/>
+<contactref element="IC1" pad="5"/>
+<wire x1="3.39" y1="-3.81" x2="-75.225" y2="-327.275" width="0" layer="19" extent="1-1"/>
 <wire x1="1.78" y1="-0.853125" x2="3.39" y2="-3.81" width="0" layer="19" extent="1-1"/>
 </signal>
@@
 <contactref element="U$9" pad="AISEN"/>
 <contactref element="R19" pad="2"/>
-<contactref element="U$15" pad="3"/>
-<wire x1="1.78" y1="0.853125" x2="-66.3194" y2="-302.5902" width="0" layer="19" extent="1-1"/>
+<contactref element="IC1" pad="3"/>
+<wire x1="1.78" y1="0.853125" x2="-75.875" y2="-333.125" width="0" layer="19" extent="1-1"/>
 <wire x1="3.39" y1="3.81" x2="1.78" y2="0.853125" width="0" layer="19" extent="1-1"/>
 </signal>
 <signal name="AMPLIFIED_I-MOT_B">
-<contactref element="U$15" pad="7"/>
 <contactref element="R52" pad="2"/>
-<wire x1="-60.6806" y1="-301.9298" x2="-67.73" y2="-320.04" width="0" layer="19" extent="1-1"/>
+<contactref element="IC1" pad="7"/>
+<wire x1="-67.73" y1="-320.04" x2="-76.525" y2="-327.275" width="0" layer="19" extent="1-1"/>
 </signal>
 <signal name="AMPLIFIED_I-MOT_A">
-<contactref element="U$15" pad="1"/>
 <contactref element="R53" pad="2"/>
-<wire x1="-66.3194" y1="-301.2948" x2="-67.73" y2="-325.12" width="0" layer="19" extent="1-1"/>
+<contactref element="IC1" pad="1"/>
+<wire x1="-67.73" y1="-325.12" x2="-77.175" y2="-333.125" width="0" layer="19" extent="1-1"/>
 </signal>
 <signal name="N$13">
@@
 </signal>
 <signal name="N$29">
-<contactref element="U$15" pad="2"/>
 <contactref element="R51" pad="2"/>
 <contactref element="R53" pad="1"/>
+<contactref element="IC1" pad="2"/>
+<wire x1="-69.43" y1="-325.12" x2="-76.525" y2="-333.125" width="0" layer="19" extent="1-1"/>
 <wire x1="-67.73" y1="-314.96" x2="-69.43" y2="-325.12" width="0" layer="19" extent="1-1"/>
-<wire x1="-66.3194" y1="-301.9298" x2="-67.73" y2="-314.96" width="0" layer="19" extent="1-1"/>
 </signal>
 <signal name="N$30">
-<contactref element="U$15" pad="6"/>
 <contactref element="R50" pad="2"/>
 <contactref element="R52" pad="1"/>
+<contactref element="IC1" pad="6"/>
+<wire x1="-69.43" y1="-320.04" x2="-75.875" y2="-327.275" width="0" layer="19" extent="1-1"/>
 <wire x1="-67.73" y1="-309.88" x2="-69.43" y2="-320.04" width="0" layer="19" extent="1-1"/>
-<wire x1="-60.6806" y1="-302.5902" x2="-67.73" y2="-309.88" width="0" layer="19" extent="1-1"/>
+</signal>
+<signal name="SCL">
+<contactref element="U$8" pad="PA3"/>
+<contactref element="IM6" pad="37"/>
+<contactref element="R31" pad="2"/>
+<wire x1="-45.295" y1="-4.445" x2="-67.73" y2="-335.28" width="0" layer="19" extent="1-1"/>
+<wire x1="57.15" y1="-12.7" x2="-45.295" y2="-4.445" width="0" layer="19" extent="1-1"/>
+</signal>
+<signal name="!RESET">
+<contactref element="U$8" pad="PA0"/>
+<contactref element="JP1" pad="1"/>
+<wire x1="-45.295" y1="-0.635" x2="-68.58" y2="-106.68" width="0" layer="19" extent="1-1"/>
 </signal>
 </signals>

Commit message: serialiyovani ir-led encoderu a zpetivoltovac I2C
Parts:
- removed R30, R31, R33, R35: (no value), resistor:R0603
- removed U$10, U$12, U$14: L-NP-3C1, led-brt:L-NP-3C1
- removed U$17, U$18, U$19: BIR-NM13C1, led-brt:BIR-NM13C1
- added Q1, Q4: (no value), transistors:SOT23_DIST
- added R36, R37, R54, R55: (no value), resistor:R0603
- added U$11, U$15, U$20: BIR-NM13C1, led-brt:BIR-NM13C1
- added U$21, U$22, U$23: L-NP-3C1, led-brt:L-NP-3C1
- R26, R27, R28, R32: value (none) -> 10k; device resistor:R0603 -> resistor:R0402
- moved R32 455.0 mm to (-76.2, -403.9), turned to 0 degrees
- moved R28 317.8 mm to (-76.2, -398.8)
- moved R26 305.1 mm to (-76.2, -381.0)
- moved R27 304.9 mm to (-76.2, -386.1)
Connections:
- removed net N$18: R26.2, U$17.PIN
- removed net N$19: R27.2, U$18.PIN
- removed net N$20: R28.2, U$19.PIN
- new net N$21: U$11.PIN, U$16.GND
- new net N$22: R36.2, U$15.PIN
- new net N$31: U$15.GND, U$20.PIN
- new net SCL-5V: Q4.3, R28.1, U$8.PA2
- new net SDA: Q1.2, R27.2
- new net SDA-5V: Q1.3, R26.1, U$8.PA1
- net +3V3: now also Q1.1, Q4.1, R27.1, R32.1; no longer R30.1, R31.1
- net +5V: now also R26.2, R28.2, R36.1, R37.1, R54.1, R55.1; no longer R26.1, R27.1, R28.1, R32.1, R33.1, R35.1
- net CDA: no longer R30.2, U$8.PA2
- net ENC-A0: now also R54.2, U$22.PIN; no longer R32.2, U$10.PIN
- net ENC-A1: now also R55.2, U$23.PIN; no longer R33.2, U$12.PIN
- net ENC-B1: now also R37.2, U$21.PIN; no longer R35.2, U$14.PIN
- net GND: now also U$11.GND, U$20.GND, U$21.GND, U$22.GND, U$23.GND; no longer U$10.GND, U$12.GND, U$14.GND, U$16.GND, U$17.GND, U$18.GND, U$19.GND
- net SCL: now also Q4.2, R32.2; no longer R31.2, U$8.PA3

Commit message: dolni propust k zesilovacum
Parts:
- added C10, C11, C12, C13: (no value), resistor:C1206
- added R30, R31, R33, R35: (no value), resistor:R0603
- moved R51 129.8 mm to (-76.2, -444.5)
- moved R53 124.7 mm to (-76.2, -449.6)
Connections:
- removed net N$29: IC1.2, R51.2, R53.1
- new net N$18: C11.1, R30.2, R31.1
- new net N$19: C10.1, IC1.5, R30.1
- new net N$20: IC1.2, R33.2, R35.1
- new net N$32: C13.1, R51.2, R53.1
- new net N$33: C12.1, IC1.3, R51.1
- net +3V3: now also IC1.8
- net AMPLIFIED_I-MOT_A: now also C13.2, R35.2; no longer R53.2
- net AMPLIFIED_I-MOT_B: now also C11.2
- net GND: now also C10.2, C12.2, R33.1; no longer R51.1
- net I-MOT_A: now also R53.2; no longer IC1.3
- net I-MOT_B: now also R31.2; no longer IC1.5
- net VCC: no longer IC1.8
