File: ele/FirstTableBot/main_board.brd (EAGLE design)
At the start: 140 x 140 mm, 116 parts, among them IC1 MCP602ST, X4 POWER_IN

Commit message: napajeni IR-led senzoru
Parts:
- removed R13, R3, R7: (no value), resistor:R0603
- added Q8: (no value), transistors:MLP3.3X3.3_HS
Connections:
- removed net N$7: R13.2, U$7.A
- new net N$29: U$6.K, U$7.A
- new net N$34: Q8.1, Q8.2, Q8.3, R1.1, R11.1, R5.1, R9.1
- net +5V: now also Q8.5, Q8.6, Q8.7, Q8.8
- net GND: no longer U$2.K, U$3.K, U$6.K
- net IR-LED-POWER: now also Q8.4; no longer R1.1, R11.1, R13.1, R3.1, R5.1, R7.1, R9.1
- net N$2: now also U$2.K; no longer R3.2
- net N$4: now also U$3.K; no longer R7.2
Changed lines of the file:
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@@
 <attribute name="VALUE" x="46.355" y="-48.895" size="1.27" layer="27" rot="R90"/>
-</element>
-<element name="R13" library="resistor" library_urn="urn:adsk.eagle:library:348" package="R0603" package3d_urn="urn:adsk.eagle:package:23555/3" value="" x="-44.45" y="-48.26" smashed="yes" rot="R270">
-<attribute name="NAME" x="-43.815" y="-47.625" size="1.27" layer="25" rot="R270"/>
-<attribute name="VALUE" x="-46.355" y="-47.625" size="1.27" layer="27" rot="R270"/>
 </element>
 <element name="R14" library="resistor" library_urn="urn:adsk.eagle:library:348" package="R0603" package3d_urn="urn:adsk.eagle:package:23555/3" value="" x="-36.83" y="-48.26" smashed="yes" rot="R90">
@@
 <attribute name="VALUE" x="-52.705" y="-9.525" size="1.27" layer="27" rot="R180"/>
 </element>
-<element name="R3" library="resistor" library_urn="urn:adsk.eagle:library:348" package="R0603" package3d_urn="urn:adsk.eagle:package:23555/3" value="" x="-59.69" y="-9.017" smashed="yes" rot="R180">
-<attribute name="NAME" x="-59.055" y="-9.652" size="1.27" layer="25" rot="R180"/>
-<attribute name="VALUE" x="-59.055" y="-7.112" size="1.27" layer="27" rot="R180"/>
-</element>
 <element name="R34" library="resistor" library_urn="urn:adsk.eagle:library:348" package="R0603" package3d_urn="urn:adsk.eagle:package:23555/3" value="" x="-31.75" y="-38.1" smashed="yes">
 <attribute name="NAME" x="-32.385" y="-37.465" size="1.27" layer="25"/>
@@
 <attribute name="NAME" x="1.27" y="-2.54" size="1.27" layer="25"/>
 <attribute name="VALUE" x="1.27" y="-6.35" size="1.27" layer="27"/>
-</element>
-<element name="R7" library="resistor" library_urn="urn:adsk.eagle:library:348" package="R0603" package3d_urn="urn:adsk.eagle:package:23555/3" value="" x="44.45" y="48.26" smashed="yes" rot="R90">
-<attribute name="NAME" x="43.815" y="47.625" size="1.27" layer="25" rot="R90"/>
-<attribute name="VALUE" x="46.355" y="47.625" size="1.27" layer="27" rot="R90"/>
 </element>
 <element name="R8" library="resistor" library_urn="urn:adsk.eagle:library:348" package="R0603" package3d_urn="urn:adsk.eagle:package:23555/3" value="" x="36.83" y="48.26" smashed="yes" rot="R270">
@@
 <attribute name="NAME" x="-77.47" y="-453.39" size="1.27" layer="25"/>
 <attribute name="VALUE" x="-77.47" y="-457.2" size="1.27" layer="27"/>
+</element>
+<element name="Q8" library="transistors" package="MLP3.3X3.3_HS" value="" x="-73.66" y="-467.36" smashed="yes">
+<attribute name="NAME" x="-76.76" y="-464.76" size="1.27" layer="25" font="vector" ratio="16"/>
+<attribute name="VALUE" x="-76.76" y="-471.26" size="1.27" layer="27" font="vector" ratio="16"/>
 </element>
 </elements>
@@
 <contactref element="IM6" pad="32"/>
 <contactref element="IM6" pad="38"/>
-<contactref element="U$2" pad="K"/>
 <contactref element="U$2" pad="E"/>
 <contactref element="U$1" pad="K"/>
 <contactref element="U$1" pad="E"/>
-<contactref element="U$3" pad="K"/>
 <contactref element="U$3" pad="E"/>
 <contactref element="U$4" pad="K"/>
@@
 <contactref element="U$5" pad="K"/>
 <contactref element="U$5" pad="E"/>
-<contactref element="U$6" pad="K"/>
 <contactref element="U$6" pad="E"/>
-<contactref element="U$7" pad="K"/>
 <contactref element="U$7" pad="E"/>
 <contactref element="X4" pad="1"/>
@@
 <contactref element="C12" pad="2"/>
 <contactref element="IC1" pad="4"/>
+<contactref element="U$7" pad="K"/>
 <wire x1="-60.2488" y1="-185.6994" x2="-66.7512" y2="-185.6994" width="0" layer="19" extent="1-1"/>
 <wire x1="-66.04" y1="-193.83" x2="-66.7512" y2="-185.6994" width="0" layer="19" extent="1-1"/>
@@
 <wire x1="-45.295" y1="-5.715" x2="-49.53" y2="-21.59" width="0" layer="19" extent="1-1"/>
 <wire x1="-50.8" y1="1.27" x2="-45.295" y2="-5.715" width="0" layer="19" extent="1-1"/>
-<wire x1="-53.34" y1="-1.27" x2="-50.8" y2="1.27" width="0" layer="19" extent="1-1"/>
-<wire x1="-58.42" y1="-3.81" x2="-53.34" y2="-1.27" width="0" layer="19" extent="1-1"/>
+<wire x1="-58.42" y1="-3.81" x2="-50.8" y2="1.27" width="0" layer="19" extent="1-1"/>
 <wire x1="-60.96" y1="-6.35" x2="-58.42" y2="-3.81" width="0" layer="19" extent="1-1"/>
-<wire x1="-60.96" y1="3.81" x2="-58.42" y2="-3.81" width="0" layer="19" extent="1-1"/>
-<wire x1="-58.42" y1="6.35" x2="-60.96" y2="3.81" width="0" layer="19" extent="1-1"/>
+<wire x1="-58.42" y1="6.35" x2="-50.8" y2="1.27" width="0" layer="19" extent="1-1"/>
 <wire x1="1.8288" y1="-7.8994" x2="-25.4" y2="-38.1" width="0" layer="19" extent="1-1"/>
 <wire x1="1.69" y1="-3.81" x2="1.8288" y2="-7.8994" width="0" layer="19" extent="1-1"/>
@@
 <wire x1="52.07" y1="-27.94" x2="44.45" y2="-12.7" width="0" layer="19" extent="1-1"/>
 <wire x1="41.91" y1="-46.99" x2="52.07" y2="-27.94" width="0" layer="19" extent="1-1"/>
-<wire x1="39.37" y1="-49.53" x2="41.91" y2="-46.99" width="0" layer="19" extent="1-1"/>
 <wire x1="39.37" y1="46.99" x2="26.67" y2="12.7" width="0" layer="19" extent="1-1"/>
 <wire x1="41.91" y1="49.53" x2="39.37" y2="46.99" width="0" layer="19" extent="1-1"/>
@@
 <contactref element="R26" pad="2"/>
 <contactref element="R28" pad="2"/>
+<contactref element="Q8" pad="7"/>
+<contactref element="Q8" pad="8"/>
+<contactref element="Q8" pad="5"/>
+<contactref element="Q8" pad="6"/>
 <wire x1="-67.63" y1="-208.28" x2="-67.63" y2="-180.34" width="0" layer="19" extent="1-1"/>
 <wire x1="-67.63" y1="-236.22" x2="-67.63" y2="-208.28" width="0" layer="19" extent="1-1"/>
@@
 <wire x1="-75.55" y1="-381" x2="-77.05" y2="-368.3" width="0" layer="19" extent="1-1"/>
 <wire x1="-75.55" y1="-398.78" x2="-75.55" y2="-381" width="0" layer="19" extent="1-1"/>
+<wire x1="-74.635" y1="-465.66" x2="-75.55" y2="-398.78" width="0" layer="19" extent="1-1"/>
+<wire x1="-73.985" y1="-465.66" x2="-74.635" y2="-465.66" width="0" layer="19" extent="1-1"/>
+<wire x1="-73.335" y1="-465.66" x2="-73.985" y2="-465.66" width="0" layer="19" extent="1-1"/>
+<wire x1="-72.685" y1="-465.66" x2="-73.335" y2="-465.66" width="0" layer="19" extent="1-1"/>
 <wire x1="-66.04" y1="-106.68" x2="-67.63" y2="-180.34" width="0" layer="19" extent="1-1"/>
 <wire x1="-69.43" y1="-76.2" x2="-66.04" y2="-106.68" width="0" layer="19" extent="1-1"/>
@@
 </signal>
 <signal name="N$2">
-<contactref element="R3" pad="2"/>
 <contactref element="U$1" pad="A"/>
-<wire x1="-60.54" y1="-9.017" x2="-60.96" y2="-3.81" width="0" layer="19" extent="1-1"/>
+<contactref element="U$2" pad="K"/>
+<wire x1="-53.34" y1="-1.27" x2="-60.96" y2="-3.81" width="0" layer="19" extent="1-1"/>
 </signal>
 <signal name="N$3">
@@
 </signal>
 <signal name="N$4">
-<contactref element="R7" pad="2"/>
 <contactref element="U$4" pad="A"/>
-<wire x1="41.91" y1="46.99" x2="44.45" y2="49.11" width="0" layer="19" extent="1-1"/>
+<contactref element="U$3" pad="K"/>
+<wire x1="-60.96" y1="3.81" x2="41.91" y2="46.99" width="0" layer="19" extent="1-1"/>
 </signal>
 <signal name="N$5">
@@
 <contactref element="U$6" pad="A"/>
 <wire x1="39.37" y1="-46.99" x2="36.83" y2="-49.11" width="0" layer="19" extent="1-1"/>
-</signal>
-<signal name="N$7">
-<contactref element="R13" pad="2"/>
-<contactref element="U$7" pad="A"/>
-<wire x1="-44.45" y1="-49.11" x2="-41.91" y2="-46.99" width="0" layer="19" extent="1-1"/>
 </signal>
 <signal name="BAT_POL+">
@@
 <signal name="IR-LED-POWER">
 <contactref element="U$8" pad="PB2"/>
-<contactref element="R11" pad="1"/>
-<contactref element="R13" pad="1"/>
-<contactref element="R1" pad="1"/>
-<contactref element="R3" pad="1"/>
-<contactref element="R5" pad="1"/>
-<contactref element="R7" pad="1"/>
-<contactref element="R9" pad="1"/>
-<wire x1="-58.84" y1="-9.017" x2="-44.45" y2="-47.41" width="0" layer="19" extent="1-1"/>
-<wire x1="-51.22" y1="3.81" x2="-58.84" y2="-9.017" width="0" layer="19" extent="1-1"/>
-<wire x1="-58.84" y1="8.89" x2="-51.22" y2="3.81" width="0" layer="19" extent="1-1"/>
-<wire x1="-35.985" y1="4.445" x2="-51.22" y2="3.81" width="0" layer="19" extent="1-1"/>
-<wire x1="-44.45" y1="47.41" x2="-58.84" y2="8.89" width="0" layer="19" extent="1-1"/>
-<wire x1="36.83" y1="-47.41" x2="-44.45" y2="-47.41" width="0" layer="19" extent="1-1"/>
-<wire x1="44.45" y1="47.41" x2="-44.45" y2="47.41" width="0" layer="19" extent="1-1"/>
+<contactref element="Q8" pad="4"/>
+<wire x1="-72.685" y1="-469.06" x2="-35.985" y2="4.445" width="0" layer="19" extent="1-1"/>
 </signal>
 <signal name="SW5">
@@
 <wire x1="-75.875" y1="-333.125" x2="-77.6" y2="-429.26" width="0" layer="19" extent="1-1"/>
 </signal>
+<signal name="N$29">
+<contactref element="U$7" pad="A"/>
+<contactref element="U$6" pad="K"/>
+<wire x1="39.37" y1="-49.53" x2="-41.91" y2="-46.99" width="0" layer="19" extent="1-1"/>
+</signal>
+<signal name="N$34">
+<contactref element="R1" pad="1"/>
+<contactref element="Q8" pad="2"/>
+<contactref element="Q8" pad="1"/>
+<contactref element="Q8" pad="3"/>
+<contactref element="R5" pad="1"/>
+<contactref element="R9" pad="1"/>
+<contactref element="R11" pad="1"/>
+<wire x1="-51.22" y1="3.81" x2="-58.84" y2="8.89" width="0" layer="19" extent="1-1"/>
+<wire x1="-44.45" y1="47.41" x2="-58.84" y2="8.89" width="0" layer="19" extent="1-1"/>
+<wire x1="36.83" y1="-47.41" x2="-51.22" y2="3.81" width="0" layer="19" extent="1-1"/>
+<wire x1="-73.335" y1="-469.06" x2="36.83" y2="-47.41" width="0" layer="19" extent="1-1"/>
+<wire x1="-73.985" y1="-469.06" x2="-73.335" y2="-469.06" width="0" layer="19" extent="1-1"/>
+<wire x1="-74.635" y1="-469.06" x2="-73.985" y2="-469.06" width="0" layer="19" extent="1-1"/>
+</signal>
 </signals>

Commit message: piniste
Parts:
- added JP2, JP7, JP8: (no value), pinhead:2X13
- moved R22 507.0 mm to (-71.1, -518.2), turned to 0 degrees
- moved R21 503.6 mm to (-76.2, -518.2), turned to 0 degrees
- moved JP6 492.0 mm to (-73.7, -513.1)
- moved Q3 490.8 mm to (-76.2, -505.5), turned to 0 degrees
Connections:
- removed net GPIO21: Q3.2, R22.2
- removed net GPIO33: R20.2
- new net BAT-REF: IM6.8, R20.2
- new net I-LED: IM6.33, Q3.2, R22.2
- new net IO13: IM6.15, JP2.19, JP2.20
- new net IO14: IM6.12, JP2.17, JP2.18
- new net IO16: IM6.27, JP2.15, JP2.16
- new net IO17: IM6.28, JP2.13, JP2.14
- new net IO18: IM6.30, JP2.11, JP2.12
- new net IO19: IM6.31, JP2.10, JP2.9
- new net IO25: IM6.9, JP2.7, JP2.8
- new net IO26: IM6.10, JP2.5, JP2.6
- new net IO27: IM6.11, JP2.3, JP2.4
- new net IO32: IM6.7, JP2.1, JP2.2
- new net IO4: IM6.26, JP2.21, JP2.22
- new net RX: IM6.34, JP2.25, JP2.26
- new net TX: IM6.35, JP2.23, JP2.24
- net +3V3: now also JP7.10, JP7.12, JP7.14, JP7.16, JP7.18, JP7.2, JP7.20, JP7.22, JP7.24, JP7.26, JP7.4, JP7.6, JP7.8, JP8.10, JP8.12, JP8.14, JP8.16, JP8.18, JP8.2, JP8.20, JP8.22, JP8.24, JP8.26, JP8.4, JP8.6, JP8.8, R34.1, R37.1, R54.1, R55.1
- net +5V: no longer R34.1, R37.1, R54.1, R55.1
- net GND: now also JP7.1, JP7.11, JP7.13, JP7.15, JP7.17, JP7.19, JP7.21, JP7.23, JP7.25, JP7.3, JP7.5, JP7.7, JP7.9, JP8.1, JP8.11, JP8.13, JP8.15, JP8.17, JP8.19, JP8.21, JP8.23, JP8.25, JP8.3, JP8.5, JP8.7, JP8.9
- net PWM_A1: now also IM6.23; no longer IM6.27
- net PWM_B0: now also IM6.25; no longer IM6.28
- net SLEEP: now also IM6.24

Commit message: zesilovace
Parts:
- R33, R50: value (none) -> 100
- R35, R52: value (none) -> 10k
- moved JP4 402.5 mm to (-71.1, -525.8)
Connections:
- removed net SW5: C3.2, JP4.8, R39.2, SW1.3, SW1.4
- new net SW1: C3.2, JP4.7, R39.2, SW1.3, SW1.4
- net GND: now also JP4.10, JP4.2, JP4.4, JP4.6, JP4.8; no longer JP4.1, JP4.3, JP4.5, JP4.7, JP4.9
- net SW0: now also JP4.9; no longer JP4.10
- net SW2: now also JP4.5; no longer JP4.6
- net SW3: now also JP4.3; no longer C8.2, JP4.4, R45.2, SW3.3, SW3.4
- net SW4: now also C8.2, JP4.1, R45.2, SW3.3, SW3.4; no longer JP4.2

Commit message: napájení z powerbanki
Parts:
- added K1: ARK550/2, #PaJa_konektory:ARK550/2
- added Q7: (no value), transistors:MLP3.3X3.3_HS
- added Q9: (no value), transistors:SOT23
- added R3: 2M, rcl_upravena:R0805
- added R7: 100k, rcl_upravena:R0805
- moved JP5 595.3 mm to (-91.4, -569.0)
- moved R16 556.8 mm to (-83.8, -538.5), turned to 0 degrees
- moved JP3 555.4 mm to (-91.4, -561.3)
Connections:
- new net N$35: Q7.4, Q9.1, R7.2
- new net N$7: Q2.5, Q2.6, Q2.7, Q2.8, Q9.2, R3.1, R7.1
- net +5V: now also JP3.2, JP5.2, K1.2, Q7.5, Q7.6, Q7.7, Q7.8
- net GND: now also K1.1, R3.2
- net VCC: now also Q7.1, Q7.2, Q7.3, Q9.3; no longer JP3.2, JP5.2, Q2.5, Q2.6, Q2.7, Q2.8
