File: ele/FirstTableBot/main_board.brd (EAGLE design)
At the start: 140 x 140 mm, 122 parts, among them IC1 MCP602ST, K1 ARK550/2, X4 POWER_IN

Commit message: nastrel_textu
Connections:
- net N$7: now also Q9.3; no longer Q9.2
- net VCC: now also Q9.2; no longer Q9.3
Changed lines of the file:
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@@
 <contactref element="C23" pad="2"/>
 <contactref element="IM3" pad="IN"/>
-<contactref element="Q9" pad="3"/>
 <contactref element="Q7" pad="1"/>
 <contactref element="Q7" pad="3"/>
 <contactref element="Q7" pad="2"/>
-<wire x1="-84.145" y1="-524.94" x2="-83.82" y2="-532.3" width="0" layer="19" extent="1-1"/>
+<contactref element="Q9" pad="2"/>
+<wire x1="-83.495" y1="-524.94" x2="-82.87" y2="-534.5" width="0" layer="19" extent="1-1"/>
+<wire x1="-84.145" y1="-524.94" x2="-83.495" y2="-524.94" width="0" layer="19" extent="1-1"/>
 <wire x1="-84.795" y1="-524.94" x2="-84.145" y2="-524.94" width="0" layer="19" extent="1-1"/>
-<wire x1="-83.495" y1="-524.94" x2="-84.145" y2="-524.94" width="0" layer="19" extent="1-1"/>
 <wire x1="49.53" y1="-27.94" x2="-83.495" y2="-524.94" width="0" layer="19" extent="1-1"/>
 <wire x1="66.04" y1="-10.15" x2="49.53" y2="-27.94" width="0" layer="19" extent="1-1"/>
@@
 <contactref element="Q2" pad="8"/>
 <contactref element="R3" pad="1"/>
-<contactref element="Q9" pad="2"/>
 <contactref element="R7" pad="1"/>
+<contactref element="Q9" pad="3"/>
 <wire x1="-84.77" y1="-546.1" x2="-84.77" y2="-553.72" width="0" layer="19" extent="1-1"/>
-<wire x1="-82.87" y1="-534.5" x2="-84.77" y2="-546.1" width="0" layer="19" extent="1-1"/>
-<wire x1="26.24" y1="-3.515" x2="-82.87" y2="-534.5" width="0" layer="19" extent="1-1"/>
+<wire x1="-83.82" y1="-532.3" x2="-84.77" y2="-546.1" width="0" layer="19" extent="1-1"/>
+<wire x1="26.24" y1="-3.515" x2="-83.82" y2="-532.3" width="0" layer="19" extent="1-1"/>
 <wire x1="26.24" y1="-2.865" x2="26.24" y2="-3.515" width="0" layer="19" extent="1-1"/>
 <wire x1="26.24" y1="-2.215" x2="26.24" y2="-2.865" width="0" layer="19" extent="1-1"/>
@@
 <signal name="N$35">
 <contactref element="Q7" pad="4"/>
+<contactref element="R7" pad="2"/>
 <contactref element="Q9" pad="1"/>
-<contactref element="R7" pad="2"/>
 <wire x1="-84.77" y1="-534.5" x2="-82.87" y2="-553.72" width="0" layer="19" extent="1-1"/>
 <wire x1="-82.845" y1="-524.94" x2="-84.77" y2="-534.5" width="0" layer="19" extent="1-1"/>

Commit message: eagle_librarys
Parts:
- added Q10: (no value), transistors:SOT23
- added R13: (no value), resistor:R0603
Connections:
- new net N$36: Q10.3, Q8.4, R13.1
- net +5V: now also R13.2
- net GND: now also Q10.2
- net IR-LED-POWER: now also Q10.1; no longer Q8.4
Changed lines of the file:
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@@
 <attribute name="VALUE" x="-95.25" y="-572.135" size="1.27" layer="27"/>
+</element>
+<element name="Q10" library="transistors" package="SOT23" value="" x="-93.98" y="-576.58" smashed="yes">
+<attribute name="NAME" x="-95.885" y="-574.675" size="1.27" layer="25"/>
+<attribute name="VALUE" x="-95.885" y="-579.755" size="1.27" layer="27"/>
+</element>
+<element name="R13" library="resistor" library_urn="urn:adsk.eagle:library:348" package="R0603" package3d_urn="urn:adsk.eagle:package:23555/3" value="" x="-93.98" y="-581.66" smashed="yes">
+<attribute name="NAME" x="-94.615" y="-581.025" size="1.27" layer="25"/>
+<attribute name="VALUE" x="-94.615" y="-583.565" size="1.27" layer="27"/>
 </element>
 </elements>
@@
 <contactref element="JP5" pad="3"/>
 <contactref element="JP3" pad="3"/>
+<contactref element="Q10" pad="2"/>
 <wire x1="-60.2488" y1="-185.6994" x2="-66.7512" y2="-185.6994" width="0" layer="19" extent="1-1"/>
 <wire x1="-66.04" y1="-193.83" x2="-66.7512" y2="-185.6994" width="0" layer="19" extent="1-1"/>
@@
 <wire x1="-88.9" y1="-561.34" x2="-93.98" y2="-551.18" width="0" layer="19" extent="1-1"/>
 <wire x1="-88.9" y1="-568.96" x2="-88.9" y2="-561.34" width="0" layer="19" extent="1-1"/>
+<wire x1="-93.03" y1="-577.68" x2="-88.9" y2="-568.96" width="0" layer="19" extent="1-1"/>
 <wire x1="-41.91" y1="-49.53" x2="-63.5" y2="-106.68" width="0" layer="19" extent="1-1"/>
 <wire x1="-39.37" y1="-46.99" x2="-41.91" y2="-49.53" width="0" layer="19" extent="1-1"/>
@@
 <contactref element="JP5" pad="2"/>
 <contactref element="JP3" pad="2"/>
+<contactref element="R13" pad="2"/>
 <wire x1="-67.63" y1="-208.28" x2="-67.63" y2="-180.34" width="0" layer="19" extent="1-1"/>
 <wire x1="-67.63" y1="-236.22" x2="-67.63" y2="-208.28" width="0" layer="19" extent="1-1"/>
@@
 <wire x1="-91.44" y1="-561.34" x2="-90.4875" y2="-551.18" width="0" layer="19" extent="1-1"/>
 <wire x1="-91.44" y1="-568.96" x2="-91.44" y2="-561.34" width="0" layer="19" extent="1-1"/>
+<wire x1="-93.13" y1="-581.66" x2="-91.44" y2="-568.96" width="0" layer="19" extent="1-1"/>
 <wire x1="-66.04" y1="-106.68" x2="-67.63" y2="-180.34" width="0" layer="19" extent="1-1"/>
 <wire x1="-69.43" y1="-76.2" x2="-66.04" y2="-106.68" width="0" layer="19" extent="1-1"/>
@@
 <signal name="IR-LED-POWER">
 <contactref element="U$8" pad="PB2"/>
-<contactref element="Q8" pad="4"/>
-<wire x1="-72.685" y1="-469.06" x2="-35.985" y2="4.445" width="0" layer="19" extent="1-1"/>
+<contactref element="Q10" pad="1"/>
+<wire x1="-35.985" y1="4.445" x2="-94.93" y2="-577.68" width="0" layer="19" extent="1-1"/>
 </signal>
 <signal name="N$26">
@@
 <contactref element="JP5" pad="1"/>
 </signal>
+<signal name="N$36">
+<contactref element="Q8" pad="4"/>
+<contactref element="Q10" pad="3"/>
+<contactref element="R13" pad="1"/>
+<wire x1="-93.98" y1="-575.48" x2="-94.83" y2="-581.66" width="0" layer="19" extent="1-1"/>
+<wire x1="-72.685" y1="-469.06" x2="-93.98" y2="-575.48" width="0" layer="19" extent="1-1"/>
+</signal>
 </signals>
