File: ele/Blackbox/board.sch (EAGLE design)
At the start: 28 parts, among them IC1 DS3231/SO

Commit message: blackbox
-led kruh
-mpu6050
-RTC
Parts:
- removed D1: (no value), diode:DIODE-DO214BA
- removed D2: (no value), diode:DIODE-D-7.5
- removed J1, J2: (no value), Wurth_Elektronik_Electromechanic_Input-Output_Connectors_rev19a:629004113921
- removed Q1, Q2, Q3: (no value), transistors:P-MOSFET-SOT23-GSD
- removed Q6: (no value), transistors:N-MOSFET-SOT23-GSD
- removed R1: 100M, rcl:R-EU_R0603
- removed R4, R5: (no value), rcl:R-EU_R0603
- removed R6: 10M, rcl:R-EU_R0603
- added C2: 2,2nf, rcl:C-EUC0603
- added C3, C4: 0,1uf, rcl:C-EUC0603
- added C5: 10nf, rcl:C-EUC0603
- added NC7, NC8: NC, NC:NC
- added U$10, U$11, U$12, U$13, U$14, U$15, U$16, U$17, U$18, U$19, U$2, U$20, U$21, U$22, U$23, U$24, U$25, U$26, U$27, U$28, U$29, U$3, U$30, U$31, U$32, U$33, U$34, U$35, U$36, U$37, U$38, U$39, U$4, U$40, U$41, U$42, U$43, U$44, U$45, U$46, U$47, U$48, U$49, U$5, U$50, U$51, U$52, U$53, U$54, U$55, U$56, U$57, U$58, U$59, U$6, U$60, U$61, U$7, U$8, U$9: WS2812, WS2812:WS2812
- added U1: MPU-6050, MPU-6050:MPU-6050
- added X1, X2: (no value), con-wago-500:W237-102
- C1: value (none) -> 1nf; device rcl:C-EUC1206 -> rcl:C-EUC0603
Connections:
- removed net !D+: J1.D+, J2.D+, Q1.D
- removed net !D-: J1.D-, J2.D-, Q2.D
- removed net D+: Q1.S
- removed net D-: Q2.S
- removed net ZAKAZ-PROGRAMOVANI: D1.C, Q3.G
- new net !GND: U$10.GND, U$11.GND, U$12.GND, U$13.GND, U$14.GND, U$15.GND, U$16.GND, U$17.GND, U$18.GND, U$19.GND, U$2.GND, U$20.GND, U$21.GND, U$22.GND, U$23.GND, U$24.GND, U$25.GND, U$26.GND, U$27.GND, U$28.GND, U$29.GND, U$3.GND, U$30.GND, U$31.GND, U$32.GND, U$33.GND, U$34.GND, U$35.GND, U$36.GND, U$37.GND, U$38.GND, U$39.GND, U$4.GND, U$40.GND, U$41.GND, U$42.GND, U$43.GND, U$44.GND, U$45.GND, U$46.GND, U$47.GND, U$48.GND, U$49.GND, U$5.GND, U$50.GND, U$51.GND, U$52.GND, U$53.GND, U$54.GND, U$55.GND, U$56.GND, U$57.GND, U$58.GND, U$59.GND, U$6.GND, U$60.GND, U$61.GND, U$7.GND, U$8.GND, U$9.GND
- new net AD0: U1.AD0
- new net AUX_CL: U1.AUX_CL
- new net AUX_DA: U1.AUX_DA
- new net CLKIN: U1.CLKIN
- new net FSYNC: U1.FSYNC
- new net IO11_NC2: IC1.SQW/INT, NC7.NC
- new net IO11_NC3: IC1.32KHZ, NC8.NC
- new net N$10: U$8.DIN, U$9.DOUT
- new net N$11: U$10.DOUT, U$9.DIN
- new net N$12: U$40.DIN, U$41.DOUT
- new net N$13: U$11.DIN, U$12.DOUT
- new net N$14: U$12.DIN, U$13.DOUT
- new net N$15: U$14.DIN, U$15.DOUT
- new net N$16: U$15.DIN, U$16.DOUT
- new net N$17: U$46.DIN, U$47.DOUT
- new net N$18: U$17.DIN, U$18.DOUT
- new net N$19: U$18.DIN, U$19.DOUT
- new net N$20: U$20.DIN, U$21.DOUT
- new net N$21: U$21.DIN, U$22.DOUT
- new net N$22: U$52.DIN, U$53.DOUT
- new net N$23: U$23.DIN, U$24.DOUT
- new net N$24: U$24.DIN, U$25.DOUT
- new net N$25: U$26.DIN, U$27.DOUT
- new net N$26: U$27.DIN, U$28.DOUT
- new net N$27: U$58.DIN, U$59.DOUT
- new net N$28: U$29.DIN, U$30.DOUT
- new net N$29: U$30.DIN, U$31.DOUT
- new net N$30: U$32.DIN, U$33.DOUT
- new net N$31: U$33.DIN, U$34.DOUT
- new net N$32: U$10.DIN, U$11.DOUT
- new net N$33: U$35.DIN, U$36.DOUT
- new net N$34: U$36.DIN, U$37.DOUT
- new net N$35: U$38.DIN, U$39.DOUT
- new net N$36: U$39.DIN, U$40.DOUT
- new net N$37: U$13.DIN, U$14.DOUT
- new net N$38: U$41.DIN, U$42.DOUT
- new net N$39: U$42.DIN, U$43.DOUT
- new net N$40: U$44.DIN, U$45.DOUT
- new net N$41: U$45.DIN, U$46.DOUT
- new net N$42: U$16.DIN, U$17.DOUT
- new net N$43: U$47.DIN, U$48.DOUT
- new net N$44: U$48.DIN, U$49.DOUT
- new net N$45: U$50.DIN, U$51.DOUT
- new net N$46: U$51.DIN, U$52.DOUT
- new net N$47: U$49.DIN, U$50.DOUT
- new net N$48: U$53.DIN, U$54.DOUT
- new net N$49: U$54.DIN, U$55.DOUT
- new net N$5: U$2.DIN, U$3.DOUT
- new net N$50: U$56.DIN, U$57.DOUT
- new net N$51: U$57.DIN, U$58.DOUT
- new net N$52: U$22.DIN, U$23.DOUT
- new net N$53: U$59.DIN, U$60.DOUT
- new net N$54: U$60.DIN, U$61.DOUT
- new net N$55: U$25.DIN, U$26.DOUT
- new net N$56: U$28.DIN, U$29.DOUT
- new net N$57: C4.2
- new net N$58: C5.1, U1.VLOGIC
- new net N$59: U$31.DIN, U$32.DOUT
- new net N$6: U$3.DIN, U$4.DOUT
- new net N$61: U$37.DIN, U$38.DOUT
- new net N$63: U$43.DIN, U$44.DOUT
- new net N$64: U$19.DIN, U$20.DOUT
- new net N$65: U$55.DIN, U$56.DOUT
- new net N$7: U$34.DIN, U$35.DOUT
- new net N$8: U$5.DIN, U$6.DOUT
- new net N$9: U$6.DIN, U$7.DOUT
- new net WS2812: IM6.IO19, U$61.DIN
- net +3V3: now also C3.1, U1.VDD; no longer R4.2, R5.2
- net +5V: now also U$10.VCC, U$11.VCC, U$12.VCC, U$13.VCC, U$14.VCC, U$15.VCC, U$16.VCC, U$17.VCC, U$18.VCC, U$19.VCC, U$2.VCC, U$20.VCC, U$21.VCC, U$22.VCC, U$23.VCC, U$24.VCC, U$25.VCC, U$26.VCC, U$27.VCC, U$28.VCC, U$29.VCC, U$3.VCC, U$30.VCC, U$31.VCC, U$32.VCC, U$33.VCC, U$34.VCC, U$35.VCC, U$36.VCC, U$37.VCC, U$38.VCC, U$39.VCC, U$4.VCC, U$40.VCC, U$41.VCC, U$42.VCC, U$43.VCC, U$44.VCC, U$45.VCC, U$46.VCC, U$47.VCC, U$48.VCC, U$49.VCC, U$5.VCC, U$50.VCC, U$51.VCC, U$52.VCC, U$53.VCC, U$54.VCC, U$55.VCC, U$56.VCC, U$57.VCC, U$58.VCC, U$59.VCC, U$6.VCC, U$60.VCC, U$61.VCC, U$7.VCC, U$8.VCC, U$9.VCC, X1-1.KL, X2-1.KL; no longer D2.A, J1.VBUS, J2.VBUS, R6.2
- net +5V_ESP: no longer D2.C
- net 3,3!KNOFLIK: no longer Q3.D
- net GND: now also C2.2, C3.2, U1.GND, X1-2.KL, X2-2.KL; no longer J1.GND, J2.GND, Q6.S, R1.1
- net INT: now also U1.INT
- net N$1: now also C2.1, U1.CPOUT; no longer IC1.SQW/INT, R5.1
- net N$2: now also U$4.DIN, U$5.DOUT; no longer D1.A, Q3.S, Q6.G, R1.2
- net N$3: now also C4.1, C5.2, U1.REGOUT; no longer IC1.32KHZ, R4.1
- net N$4: now also U$7.DIN, U$8.DOUT; no longer Q1.G, Q2.G, Q6.D, R6.1
- net SCL: now also U1.SCL
- net SDA: now also U1.SDA

Commit message: blackbox-sch
Parts:
- removed JP1: (no value), pinhead:PINHD-1X8
- added R1, R4, R5: (no value), rcl:R-EU_R0603
- added U$62: EC11-1S, EC11-1S:EC11-1S
Connections:
- new net ENC-A: IM6.IO18, R4.1, U$62.A
- new net ENC-B: IM6.IO17, R5.1, U$62.B
- new net SW0: IM6.IO5, R1.1, U$62.SW-A
- net +3V3: now also R1.2, R4.2, R5.2; no longer JP1.1
- net ADO: no longer JP1.7
- net GND: now also U$62.IN, U$62.SW-B; no longer JP1.2
- net INT: no longer JP1.8
- net RX-GPS: now also IM6.IO16
- net SCL: no longer JP1.3
- net SDA: no longer JP1.4
- net TX-GPS: now also IM6.IO4
- net XCL: no longer JP1.6
- net XDA: no longer JP1.5
Other:
- moved on the sheet: JP2, JP4

Commit message: max485
-max485
-nejake datashity pouzitych soucastek
Parts:
- added C10, C11, C12, C13, C14, C15, C16, C17, C18, C19, C20, C21, C22, C23, C24, C25, C26, C27, C28, C29, C30, C31, C32, C33, C34, C35, C36, C37, C38, C39, C40, C41, C42, C43, C44, C45, C46, C47, C48, C49, C50, C51, C52, C53, C54, C55, C56, C57, C58, C59, C60, C61, C62, C63, C64, C65, C66, C67, C68, C9: (no value), rcl:C-EUC0402K
- added C6: 0.22uf, rcl:C-EUC0402K
- added C69, C70: 10uf, rcl:C-EUC0402K
- added C7: 4.7uf, rcl:C-EUC0402K
- added C8: 0.1uf, rcl:C-EUC0402K
- added IC2: QMC5883L-TR, QMC5883L-TR:QMC5883L-TR
- added JP1: (no value), pinhead:PINHD-1X4
- added MOTOR: (no value), con-wago-500:W237-102
- added NC10, NC11, NC12, NC9: NC, NC:NC
- added Q1, Q6: (no value), transistors:N-MOSFET-SOT23-GSD
- added Q3: (no value), transistors:N-MOSFET-SO8
- added Q5: (no value), transistors:P-MOSFET-MLP
- added R10, R12: 220, rcl:R-EU_R0402
- added R11: 100k, rcl:R-EU_R0402
- added R13, R14: 20k, rcl:R-EU_R0402
- added R16, R17, R18, R8, R9: 10k, rcl:R-EU_R0402
- added R6: 1M, rcl:R-EU_R0402
- added R7: 220, rcl:R-EU_R0603
- added U2: MAX485ESA+, MAX485ESA_:MAX485ESA+
- C1, C2, C3, C4, C5: device rcl:C-EUC0603 -> rcl:C-EUC0402K
- R1, R4, R5: value (none) -> 10k; device rcl:R-EU_R0603 -> rcl:R-EU_R0402
Connections:
- removed net !GND: U$10.GND, U$11.GND, U$12.GND, U$13.GND, U$14.GND, U$15.GND, U$16.GND, U$17.GND, U$18.GND, U$19.GND, U$2.GND, U$20.GND, U$21.GND, U$22.GND, U$23.GND, U$24.GND, U$25.GND, U$26.GND, U$27.GND, U$28.GND, U$29.GND, U$3.GND, U$30.GND, U$31.GND, U$32.GND, U$33.GND, U$34.GND, U$35.GND, U$36.GND, U$37.GND, U$38.GND, U$39.GND, U$4.GND, U$40.GND, U$41.GND, U$42.GND, U$43.GND, U$44.GND, U$45.GND, U$46.GND, U$47.GND, U$48.GND, U$49.GND, U$5.GND, U$50.GND, U$51.GND, U$52.GND, U$53.GND, U$54.GND, U$55.GND, U$56.GND, U$57.GND, U$58.GND, U$59.GND, U$6.GND, U$60.GND, U$61.GND, U$7.GND, U$8.GND, U$9.GND
- new net IO10_NC2: IC2.NC-2, NC9.NC
- new net IO10_NC3: IC2.NC-5, NC12.NC
- new net IO9_NC2: IC2.NC-1, NC7.NC
- new net IO9_NC3: IC2.NC-4, NC11.NC
- new net LED-SHUTDOWN: IM6.IO2, R7.2
- new net MODE-485: IM6.IO0, R16.1, U2.!RE, U2.DE
- new net MOTOR: IM6.IO12, R10.2
- new net N$60: C6.1, IC2.SETC
- new net N$62: C6.2, IC2.STEP
- new net N$66: C7.1, IC2.C1
- new net N$68: Q5.G, Q6.D, R6.2
- new net N$69: Q6.G, R7.1
- new net N$70: MOTOR-2.KL, Q3.D
- new net N$71: Q3.G, R10.1, R11.2
- new net N$72: JP1.2, R12.1, R14.1, U2.B
- new net N$73: JP1.3, R12.2, R13.1, U2.A
- new net N$74: Q3.S
- new net QMC5883-INTERRUPT: IC2.DRDY, IM6.IO13
- new net RX-485: R18.1, U2.RO
- new net SQW/INT: IC1.SQW/INT, IM6.IO15
- new net TX-485: R17.1, U2.DI
- new net VCC: C10.1, C11.1, C12.1, C13.1, C14.1, C15.1, C16.1, C17.1, C18.1, C19.1, C20.1, C21.1, C22.1, C23.1, C24.1, C25.1, C26.1, C27.1, C28.1, C29.1, C30.1, C31.1, C32.1, C33.1, C34.1, C35.1, C36.1, C37.1, C38.1, C39.1, C40.1, C41.1, C42.1, C43.1, C44.1, C45.1, C46.1, C47.1, C48.1, C49.1, C50.1, C51.1, C52.1, C53.1, C54.1, C55.1, C56.1, C57.1, C58.1, C59.1, C60.1, C61.1, C62.1, C63.1, C64.1, C65.1, C66.1, C67.1, C68.1, C9.1, Q5.D, U$10.VCC, U$11.VCC, U$12.VCC, U$13.VCC, U$14.VCC, U$15.VCC, U$16.VCC, U$17.VCC, U$18.VCC, U$19.VCC, U$2.VCC, U$20.VCC, U$21.VCC, U$22.VCC, U$23.VCC, U$24.VCC, U$25.VCC, U$26.VCC, U$27.VCC, U$28.VCC, U$29.VCC, U$3.VCC, U$30.VCC, U$31.VCC, U$32.VCC, U$33.VCC, U$34.VCC, U$35.VCC, U$36.VCC, U$37.VCC, U$38.VCC, U$39.VCC, U$4.VCC, U$40.VCC, U$41.VCC, U$42.VCC, U$43.VCC, U$44.VCC, U$45.VCC, U$46.VCC, U$47.VCC, U$48.VCC, U$49.VCC, U$5.VCC, U$50.VCC, U$51.VCC, U$52.VCC, U$53.VCC, U$54.VCC, U$55.VCC, U$56.VCC, U$57.VCC, U$58.VCC, U$59.VCC, U$6.VCC, U$60.VCC, U$61.VCC, U$7.VCC, U$8.VCC, U$9.VCC
- new net WS2812-5V: Q1.D, R9.2, U$61.DIN
- net +3V3: now also C8.1, IC2.S1, IC2.VDD, IC2.VDDIO, Q1.G, R8.1
- net +5V: now also C69.1, C70.1, JP1.4, MOTOR-1.KL, Q5.S, R13.2, R16.2, R17.2, R18.2, R6.1, R9.1, U2.VCC; no longer U$10.VCC, U$11.VCC, U$12.VCC, U$13.VCC, U$14.VCC, U$15.VCC, U$16.VCC, U$17.VCC, U$18.VCC, U$19.VCC, U$2.VCC, U$20.VCC, U$21.VCC, U$22.VCC, U$23.VCC, U$24.VCC, U$25.VCC, U$26.VCC, U$27.VCC, U$28.VCC, U$29.VCC, U$3.VCC, U$30.VCC, U$31.VCC, U$32.VCC, U$33.VCC, U$34.VCC, U$35.VCC, U$36.VCC, U$37.VCC, U$38.VCC, U$39.VCC, U$4.VCC, U$40.VCC, U$41.VCC, U$42.VCC, U$43.VCC, U$44.VCC, U$45.VCC, U$46.VCC, U$47.VCC, U$48.VCC, U$49.VCC, U$5.VCC, U$50.VCC, U$51.VCC, U$52.VCC, U$53.VCC, U$54.VCC, U$55.VCC, U$56.VCC, U$57.VCC, U$58.VCC, U$59.VCC, U$6.VCC, U$60.VCC, U$61.VCC, U$7.VCC, U$8.VCC, U$9.VCC
- net GND: now also C10.2, C11.2, C12.2, C13.2, C14.2, C15.2, C16.2, C17.2, C18.2, C19.2, C20.2, C21.2, C22.2, C23.2, C24.2, C25.2, C26.2, C27.2, C28.2, C29.2, C30.2, C31.2, C32.2, C33.2, C34.2, C35.2, C36.2, C37.2, C38.2, C39.2, C40.2, C41.2, C42.2, C43.2, C44.2, C45.2, C46.2, C47.2, C48.2, C49.2, C5.2, C50.2, C51.2, C52.2, C53.2, C54.2, C55.2, C56.2, C57.2, C58.2, C59.2, C60.2, C61.2, C62.2, C63.2, C64.2, C65.2, C66.2, C67.2, C68.2, C69.2, C7.2, C70.2, C8.2, C9.2, IC2.GND, JP1.1, Q6.S, R11.1, R14.2, U$10.GND, U$11.GND, U$12.GND, U$13.GND, U$14.GND, U$15.GND, U$16.GND, U$17.GND, U$18.GND, U$19.GND, U$2.GND, U$20.GND, U$21.GND, U$22.GND, U$23.GND, U$24.GND, U$25.GND, U$26.GND, U$27.GND, U$28.GND, U$29.GND, U$3.GND, U$30.GND, U$31.GND, U$32.GND, U$33.GND, U$34.GND, U$35.GND, U$36.GND, U$37.GND, U$38.GND, U$39.GND, U$4.GND, U$40.GND, U$41.GND, U$42.GND, U$43.GND, U$44.GND, U$45.GND, U$46.GND, U$47.GND, U$48.GND, U$49.GND, U$5.GND, U$50.GND, U$51.GND, U$52.GND, U$53.GND, U$54.GND, U$55.GND, U$56.GND, U$57.GND, U$58.GND, U$59.GND, U$6.GND, U$60.GND, U$61.GND, U$7.GND, U$8.GND, U$9.GND, U2.GND
- net IO11_NC2: now also IC2.NC-3, NC10.NC; no longer IC1.SQW/INT, NC7.NC
- net N$3: no longer C5.2
- net SCL: now also IC2.SCL
- net SDA: now also IC2.SDA
- net WS2812: now also Q1.S, R8.2; no longer U$61.DIN
