File: ele/Blackbox/mein_board/board.brd (EAGLE design)
At the start: 111.7 x 112.7 mm, 166 parts, among them IC1 DS3231/SO, IC2 QMC5883L-TR, U1 MPU-6050, U2 MAX485ESA+

Commit message: prvni_konzultace_s_kubou
Parts:
- removed JP6: (no value), pinhead:2X10
- removed U2: MAX485ESA+, MAX485ESA_:SOIC127P600X175-8N
- added D1: (no value), diode:DO214BA
- added JP7: (no value), pinhead:1X03
- added JP8: (no value), pinhead:1X01
- added LED4: powerled, led:SML0603
- added MAX1: MAX485, maxim:SO08
- added Q10, Q4, Q5: (no value), transistors:SOT23
- added Q8, Q9: BSO201SP, transistor-fet:SO-8
- added R15: 300k, rcl:R0603
- added R19, R22: 100k, rcl:R0402
- added R20: 47k, rcl:R0603
- added R21: 100k, rcl:R0603
- added R23, R24: 10k, rcl:R0402
- added R25: 1k, resistor:R0402
- added SJ1: (no value), jumper:SJ
- C2: value 2,2nf -> 2.2nf
- C3, C4: value 0,1uf -> 100nf
- C6: value 0.22uf -> 220nf
- C7: device rcl:C0402K -> rcl:C0603
- C8: value 0.1uf -> 100nf
- JP2: device pinhead:1X08 -> pinhead:2X06
- Q2: value (none) -> BSO201SP; device transistor-power:SO-08 -> transistor-fet:SO-8
- R12: value 220 -> 120
- R17: value 10k -> 100k
- R2, R3: value (none) -> 47k; device rcl:R0603 -> rcl:R0402
- R6: value 1M -> 300k
- R7: device rcl:R0603 -> rcl:R0402
- moved R12 79.1 mm to (-18.4, -34.0)
- moved C69 76.2 mm to (-17.8, -29.2), turned to 90 degrees
- moved JP1 75.1 mm to (-17.1, -36.8), turned to 0 degrees
- moved R14 71.0 mm to (-26.0, -26.7)
- moved C70 70.0 mm to (-16.5, -29.2), turned to 90 degrees
- moved R13 69.8 mm to (-16.5, -34.0), turned to 90 degrees
- moved R18 66.7 mm to (-14.0, -26.7), turned to 270 degrees
- moved R17 61.4 mm to (-17.1, -24.1), turned to 0 degrees
- moved JP4 59.5 mm to (-24.1, 16.5), turned to 0 degrees
- moved JP3 50.0 mm to (-24.1, 10.2), turned to 180 degrees
- moved IM1 48.3 mm to (24.1, -22.9), flipped to the bottom
- moved R8 40.1 mm to (30.5, -1.27), turned to 180 degrees
- moved X1 33.6 mm to (31.8, -31.8), turned to 135 degrees
- moved U$1 33.0 mm to (-29.2, 27.9), turned to 135 degrees
- moved JP2 31.6 mm to (41.3, 3.17), turned to 270 degrees
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Connections:
- removed net ADO: JP2.7
- removed net INT: JP2.8, U1.12
- removed net IO11_NC3: IC1.1
- removed net IO12: IM1.12, JP6.19
- removed net IO25: IM1.9, JP6.13
- removed net IO26: IM1.10, JP6.15
- removed net IO27: IM1.11, JP6.17
- removed net MODE-485: IM1.25, R16.1, U2.2, U2.3
- removed net N$58: C5.1, U1.8
- removed net N$72: JP1.2, R12.1, R14.1, U2.7
- removed net N$73: JP1.3, R12.2, R13.1, U2.6
- removed net RX-485: R18.1, U2.1
- removed net TX-485: R17.1, U2.4
- removed net XCL: JP2.6
- removed net XDA: JP2.5
- new net A: JP1.2, MAX1.6, R12.2, R14.1
- new net B: JP1.3, MAX1.7, R13.1, SJ1.2
- new net ESP_SHUTDOWN: IM1.33, Q5.1, R19.1
- new net INT_MPU5060: IM1.9, U1.12
- new net LED4: LED4.C, R25.1
- new net MODE_485: IM1.24, MAX1.2, MAX1.3, R17.1
- new net N$10: IM1.2, JP8.1
- new net N$4: Q8.5, Q8.6, Q8.7, Q8.8, X1.1, X2.1
- new net N$5: Q8.1, Q8.2, Q8.3, Q9.1, Q9.2, Q9.3, R15.2
- new net N$6: Q5.3, Q9.4, R15.1
- new net N$7: IC1.1, R21.1
- new net N$8: R12.1, SJ1.1
- new net N$9: JP7.3, U$2.DOUT
- new net RX-485-5V: MAX1.1, Q10.3, R18.1
- new net RX_485: IM1.11, Q10.2, R16.1
- new net TX_485: IM1.10, Q4.2, R23.2
- new net TX_485-5V: MAX1.4, Q4.3, R24.2
- net +3V3: now also C1.1, C5.1, Q10.1, Q4.1, R16.2, R19.2, R20.2, R21.2, R23.1, U1.8; no longer JP2.1
- net +5V: now also D1.C, LED4.A, MAX1.8, Q9.5, Q9.6, Q9.7, Q9.8, R24.1; no longer R16.2, R17.2, U2.8, X1.1, X2.1
- net DS3231/RST: now also IM1.23; no longer C1.1, IM1.33
- net GND: now also JP2.1, JP2.11, JP2.3, JP2.5, JP2.7, JP2.9, JP7.1, MAX1.5, Q5.2, Q8.4, R17.2, R22.1, R25.2; no longer JP2.2, JP6.10, JP6.12, JP6.14, JP6.16, JP6.18, JP6.2, JP6.20, JP6.4, JP6.6, JP6.8, U2.5
- net IO32: now also JP2.10; no longer JP6.9
- net IO33: now also JP2.12; no longer JP6.11
- net IO34: now also JP2.6; no longer JP6.5
- net IO35: now also JP2.8; no longer JP6.7
- net LED-SHUTDOWN: now also IM1.13; no longer IM1.24
- net MOTOR: now also IM1.15; no longer IM1.13
- net N$2: now also D1.A
- net N$69: now also R22.2
- net QMC5883-INTERRUPT: now also IM1.31; no longer IM1.15
- net RX-GPS: now also IM1.26; no longer IM1.27
- net SCL: no longer JP2.3
- net SDA: no longer JP2.4
- net SQW/INT: now also IM1.25, R20.1; no longer IM1.23
- net SVN: now also JP2.4; no longer JP6.3
- net SVP: now also JP2.2; no longer JP6.1
- net TX-GPS: now also IM1.27; no longer IM1.26
- net VCC: now also JP7.2
- net WS2812: now also IM1.12; no longer IM1.31
Routing:
- net +3V3: track 135.9 -> 208.9 mm, vias 0 -> 5
- net RX-485-5V: track 0.00 -> 62.0 mm
- net TX_485-5V: track 0.00 -> 59.4 mm
- net DS3231/RST: track 11.7 -> 65.5 mm, vias 0 -> 1
- net N$4: track 0.00 -> 53.5 mm
- net ESP_SHUTDOWN: track 0.00 -> 51.4 mm, vias 0 -> 2
- net INT_MPU5060: track 0.00 -> 49.4 mm, vias 0 -> 2
- net +5V: track 160.9 -> 112.3 mm, vias 0 -> 3
- net MODE_485: track 0.00 -> 47.2 mm
- net RX-GPS: track 0.00 -> 46.6 mm
- net LED-SHUTDOWN: track 15.6 -> 61.4 mm
- net TX-GPS: track 0.00 -> 44.1 mm
- net SDA: track 51.1 -> 93.2 mm, vias 0 -> 2
- net QMC5883-INTERRUPT: track 0.00 -> 40.8 mm, vias 0 -> 1
- net SCL: track 51.6 -> 90.4 mm
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- added copper zone on layer 1, net +3V3
- added copper zone on layer 16, net GND
- added copper zone on layer 1, net N$4
- added copper zone on layer 1, net N$5
