File: ele/Blackbox/mein_board/board.sch (EAGLE design)
At the start: 177 parts, among them IC1 DS3231/SO, IC2 QMC5883L-TR, U1 MPU-6050, U2 MAX485ESA+

Commit message: eagle_librarys
Parts:
- removed Q5: (no value), transistors:P-MOSFET-MLP
- added JP6: (no value), pinhead:PINHD-2X10
- added Q2: (no value), transistor-power:P-MOSFET-SO8
- renumbered IM6 to IM1
Connections:
- net N$10 renamed WS2812-6
- net N$11 renamed WS2812-7
- net N$12 renamed WS2812-38
- net N$13 renamed WS2812-9
- net N$14 renamed WS2812-10
- net N$15 renamed WS2812-12
- net N$16 renamed WS2812-13
- net N$17 renamed WS2812-44
- net N$18 renamed WS2812-15
- net N$19 renamed WS2812-16
- net N$2 renamed WS2812-2
- net N$20 renamed WS2812-18
- net N$21 renamed WS2812-19
- net N$22 renamed WS2812-50
- net N$23 renamed WS2812-21
- net N$24 renamed WS2812-22
- net N$25 renamed WS2812-24
- net N$26 renamed WS2812-25
- net N$27 renamed WS2812-56
- net N$28 renamed WS2812-27
- net N$29 renamed WS2812-28
- net N$30 renamed WS2812-30
- net N$31 renamed WS2812-31
- net N$32 renamed WS2812-8
- net N$33 renamed WS2812-33
- net N$34 renamed WS2812-34
- net N$35 renamed WS2812-36
- net N$36 renamed WS2812-37
- net N$37 renamed WS2812-11
- net N$38 renamed WS2812-39
- net N$39 renamed WS2812-40
- net N$4 renamed WS2812-5
- net N$40 renamed WS2812-42
- net N$41 renamed WS2812-43
- net N$42 renamed WS2812-14
- net N$43 renamed WS2812-45
- net N$44 renamed WS2812-46
- net N$45 renamed WS2812-48
- net N$46 renamed WS2812-49
- net N$48 renamed WS2812-51
- net N$49 renamed WS2812-52
- net N$5 renamed WS2812-0
- net N$50 renamed WS2812-54
- net N$51 renamed WS2812-55
- net N$52 renamed WS2812-20
- net N$53 renamed WS2812-57
- net N$54 renamed WS2812-58
- net N$55 renamed WS2812-23
- net N$56 renamed WS2812-26
- net N$59 renamed WS2812-29
- net N$6 renamed WS2812-1
- net N$61 renamed WS2812-35
- net N$63 renamed WS2812-41
- net N$64 renamed WS2812-17
- net N$65 renamed WS2812-53
- net N$7 renamed WS2812-32
- net N$8 renamed WS2812-3
- net N$9 renamed WS2812-4
- removed net +5V_ESP: IM1.5V
- removed net N$57: C4.2
- removed net N$70: MOTOR-2.KL, Q3.D
- removed net N$74: Q3.S
- new net IO12: IM1.IO14, JP6.19
- new net IO25: IM1.IO25, JP6.13
- new net IO26: IM1.IO26, JP6.15
- new net IO27: IM1.IO27, JP6.17
- new net IO32: IM1.IO32, JP6.9
- new net IO33: IM1.IO33, JP6.11
- new net IO34: IM1.IO34, JP6.5
- new net IO35: IM1.IO35, JP6.7
- new net N$2: MOTOR-1.KL, Q3.D
- new net SVN: IM1.SVN, JP6.3
- new net SVP: IM1.SVP, JP6.1
- net +5V: now also IM1.5V, MOTOR-2.KL, Q2.S; no longer MOTOR-1.KL, Q5.S
- net GND: now also C4.2, JP6.10, JP6.12, JP6.14, JP6.16, JP6.18, JP6.2, JP6.20, JP6.4, JP6.6, JP6.8, Q3.S
- net N$68: now also Q2.G; no longer Q5.G
- net VCC: now also Q2.D; no longer Q5.D
Other:
- moved on the sheet: MOTOR-1, MOTOR-2

Commit message: prvni_konzultace_s_kubou
Parts:
- removed JP6: (no value), pinhead:PINHD-2X10
- removed NC8: NC, NC:NC
- removed U2: MAX485ESA+, MAX485ESA_:MAX485ESA+
- added D1: (no value), diode:DIODE-DO214BA
- added JP7: (no value), pinhead:PINHD-1X3
- added JP8: (no value), pinhead:PINHD-1X1
- added LED4: powerled, led:LEDSML0603
- added MAX1: MAX485, maxim:MAX485
- added Q10, Q4, Q5: (no value), transistors:N-MOSFET-SOT23-GSD
- added Q8, Q9: BSO201SP, transistor-fet:BSO201SP
- added R15: 300k, rcl:R-EU_R0603
- added R19, R22: 100k, rcl:R-EU_R0402
- added R20: 47k, rcl:R-EU_R0603
- added R21: 100k, rcl:R-EU_R0603
- added R23, R24: 10k, rcl:R-EU_R0402
- added R25: 1k, resistor:R-EU_R0402
- added SJ1: (no value), jumper:SJ
- C2: value 2,2nf -> 2.2nf
- C3, C4: value 0,1uf -> 100nf
- C6: value 0.22uf -> 220nf
- C7: device rcl:C-EUC0402K -> rcl:C-EUC0603
- C8: value 0.1uf -> 100nf
- JP2: device pinhead:PINHD-1X8 -> pinhead:PINHD-2X6
- Q2: value (none) -> BSO201SP; device transistor-power:P-MOSFET-SO8 -> transistor-fet:BSO201SP
- R12: value 220 -> 120
- R17: value 10k -> 100k
- R2, R3: value (none) -> 47k; device rcl:R-EU_R0603 -> rcl:R-EU_R0402
- R6: value 1M -> 300k
- R7: device rcl:R-EU_R0603 -> rcl:R-EU_R0402
Connections:
- removed net ADO: JP2.7
- removed net INT: JP2.8, U1.INT
- removed net IO11_NC3: IC1.32KHZ, NC8.NC
- removed net IO12: IM1.IO14, JP6.19
- removed net IO25: IM1.IO25, JP6.13
- removed net IO26: IM1.IO26, JP6.15
- removed net IO27: IM1.IO27, JP6.17
- removed net MODE-485: IM1.IO0, R16.1, U2.!RE, U2.DE
- removed net N$58: C5.1, U1.VLOGIC
- removed net N$72: JP1.2, R12.1, R14.1, U2.B
- removed net N$73: JP1.3, R12.2, R13.1, U2.A
- removed net RX-485: R18.1, U2.RO
- removed net TX-485: R17.1, U2.DI
- removed net XCL: JP2.6
- removed net XDA: JP2.5
- new net A: JP1.2, MAX1.A, R12.2, R14.1
- new net B: JP1.3, MAX1.B, R13.1, SJ1.2
- new net ESP_SHUTDOWN: IM1.IO21, Q5.G, R19.1
- new net INT_MPU5060: IM1.IO25, U1.INT
- new net LED4: LED4.C, R25.1
- new net MODE_485: IM1.IO2, MAX1.DE, MAX1.RE/, R17.1
- new net N$10: IM1.EN, JP8.1
- new net N$4: Q8.D, X1-1.KL, X2-1.KL
- new net N$5: Q8.S, Q9.S, R15.2
- new net N$6: Q5.D, Q9.G, R15.1
- new net N$7: IC1.32KHZ, R21.1
- new net N$8: R12.1, SJ1.1
- new net N$9: JP7.3, U$2.DOUT
- new net RX-485-5V: MAX1.RO, Q10.D, R18.1
- new net RX_485: IM1.IO27, Q10.S, R16.1
- new net TX_485: IM1.IO26, Q4.S, R23.2
- new net TX_485-5V: MAX1.DI, Q4.D, R24.2
- net +3V3: now also C1.1, C5.1, Q10.G, Q4.G, R16.2, R19.2, R20.2, R21.2, R23.1, U1.VLOGIC; no longer JP2.1
- net +5V: now also D1.C, LED4.A, MAX1.VCC, Q9.D, R24.1; no longer R16.2, R17.2, U2.VCC, X1-1.KL, X2-1.KL
- net DS3231/RST: now also IM1.IO15; no longer C1.1, IM1.IO21
- net GND: now also JP2.1, JP2.11, JP2.3, JP2.5, JP2.7, JP2.9, JP7.1, MAX1.GND, Q5.S, Q8.G, R17.2, R22.1, R25.2; no longer JP2.2, JP6.10, JP6.12, JP6.14, JP6.16, JP6.18, JP6.2, JP6.20, JP6.4, JP6.6, JP6.8, U2.GND
- net IO32: now also JP2.10; no longer JP6.9
- net IO33: now also JP2.12; no longer JP6.11
- net IO34: now also JP2.6; no longer JP6.5
- net IO35: now also JP2.8; no longer JP6.7
- net LED-SHUTDOWN: now also IM1.IO12; no longer IM1.IO2
- net MOTOR: now also IM1.IO13; no longer IM1.IO12
- net N$2: now also D1.A
- net N$69: now also R22.2
- net QMC5883-INTERRUPT: now also IM1.IO19; no longer IM1.IO13
- net RX-GPS: now also IM1.IO4; no longer IM1.IO16
- net SCL: no longer JP2.3
- net SDA: no longer JP2.4
- net SQW/INT: now also IM1.IO0, R20.1; no longer IM1.IO15
- net SVN: now also JP2.4; no longer JP6.3
- net SVP: now also JP2.2; no longer JP6.1
- net TX-GPS: now also IM1.IO16; no longer IM1.IO4
- net VCC: now also JP7.2
- net WS2812: now also IM1.IO14; no longer IM1.IO19
Other:
- moved on the sheet: C1, C3, C5, C6, C69, C7, C70, C8, IC1, JP1, JP4, MOTOR-1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
