File: ele/Blackbox/main_board/board.sch (EAGLE design)
At the start: 194 parts, among them IC1 DS3231/SO, IC2 QMC5883L-TR, Q2 BSO201SP, Q8 BSO201SP, Q9 BSO201SP, U1 MPU-6050

Commit message: 2.KSK
Parts:
- removed Q4: (no value), transistors:N-MOSFET-SOT23-GSD
- removed R21: 100k, rcl:R-EU_R0603
- removed R23, R24: 10k, rcl:R-EU_R0402
- added C71: 4.7uf, rcl:C-EUC0603
- added NC13, NC14, NC8: NC, NC:NC
- R18: value 10k -> 2M; device rcl:R-EU_R0402 -> rcl:R-EU_R0603
Connections:
- removed net N$7: IC1.32KHZ, R21.1
- removed net TX_485-5V: MAX1.DI, Q4.D, R24.2
- new net IO10_NC4: NC13.NC, U1.RESV
- new net IO9_NC4: NC8.NC, U1.RESV@1
- new net IO9_NC5: NC14.NC, U1.RESV@2
- net +3V3: no longer Q4.G, R21.2, R23.1
- net +5V: no longer R18.2, R24.1
- net ESP_SHUTDOWN: now also IM1.IO0; no longer IM1.IO21
- net N$6: now also C71.1, R18.1
- net RX-485-5V: no longer R18.1
- net SQW/INT: now also IM1.IO21; no longer IM1.IO0
- net SW0: now also C71.2, R18.2
- net TX_485: now also MAX1.DI; no longer Q4.S, R23.2
Other:
- moved on the sheet: C2, C3, C4, C5, C6, C7, C8, JP2, LED4, Q10, Q5, Q8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

Commit message: dovetek_2.KSK
Connections:
- net MODE_485: now also IM1.IO13; no longer IM1.IO2
- net MOTOR: now also IM1.IO2; no longer IM1.IO13
Changed lines of the file:
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@@
 <grid distance="0.1" unitdist="inch" unit="inch" style="lines" multiple="1" display="no" altdistance="0.01" altunitdist="inch" altunit="inch"/>
 <layers>
-<layer number="1" name="Top" color="4" fill="1" visible="yes" active="no"/>
-<layer number="2" name="Route2" color="16" fill="1" visible="yes" active="no"/>
-<layer number="3" name="Route3" color="17" fill="1" visible="yes" active="no"/>
-<layer number="4" name="Route4" color="18" fill="1" visible="yes" active="no"/>
-<layer number="5" name="Route5" color="19" fill="1" visible="yes" active="no"/>
-<layer number="6" name="Route6" color="25" fill="1" visible="yes" active="no"/>
-<layer number="7" name="Route7" color="26" fill="1" visible="yes" active="no"/>
-<layer number="8" name="Route8" color="27" fill="1" visible="yes" active="no"/>
-<layer number="9" name="Route9" color="28" fill="1" visible="yes" active="no"/>
-<layer number="10" name="Route10" color="29" fill="1" visible="yes" active="no"/>
-<layer number="11" name="Route11" color="30" fill="1" visible="yes" active="no"/>
-<layer number="12" name="Route12" color="20" fill="1" visible="yes" active="no"/>
-<layer number="13" name="Route13" color="21" fill="1" visible="yes" active="no"/>
-<layer number="14" name="Route14" color="22" fill="1" visible="yes" active="no"/>
-<layer number="15" name="Route15" color="23" fill="1" visible="yes" active="no"/>
-<layer number="16" name="Bottom" color="1" fill="1" visible="yes" active="no"/>
-<layer number="17" name="Pads" color="2" fill="1" visible="yes" active="no"/>
-<layer number="18" name="Vias" color="2" fill="1" visible="yes" active="no"/>
-<layer number="19" name="Unrouted" color="6" fill="1" visible="yes" active="no"/>
-<layer number="20" name="Dimension" color="24" fill="1" visible="yes" active="no"/>
-<layer number="21" name="tPlace" color="7" fill="1" visible="yes" active="no"/>
-<layer number="22" name="bPlace" color="7" fill="1" visible="yes" active="no"/>
-<layer number="23" name="tOrigins" color="15" fill="1" visible="yes" active="no"/>
-<layer number="24" name="bOrigins" color="15" fill="1" visible="yes" active="no"/>
-<layer number="25" name="tNames" color="7" fill="1" visible="yes" active="no"/>
-<layer number="26" name="bNames" color="7" fill="1" visible="yes" active="no"/>
-<layer number="27" name="tValues" color="7" fill="1" visible="yes" active="no"/>
-<layer number="28" name="bValues" color="7" fill="1" visible="yes" active="no"/>
+<layer number="1" name="Top" color="4" fill="1" visible="no" active="no"/>
+<layer number="2" name="Route2" color="16" fill="1" visible="no" active="no"/>
+<layer number="3" name="Route3" color="17" fill="1" visible="no" active="no"/>
+<layer number="4" name="Route4" color="18" fill="1" visible="no" active="no"/>
+<layer number="5" name="Route5" color="19" fill="1" visible="no" active="no"/>
+<layer number="6" name="Route6" color="25" fill="1" visible="no" active="no"/>
+<layer number="7" name="Route7" color="26" fill="1" visible="no" active="no"/>
+<layer number="8" name="Route8" color="27" fill="1" visible="no" active="no"/>
+<layer number="9" name="Route9" color="28" fill="1" visible="no" active="no"/>
+<layer number="10" name="Route10" color="29" fill="1" visible="no" active="no"/>
+<layer number="11" name="Route11" color="30" fill="1" visible="no" active="no"/>
+<layer number="12" name="Route12" color="20" fill="1" visible="no" active="no"/>
+<layer number="13" name="Route13" color="21" fill="1" visible="no" active="no"/>
+<layer number="14" name="Route14" color="22" fill="1" visible="no" active="no"/>
+<layer number="15" name="Route15" color="23" fill="1" visible="no" active="no"/>
+<layer number="16" name="Bottom" color="1" fill="1" visible="no" active="no"/>
+<layer number="17" name="Pads" color="2" fill="1" visible="no" active="no"/>
+<layer number="18" name="Vias" color="2" fill="1" visible="no" active="no"/>
+<layer number="19" name="Unrouted" color="6" fill="1" visible="no" active="no"/>
+<layer number="20" name="Dimension" color="24" fill="1" visible="no" active="no"/>
+<layer number="21" name="tPlace" color="7" fill="1" visible="no" active="no"/>
+<layer number="22" name="bPlace" color="7" fill="1" visible="no" active="no"/>
+<layer number="23" name="tOrigins" color="15" fill="1" visible="no" active="no"/>
+<layer number="24" name="bOrigins" color="15" fill="1" visible="no" active="no"/>
+<layer number="25" name="tNames" color="7" fill="1" visible="no" active="no"/>
+<layer number="26" name="bNames" color="7" fill="1" visible="no" active="no"/>
+<layer number="27" name="tValues" color="7" fill="1" visible="no" active="no"/>
+<layer number="28" name="bValues" color="7" fill="1" visible="no" active="no"/>
 <layer number="29" name="tStop" color="7" fill="3" visible="no" active="no"/>
 <layer number="30" name="bStop" color="7" fill="6" visible="no" active="no"/>
@@
 <layer number="35" name="tGlue" color="7" fill="4" visible="no" active="no"/>
 <layer number="36" name="bGlue" color="7" fill="5" visible="no" active="no"/>
-<layer number="37" name="tTest" color="7" fill="1" visible="yes" active="no"/>
-<layer number="38" name="bTest" color="7" fill="1" visible="yes" active="no"/>
+<layer number="37" name="tTest" color="7" fill="1" visible="no" active="no"/>
+<layer number="38" name="bTest" color="7" fill="1" visible="no" active="no"/>
 <layer number="39" name="tKeepout" color="4" fill="11" visible="no" active="no"/>
 <layer number="40" name="bKeepout" color="1" fill="11" visible="no" active="no"/>
@@
 <layer number="44" name="Drills" color="7" fill="1" visible="no" active="no"/>
 <layer number="45" name="Holes" color="7" fill="1" visible="no" active="no"/>
-<layer number="46" name="Milling" color="3" fill="1" visible="yes" active="no"/>
-<layer number="47" name="Measures" color="7" fill="1" visible="yes" active="no"/>
-<layer number="48" name="Document" color="7" fill="1" visible="yes" active="no"/>
-<layer number="49" name="Reference" color="7" fill="1" visible="yes" active="no"/>
-<layer number="50" name="dxf" color="7" fill="1" visible="yes" active="no"/>
-<layer number="51" name="tDocu" color="7" fill="1" visible="yes" active="no"/>
-<layer number="52" name="bDocu" color="7" fill="1" visible="yes" active="no"/>
-<layer number="53" name="tGND_GNDA" color="7" fill="9" visible="yes" active="no"/>
-<layer number="54" name="bGND_GNDA" color="1" fill="9" visible="yes" active="no"/>
-<layer number="55" name="tPotisk" color="7" fill="1" visible="yes" active="no"/>
-<layer number="56" name="wert" color="7" fill="1" visible="yes" active="no"/>
-<layer number="57" name="tCAD" color="7" fill="1" visible="yes" active="no"/>
-<layer number="58" name="bNC" color="7" fill="1" visible="yes" active="no"/>
-<layer number="59" name="tCarbon" color="7" fill="1" visible="yes" active="no"/>
-<layer number="60" name="bCarbon" color="7" fill="1" visible="yes" active="no"/>
-<layer number="61" name="stand" color="7" fill="1" visible="yes" active="no"/>
+<layer number="46" name="Milling" color="3" fill="1" visible="no" active="no"/>
+<layer number="47" name="Measures" color="7" fill="1" visible="no" active="no"/>
+<layer number="48" name="Document" color="7" fill="1" visible="no" active="no"/>
+<layer number="49" name="Reference" color="7" fill="1" visible="no" active="no"/>
+<layer number="50" name="dxf" color="7" fill="1" visible="no" active="no"/>
+<layer number="51" name="tDocu" color="7" fill="1" visible="no" active="no"/>
+<layer number="52" name="bDocu" color="7" fill="1" visible="no" active="no"/>
+<layer number="53" name="tGND_GNDA" color="7" fill="9" visible="no" active="no"/>
+<layer number="54" name="bGND_GNDA" color="1" fill="9" visible="no" active="no"/>
+<layer number="55" name="tPotisk" color="7" fill="1" visible="no" active="no"/>
+<layer number="56" name="wert" color="7" fill="1" visible="no" active="no"/>
+<layer number="57" name="tCAD" color="7" fill="1" visible="no" active="no"/>
+<layer number="58" name="bNC" color="7" fill="1" visible="no" active="no"/>
+<layer number="59" name="tCarbon" color="7" fill="1" visible="no" active="no"/>
+<layer number="60" name="bCarbon" color="7" fill="1" visible="no" active="no"/>
+<layer number="61" name="stand" color="7" fill="1" visible="no" active="no"/>
 <layer number="88" name="SimResults" color="9" fill="1" visible="yes" active="yes"/>
 <layer number="89" name="SimProbes" color="9" fill="1" visible="yes" active="yes"/>
@@
 </segment>
 <segment>
-<wire x1="73.66" y1="190.5" x2="71.12" y2="190.5" width="0.1524" layer="91"/>
-<label x="71.12" y="190.5" size="1.27" layer="95" rot="R180" xref="yes"/>
-<pinref part="IM1" gate="G$1" pin="IO13"/>
-</segment>
-</net>
-<net name="MODE_485" class="0">
-<segment>
 <wire x1="114.3" y1="193.04" x2="116.84" y2="193.04" width="0.1524" layer="91"/>
 <label x="116.84" y="193.04" size="1.27" layer="95" xref="yes"/>
@@
 </segment>
 </net>
+<net name="MODE_485" class="0">
+<segment>
+<wire x1="73.66" y1="190.5" x2="71.12" y2="190.5" width="0.1524" layer="91"/>
+<label x="71.12" y="190.5" size="1.27" layer="95" rot="R180" xref="yes"/>
+<pinref part="IM1" gate="G$1" pin="IO13"/>
+</segment>
+</net>

Commit message: 3.KSK
Parts:
- added Q4: BSS84, Transistor:BSS84
- added R21, R23, R26: 180, rcl:R-EU_R0402
Connections:
- new net !ENC-A: R23.1, U$62.A
- new net !ENC-B: R21.1, U$62.B
- new net !SW0: C71.2, Q4.G, R1.1, R18.2, U$62.SW-A
- new net SW!0: Q4.D, R26.1
- net +3V3: now also Q4.S
- net ENC-A: now also IM1.IO5, R23.2; no longer IM1.IO18, U$62.A
- net ENC-B: now also R21.2; no longer U$62.B
- net MOTOR: now also IM1.IO26; no longer IM1.IO2
- net SW0: now also IM1.IO18, R26.2; no longer C71.2, IM1.IO5, R1.1, R18.2, U$62.SW-A
- net TX_485: now also IM1.IO2; no longer IM1.IO26
Other:
- moved on the sheet: C2, C3, C4, C5, C71, Q5, Q9, R1, R15, R18, R19, R4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

Commit message: ladeni_drah
Parts:
- removed R1: 10k, rcl:R-EU_R0402
- added D2: (no value), diode:DIODE-DO214BA
- added R24: 10k, rcl:R-EU_R0402
- C6: device rcl:C-EUC0402K -> rcl:C-EUC0603
- C7: device rcl:C-EUC0603 -> rcl:C-EUC0402
- R26: value 180 -> 220
Connections:
- removed net AD0: U1.AD0
- removed net CLKIN: U1.CLKIN
- removed net FSYNC: U1.FSYNC
- net !SW0: no longer R1.1
- net +3V3: no longer R1.2
- net GND: now also D2.A, R24.2, U1.AD0, U1.CLKIN, U1.FSYNC
- net RX-GPS: now also IM1.IO16; no longer IM1.IO4
- net SW0: now also R24.1
- net TX-GPS: now also IM1.IO4; no longer IM1.IO16
- net VCC: now also D2.C
Other:
- moved on the sheet: R21, R23, R4, R5

Commit message: ladeni_drah
Parts:
- removed NC12: NC, NC:NC
- added C72, C73, C74: 10uf, rcl_upravena:C-EUC0402
- added JP5: (no value), pinhead:PINHD-1X4
- added NC15: NC, NC:NC
- C1, C10, C11, C12, C13, C14, C15, C16, C17, C18, C19, C2, C20, C21, C22, C23, C24, C25, C26, C27, C28, C29, C3, C30, C31, C32, C33, C34, C35, C36, C37, C38, C39, C40, C42, C43, C44, C45, C46, C47, C48, C49, C5, C50, C51, C52, C53, C54, C55, C56, C57, C58, C59, C60, C61, C62, C63, C64, C65, C66, C67, C68, C9: device rcl:C-EUC0402K -> rcl_upravena:C-EUC0402
- C41: value (none) -> 100pf; device rcl:C-EUC0402K -> rcl_upravena:C-EUC0402
- C6: device rcl:C-EUC0603 -> rcl_upravena:C-EUC0402
- C7: device rcl:C-EUC0402 -> rcl_upravena:C-EUC0402
- C71: device rcl:C-EUC0603 -> rcl_upravena:C-EUC0603
- C8: device rcl:C-EUC0402K -> rcl_upravena:C-EU
- R18: value 2M -> 1M
- R24: value 10k -> 47k
- U$1: value CR2032THM -> CR2032; device CR2032:CR2032THM -> CR2032:CR2032
Connections:
- removed net IO10_NC3: IC2.NC-5, NC12.NC
- removed net IO11_NC2: IC2.NC-3, NC10.NC
- removed net SW!0: Q4.D, R26.1
- new net IO9_NC6: IC2.NC-5, NC11.NC
- new net IO9_NC7: IC2.NC-4, NC15.NC
- new net N$7: Q4.S, R26.1
- net +3V3: now also C72.1, C73.1, C74.1, JP5.4, R24.2; no longer Q4.S
- net 3,3!KNOFLIK: no longer U$1.+1
- net GND: now also C72.2, C73.2, C74.2, JP5.3, Q4.D; no longer R24.2
- net IO10_NC2: now also IC2.NC-3; no longer IC2.NC-2
- net IO9_NC2: now also IC2.NC-2; no longer IC2.NC-1
- net IO9_NC3: now also IC2.NC-1, NC10.NC; no longer IC2.NC-4, NC11.NC
- net SCL: now also JP5.2
- net SDA: now also JP5.1
Other:
- moved on the sheet: C6, C69, C7, C70, C71, C8, D2, JP1, MAX1, Q1, Q10, Q2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

Commit message: srazeni_ceny
-vymena_tranzistoru
Parts:
- C8: device rcl_upravena:C-EU -> rcl_upravena:C-EUC0603
- Q2, Q8, Q9: value BSO201SP -> AO3401ASOP-8_EP_5.0X5.0X1.27P; device transistor-fet:BSO201SP -> transistor-fet:AO3401ASOP-8_EP_5.0X5.0X1.27P
- Q3: value (none) -> AO3401ASOP-8_EP_5.0X5.0X1.27P; device transistors:N-MOSFET-SO8 -> transistor-fet:AO3401ASOP-8_EP_5.0X5.0X1.27P

Commit message: diry_pro_srouby
Parts:
- C8: device rcl_upravena:C-EUC0603 -> rcl_upravena:C-EU
- R2, R3: value 47k -> 10k
- R20: device rcl:R-EU_R0603 -> rcl:R-EU_R0402
- R25: value 1k -> 270
Other:
- moved on the sheet: Q2, Q3
Changed lines of the file:
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@@
 <part name="C1" library="rcl_upravena" deviceset="C-EU" device="C0402" value="1nf"/>
 <part name="GND5" library="supply1" deviceset="GND" device=""/>
-<part name="R2" library="rcl" library_urn="urn:adsk.eagle:library:334" deviceset="R-EU_" device="R0402" package3d_urn="urn:adsk.eagle:package:23547/3" value="47k"/>
-<part name="R3" library="rcl" library_urn="urn:adsk.eagle:library:334" deviceset="R-EU_" device="R0402" package3d_urn="urn:adsk.eagle:package:23547/3" value="47k"/>
+<part name="R2" library="rcl" library_urn="urn:adsk.eagle:library:334" deviceset="R-EU_" device="R0402" package3d_urn="urn:adsk.eagle:package:23547/3" value="10k"/>
+<part name="R3" library="rcl" library_urn="urn:adsk.eagle:library:334" deviceset="R-EU_" device="R0402" package3d_urn="urn:adsk.eagle:package:23547/3" value="10k"/>
 <part name="+3V2" library="supply1" deviceset="+3V3" device=""/>
 <part name="+3V3" library="supply1" deviceset="+3V3" device=""/>
@@
 <part name="C7" library="rcl_upravena" deviceset="C-EU" device="C0402" value="4.7uf"/>
 <part name="GND15" library="supply1" deviceset="GND" device=""/>
-<part name="C8" library="rcl_upravena" deviceset="C-EU" device="C0603" value="100nf"/>
+<part name="C8" library="rcl_upravena" deviceset="C-EU" device="" value="100nf"/>
 <part name="GND17" library="supply1" deviceset="GND" device=""/>
 <part name="C9" library="rcl_upravena" deviceset="C-EU" device="C0402"/>
@@
 <part name="Q9" library="transistor-fet" deviceset="AO3401A" device="SOP-8_EP_5.0X5.0X1.27P" value="AO3401ASOP-8_EP_5.0X5.0X1.27P"/>
 <part name="D1" library="diode" library_urn="urn:adsk.eagle:library:210" deviceset="DIODE-" device="DO214BA" package3d_urn="urn:adsk.eagle:package:43453/2"/>
-<part name="R20" library="rcl" library_urn="urn:adsk.eagle:library:334" deviceset="R-EU_" device="R0603" package3d_urn="urn:adsk.eagle:package:23555/3" value="47k"/>
+<part name="R20" library="rcl" library_urn="urn:adsk.eagle:library:334" deviceset="R-EU_" device="R0402" package3d_urn="urn:adsk.eagle:package:23547/3" value="47k"/>
 <part name="+3V13" library="supply1" deviceset="+3V3" device=""/>
 <part name="R22" library="rcl" library_urn="urn:adsk.eagle:library:334" deviceset="R-EU_" device="R0402" package3d_urn="urn:adsk.eagle:package:23547/3" value="100k"/>
@@
 <part name="JP8" library="pinhead" library_urn="urn:adsk.eagle:library:325" deviceset="PINHD-1X1" device="" package3d_urn="urn:adsk.eagle:package:22485/2"/>
 <part name="LED4" library="led" library_urn="urn:adsk.eagle:library:259" deviceset="LED" device="SML0603" package3d_urn="urn:adsk.eagle:package:15832/1" value="powerled"/>
-<part name="R25" library="resistor" library_urn="urn:adsk.eagle:library:348" deviceset="R-EU_" device="R0402" package3d_urn="urn:adsk.eagle:package:26058/1" value="1k"/>
+<part name="R25" library="resistor" library_urn="urn:adsk.eagle:library:348" deviceset="R-EU_" device="R0402" package3d_urn="urn:adsk.eagle:package:26058/1" value="270"/>
 <part name="GND153" library="supply1" deviceset="GND" device=""/>
 <part name="MAX1" library="maxim" deviceset="MAX485" device="" package3d_urn="urn:adsk.eagle:package:17511/1"/>
@@
 <attribute name="NAME" x="121.92" y="74.549" size="1.778" layer="95" rot="R180"/>
 </instance>
-<instance part="Q3" gate="G$1" x="137.16" y="66.04" smashed="yes" rot="MR270">
-<attribute name="VALUE" x="137.16" y="77.47" size="1.778" layer="96" rot="MR270"/>
-<attribute name="NAME" x="138.684" y="66.802" size="1.778" layer="95" rot="MR0"/>
+<instance part="Q3" gate="G$1" x="137.16" y="63.5" smashed="yes" rot="MR270">
+<attribute name="VALUE" x="140.97" y="55.88" size="1.778" layer="96" rot="MR0"/>
+<attribute name="NAME" x="136.144" y="66.802" size="1.778" layer="95" rot="MR0"/>
 </instance>
 <instance part="GND140" gate="1" x="144.78" y="53.34" smashed="yes">
@@
 <pinref part="Q3" gate="G$1" pin="S"/>
 <pinref part="GND140" gate="1" pin="GND"/>
-<wire x1="142.24" y1="66.04" x2="144.78" y2="63.5" width="0.1524" layer="91"/>
+<wire x1="142.24" y1="63.5" x2="144.78" y2="63.5" width="0.1524" layer="91"/>
 <wire x1="144.78" y1="63.5" x2="144.78" y2="55.88" width="0.1524" layer="91"/>
 </segment>
@@
 <wire x1="139.7" y1="76.2" x2="139.7" y2="71.12" width="0.1524" layer="91"/>
 <pinref part="R11" gate="G$1" pin="2"/>
+<wire x1="139.7" y1="71.12" x2="139.7" y2="68.58" width="0.1524" layer="91"/>
 <wire x1="152.4" y1="68.58" x2="152.4" y2="71.12" width="0.1524" layer="91"/>
-<wire x1="152.4" y1="71.12" x2="139.7" y2="71.12" width="0.1524" layer="91"/>
 <pinref part="Q3" gate="G$1" pin="G"/>
+<wire x1="152.4" y1="71.12" x2="139.7" y2="71.12" width="0.1524" layer="91"/>
 <junction x="139.7" y="71.12"/>
 </segment>
@@
 <wire x1="127" y1="63.5" x2="129.54" y2="63.5" width="0.1524" layer="91"/>
 <pinref part="D1" gate="G$1" pin="A"/>
-<wire x1="129.54" y1="63.5" x2="132.08" y2="66.04" width="0.1524" layer="91"/>
+<wire x1="129.54" y1="63.5" x2="132.08" y2="63.5" width="0.1524" layer="91"/>
 <wire x1="129.54" y1="66.04" x2="129.54" y2="63.5" width="0.1524" layer="91"/>
 <junction x="129.54" y="63.5"/>
@@
 <attribute name="VALUE" x="25.4" y="50.8" size="1.778" layer="96" rot="R90"/>
 </instance>
-<instance part="Q2" gate="G$1" x="25.4" y="111.76" smashed="yes" rot="R90">
-<attribute name="NAME" x="22.86" y="116.84" size="1.778" layer="95" rot="R90"/>
-<attribute name="VALUE" x="25.4" y="116.84" size="1.778" layer="96" rot="R90"/>
+<instance part="Q2" gate="G$1" x="25.4" y="114.3" smashed="yes" rot="MR90">
+<attribute name="NAME" x="22.86" y="116.84" size="1.778" layer="95" rot="MR90"/>
+<attribute name="VALUE" x="25.4" y="119.38" size="1.778" layer="96" rot="MR90"/>
 </instance>
 <instance part="R22" gate="G$1" x="30.48" y="81.28" smashed="yes" rot="R90">
@@
 </segment>
 <segment>
-<wire x1="20.32" y1="111.76" x2="33.02" y2="114.3" width="0.1524" layer="91"/>
+<wire x1="30.48" y1="114.3" x2="33.02" y2="114.3" width="0.1524" layer="91"/>
 <wire x1="33.02" y1="114.3" x2="33.02" y2="116.84" width="0.1524" layer="91"/>
 <pinref part="P+63" gate="VCC" pin="VCC"/>
@@
 <wire x1="22.86" y1="96.52" x2="22.86" y2="99.06" width="0.1524" layer="91"/>
 <pinref part="R6" gate="G$1" pin="2"/>
-<wire x1="22.86" y1="99.06" x2="27.94" y2="106.68" width="0.1524" layer="91"/>
+<wire x1="22.86" y1="99.06" x2="22.86" y2="109.22" width="0.1524" layer="91"/>
 <wire x1="17.78" y1="101.6" x2="17.78" y2="99.06" width="0.1524" layer="91"/>
 <wire x1="17.78" y1="99.06" x2="22.86" y2="99.06" width="0.1524" layer="91"/>
@@
 <net name="+5V" class="0">
 <segment>
-<wire x1="30.48" y1="111.76" x2="17.78" y2="114.3" width="0.1524" layer="91"/>
+<wire x1="20.32" y1="114.3" x2="17.78" y2="114.3" width="0.1524" layer="91"/>
 <wire x1="17.78" y1="114.3" x2="17.78" y2="116.84" width="0.1524" layer="91"/>
 <pinref part="P+64" gate="1" pin="+5V"/>
