File: ele/Blackbox/main_board/board.sch (EAGLE design)
At the start: 203 parts, among them IC1 DS3231/SO, IC2 QMC5883L-TR, Q2 AO3401ASOP-8_EP_5.0X5.0X1.27P, Q3 AO3401ASOP-8_EP_5.0X5.0X1.27P, Q4 BSS84, Q8 AO3401ASOP-8_EP_5.0X5.0X1.27P, Q9 AO3401ASOP-8_EP_5.0X5.0X1.27P, U1 MPU-6050

Commit message: kondikyí_k_encoderu
Parts:
- added C75, C76: 220nf, rcl_upravena:C-EUC0402
Connections:
- net !ENC-A: now also C75.1
- net !ENC-B: now also C76.1
- net GND: now also C75.2, C76.2

Commit message: dokumentace ke SchoolBoardu
Parts:
- removed Q8: AO3401ASOP-8_EP_5.0X5.0X1.27P, transistor-fet:AO3401ASOP-8_EP_5.0X5.0X1.27P
- added C77, C78, C79, C80, C82, C83, C84: 10uf, rcl_upravena:C-EUC0805
- added C81: (no value), rcl:CPOL-EU
- added D3, D4, D5: BAT60JDO-214-AB, diode:BAT60JDO-214-AB
- added J1: (no value), SD-kart:693072010801
- added NC12, NC16, NC17, NC18, NC19, NC20: NC, NC:NC
- added Q11, Q7: (no value), transistors:N-MOSFET-SOT23-GSD
- added R1: 300k, rcl:R-EU_R0402
- added R27, R28, R29: (no value), rcl:R-EU_R0402
- added U2: V_REG_317SMD, SparkFun-IC-Power:V_REG_317SMD
- C4: device rcl:C-EUC0402K -> rcl_upravena:C-EU
- C69, C70: device rcl:C-EUC0402K -> rcl:C-EUC0805
- C7, C72, C73, C74: device rcl_upravena:C-EUC0402 -> rcl_upravena:C-EUC0805
- C71: value 4.7uf -> 100nf; device rcl_upravena:C-EUC0603 -> rcl_upravena:C-EU
- JP2: device pinhead:PINHD-2X6 -> pinhead:PINHD-2X2
- Q4: value BSS84 -> (none); device Transistor:BSS84 -> transistors:N-MOSFET-SOT23-GSD
- R15: value 300k -> 100k; device rcl:R-EU_R0603 -> rcl:R-EU_R0402
- R18: value 1M -> (none); device rcl:R-EU_R0603 -> rcl:R-EU_R0402
- R24: value 47k -> 10k
- R25: value 270 -> 1k
- R26: value 220 -> 100k
Connections:
- removed net !SW0: C71.2, Q4.G, R18.2, U$62.SW-A
- removed net IO32: IM1.IO32, JP2.10
- removed net IO33: IM1.IO33, JP2.12
- removed net IO35: IM1.IO35, JP2.8
- removed net N$71: Q3.G, R10.1, R11.2
- removed net SVP: IM1.SVP, JP2.2
- new net +5VA: C79.1, C80.1, C81.+, D5.C, IM1.5V, LED4.A
- new net CLK: IM1.IO18, J1.CLK, R27.2
- new net IO11_NC2: J1.P$10, NC12.NC
- new net IO11_NC3: J1.P$12, NC16.NC
- new net IO11_NC4: J1.P$11, NC17.NC
- new net IO11_NC5: J1.P$9, NC18.NC
- new net MISO: IM1.IO19, J1.DAT0, R18.2
- new net MOSI: IM1.IO22, J1.CMD, R28.2, R29.2
- new net N$11: D1.C, MOTOR-2.KL, Q3.D
- new net N$12: Q3.G, Q7.D, R1.1
- new net N$13: Q7.G, R10.1
- new net N$14: C77.1, D4.C, Q3.S, R1.2
- new net N$20: J1.DAT2, NC20.NC
- new net SS: IM1.IO5, J1.CD/DAT3
- new net SW: IM1.IO35, Q11.D, R24.1
- new net SW1: Q11.G, Q4.G, R26.1, U$62.SW-B
- net +5V: now also C84.2, D3.A, D4.A, D5.A, U2.IN; no longer D1.C, IM1.5V, LED4.A, MOTOR-2.KL, Q2.S, R6.1, R9.1
- net ENC-A: now also IM1.IO21; no longer IM1.IO5
- net GND: now also C77.2, C78.2, C79.2, C80.2, C81.-, C82.1, C83.2, C84.1, D1.A, J1.VSS, MOTOR-1.KL, Q11.S, Q4.S, Q7.S, R18.1, R26.2, R27.1, R28.1, R29.1, U2.ADJ; no longer JP2.11, JP2.5, JP2.7, JP2.9, Q3.S, Q4.D, Q8.G, R11.1, U$62.SW-B
- net IO34: now also JP2.2; no longer JP2.6
- net N$2: now also C71.2, Q4.D, R11.2; no longer D1.A, MOTOR-1.KL, Q3.D
- net N$4: now also J1.DAT1, NC19.NC; no longer Q8.D, X1-1.KL, X2-1.KL
- net N$5: now also C82.2, C83.1, J1.VDD, U2.OUT; no longer Q8.S, Q9.S, R15.2
- net N$6: now also R11.1; no longer R18.1
- net N$7: now also C78.1, D3.C, Q2.S, R6.1; no longer Q4.S, R26.1
- net QMC5883-INTERRUPT: now also IM1.IO32; no longer IM1.IO19
- net RX-GPS: now also IM1.IO4; no longer IM1.IO16
- net SCL: now also IM1.SVP; no longer IM1.IO22
- net SQW/INT: now also IM1.IO33; no longer IM1.IO21
- net SW0: now also Q9.S, R15.2, U$62.SW-A, X1-1.KL, X2-1.KL; no longer IM1.IO18, R24.1, R26.2
- net TX-GPS: now also IM1.IO16; no longer IM1.IO4
- net VCC: now also R9.1
Other:
- moved on the sheet: C1, C6, C7, C71, C8, D1, D2, IC1, IM1, JP8, LED4, MOTOR-1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

Commit message: SD-karta_na_BlackBoxu
Parts:
- removed U2: V_REG_317SMD, SparkFun-IC-Power:V_REG_317SMD
- added C85, C86, C87: 10uf, rcl_upravena:C-EUC0805
- R18, R27, R28, R29: value (none) -> 10k
Connections:
- removed net N$5: C82.2, C83.1, J1.VDD, U2.OUT
- net +3V3: now also C82.2, C83.2, C84.2, C85.2, C86.1, C87.1, J1.VDD
- net +5V: no longer C84.2, U2.IN
- net GND: now also C83.1, C85.1, C86.2, C87.2; no longer C83.2, U2.ADJ
- net MOSI: no longer R29.2
- net SS: now also R29.2
Other:
- moved on the sheet: C82, C83, C84, R18, R27, R28, R29

Commit message: dalsi_text_a_firstbot
Parts:
- removed C82, C83, C84, C85, C87: 10uf, rcl_upravena:C-EUC0805
- removed J1: (no value), SD-kart:693072010801
- removed NC12, NC16, NC17, NC18, NC19, NC20: NC, NC:NC
- removed R18, R27, R28, R29, R8: 10k, rcl:R-EU_R0402
- JP2: device pinhead:PINHD-2X2 -> pinhead:PINHD-2X6
Connections:
- removed net CLK: IM1.IO18, J1.CLK, R27.2
- removed net IO11_NC2: J1.P$10, NC12.NC
- removed net IO11_NC3: J1.P$12, NC16.NC
- removed net IO11_NC4: J1.P$11, NC17.NC
- removed net IO11_NC5: J1.P$9, NC18.NC
- removed net MISO: IM1.IO19, J1.DAT0, R18.2
- removed net MOSI: IM1.IO22, J1.CMD, R28.2
- removed net N$20: J1.DAT2, NC20.NC
- removed net N$4: J1.DAT1, NC19.NC
- removed net SS: IM1.IO5, J1.CD/DAT3, R29.2
- new net IO32: IM1.IO32, JP2.10
- new net IO33: IM1.IO33, JP2.12
- new net IO35: IM1.IO35, JP2.8
- new net SVP: IM1.SVP, JP2.2
- net +3V3: no longer C82.2, C83.2, C84.2, C85.2, C87.1, J1.VDD, R8.1
- net ENC-A: now also IM1.IO5; no longer IM1.IO21
- net GND: now also JP2.11, JP2.5, JP2.7, JP2.9; no longer C82.1, C83.1, C84.1, C85.1, C87.2, J1.VSS, R18.1, R27.1, R28.1, R29.1
- net IO34: now also JP2.6; no longer JP2.2
- net QMC5883-INTERRUPT: now also IM1.IO19; no longer IM1.IO32
- net SCL: now also IM1.IO22; no longer IM1.SVP
- net SQW/INT: now also IM1.IO21; no longer IM1.IO33
- net SW: now also IM1.IO18; no longer IM1.IO35
- net WS2812: no longer R8.2
Other:
- moved on the sheet: LED4, R25

Commit message: trochu v tom delam bordel
proste to neumim delat poredne tak tet delam tenhle bordel commit bych mel vse na gitu a budu se snazit to dal delat poradne
Connections:
- net +3V3: now also U1.AD0
- net GND: no longer U1.AD0
- net N$62: now also IC2.SETP; no longer IC2.STEP
