File: ele/Blackbox/main_board/board.brd (EAGLE design)
At the start: 112.7 x 112.7 mm, 189 parts, among them IC1 DS3231/SO, IC2 QMC5883L-TR, Q2 AO3401ASOP-8_EP_5.0X5.0X1.27P, Q3 AO3401ASOP-8_EP_5.0X5.0X1.27P, Q4 BSS84, Q8 AO3401ASOP-8_EP_5.0X5.0X1.27P, Q9 AO3401ASOP-8_EP_5.0X5.0X1.27P, U1 MPU-6050

Commit message: vyrobni_data
Parts:
- moved Q3 1.50 mm to (70.1, 26.7)
- moved Q9 1.50 mm to (48.7, 27.0)
- moved Q2 1.40 mm to (47.0, 17.6)
- moved Q8 1.40 mm to (53.3, 17.6)
- moved R10 0.60 mm to (75.5, 30.5)
- moved R11 0.60 mm to (75.5, 29.2)
Routing:
- net N$68: track 12.2 -> 8.25 mm
- net N$71: track 10.3 -> 14.2 mm
- net N$6: track 16.7 -> 12.9 mm, vias 2 -> 0
- net GND: track 2.42 -> 0.95 mm, vias 145 -> 146
- net MOTOR: track 39.3 -> 38.7 mm

Commit message: kondikyí_k_encoderu
Parts:
- added C75, C76: 220nf, rcl_upravena:C0402
Connections:
- net !ENC-A: now also C75.1
- net !ENC-B: now also C76.1
- net GND: now also C75.2, C76.2
Routing:
- net !ENC-A: track 13.5 -> 16.1 mm
- net !ENC-B: track 7.94 -> 10.2 mm
Changed lines of the file:
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@@
 <text x="40.64" y="16.51" size="1.778" layer="26" rot="MR270">B</text>
 <text x="43.18" y="16.51" size="1.778" layer="26" rot="MR270">+5v</text>
-<text x="36.83" y="91.44" size="1.778" layer="26" rot="MR180">RB3203_BLACK-BOX-BOARD_V1</text>
+<text x="38.1" y="88.9" size="1.778" layer="26" rot="MR180">RB3203_BLACK-BOX-BOARD_V1</text>
 <wire x1="74.041" y1="73.9267" x2="73.533" y2="73.9267" width="0.15" layer="41"/>
 <wire x1="74.0537" y1="74.8792" x2="73.5457" y2="74.8792" width="0.15" layer="41"/>
@@
 <hole x="100.33" y="12.7" drill="3.5"/>
 <hole x="12.7" y="12.7" drill="3.5"/>
+<wire x1="58.808" y1="44.9762" x2="58.808" y2="45.4842" width="0.15" layer="41"/>
+<wire x1="57.988" y1="44.9262" x2="57.988" y2="45.4342" width="0.15" layer="41"/>
+<wire x1="55.068" y1="45.0062" x2="55.068" y2="45.5142" width="0.15" layer="41"/>
+<wire x1="54.158" y1="44.9862" x2="54.158" y2="45.4942" width="0.15" layer="41"/>
 </plain>
 <attributes>
@@
 <attribute name="MF" value="Maxim Integrated" x="76.2" y="17.78" size="1.778" layer="27" display="off"/>
 <attribute name="MP" value="DS3231" x="76.2" y="17.78" size="1.778" layer="27" display="off"/>
-<attribute name="NAME" x="38.1" y="83.185" size="1.27" layer="25" rot="R270"/>
+<attribute name="NAME" x="24.6" y="82.585" size="1.27" layer="25" rot="R270"/>
 <attribute name="PACKAGE" value="SOIC-16 Maxim Integrated" x="76.2" y="17.78" size="1.778" layer="27" display="off"/>
 <attribute name="PRICE" value="None" x="76.2" y="17.78" size="1.778" layer="27" display="off"/>
-<attribute name="VALUE" x="39.37" y="86.36" size="1.27" layer="27"/>
+<attribute name="VALUE" x="39.37" y="76.2" size="1.27" layer="27" rot="R90"/>
 </element>
 <element name="JP3" library="pinhead" library_urn="urn:adsk.eagle:library:325" package="1X04" package3d_urn="urn:adsk.eagle:package:22407/2" value="" x="81.28" y="45.72" smashed="yes" rot="MR0">
@@
 <attribute name="VALUE" x="89.535" y="81.915" size="1.27" layer="27" rot="R180"/>
 </element>
+<element name="C75" library="rcl_upravena" package="C0402" value="220nf" x="54.61" y="45.72" smashed="yes" rot="R270">
+<attribute name="NAME" x="55.245" y="46.355" size="1.27" layer="25" rot="R270"/>
+<attribute name="VALUE" x="52.705" y="46.355" size="1.27" layer="27" rot="R270"/>
+</element>
+<element name="C76" library="rcl_upravena" package="C0402" value="220nf" x="58.42" y="45.72" smashed="yes" rot="R270">
+<attribute name="NAME" x="59.055" y="46.355" size="1.27" layer="25" rot="R270"/>
+<attribute name="VALUE" x="56.515" y="46.355" size="1.27" layer="27" rot="R270"/>
+</element>
 </elements>
 <signals>
@@
 <wire x1="51.445" y1="20.57" x2="51.445" y2="21.475" width="0.254" layer="1"/>
 <via x="51.439" y="21.469" extent="1-16" drill="0.35"/>
+<contactref element="C76" pad="2"/>
+<contactref element="C75" pad="2"/>
 </signal>
 <signal name="+5V">
@@
 <wire x1="63.5" y1="54.61" x2="64.27" y2="54.61" width="0.3048" layer="1"/>
 <wire x1="58.6424" y1="49.7524" x2="63.5" y2="54.61" width="0.3048" layer="1"/>
+<contactref element="C75" pad="1"/>
+<wire x1="53.38" y1="48.38" x2="54.61" y2="47.15" width="0.2" layer="1"/>
+<wire x1="54.61" y1="47.15" x2="54.61" y2="46.22" width="0.2" layer="1"/>
 </signal>
 <signal name="!ENC-B">
@@
 <wire x1="58.38" y1="48.38" x2="58.54" y2="48.38" width="0.3048" layer="1"/>
 <wire x1="63.5" y1="53.34" x2="58.54" y2="48.38" width="0.3048" layer="1"/>
+<contactref element="C76" pad="1"/>
+<wire x1="58.42" y1="46.22" x2="58.42" y2="48.26" width="0.2" layer="1"/>
+<wire x1="58.42" y1="48.26" x2="58.54" y2="48.38" width="0.2" layer="1"/>
 </signal>
 <signal name="!SW0">

Commit message: dokumentace ke SchoolBoardu
Parts:
- removed Q8: AO3401ASOP-8_EP_5.0X5.0X1.27P, transistor-fet:SOP-8_EP_5.0X5.0X1.27P
- added C77, C78, C79, C80, C82, C83, C84: 10uf, rcl_upravena:C0805
- added C81: (no value), rcl:E5-10,5-H
- added D3, D4, D5: BAT60JDO-214-AB, diode:DO214BA
- added J1: (no value), SD-kart:693072010801
- added Q11, Q7: (no value), transistors:SOT23
- added R1: 300k, rcl:R0402
- added R27, R28, R29: (no value), rcl:R0402
- added U2: V_REG_317SMD, SparkFun-IC-Power:SOT223
- C4: device rcl:C0402K -> rcl_upravena:C0402P
- C69, C70: device rcl:C0402K -> rcl:C0805
- C7, C72, C73, C74: device rcl_upravena:C0402 -> rcl_upravena:C0805
- C71: value 4.7uf -> 100nf; device rcl_upravena:C0603 -> rcl_upravena:C0402P
- JP2: device pinhead:2X06 -> pinhead:2X02
- Q4: value BSS84 -> (none); device Transistor:SOT23 -> transistors:SOT23
- R15: value 300k -> 100k; device rcl:R0603 -> rcl:R0402
- R18: value 1M -> (none); device rcl:R0603 -> rcl:R0402
- R24: value 47k -> 10k
- R25: value 270 -> 1k
- R26: value 220 -> 100k
- moved R18 79.3 mm to (-1.27, -25.4), turned to 0 degrees
- moved R11 21.0 mm to (54.6, 27.9)
- moved U$1 18.9 mm to (39.4, 68.6), turned to 90 degrees
- moved R26 18.9 mm to (52.1, 45.7), turned to 270 degrees
- moved C74 18.7 mm to (70.2, 80.1)
- moved JP3 15.3 mm to (80.0, 61.0)
- moved Q9 9.74 mm to (53.7, 18.6), turned to 180 degrees
- moved JP2 5.08 mm to (97.2, 64.1), flipped to the top, turned to 90 degrees
- moved C71 4.84 mm to (54.6, 29.2), turned to 180 degrees
- moved R5 4.02 mm to (71.1, 54.6)
- moved R19 4.02 mm to (71.1, 53.3)
- moved R4 4.02 mm to (71.1, 55.9)
- moved R24 3.10 mm to (71.1, 57.1)
- moved R10 2.64 mm to (78.2, 30.5), turned to 90 degrees
- moved R15 2.63 mm to (57.0, 28.6)
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Connections:
- removed net !SW0: C71.2, Q4.1, R18.2, U$62.P$4
- removed net IO32: IM1.7, JP2.10
- removed net IO33: IM1.8, JP2.12
- removed net IO35: IM1.6, JP2.8
- removed net N$71: Q3.4, R10.1, R11.2
- removed net SVP: IM1.3, JP2.2
- new net +5VA: C79.1, C80.1, C81.+, D5.C, IM1.19, LED4.A
- new net CLK: IM1.30, J1.5, R27.2
- new net IO11_NC2: J1.Z2
- new net IO11_NC3: J1.Z4
- new net IO11_NC4: J1.Z3
- new net IO11_NC5: J1.Z1
- new net MISO: IM1.31, J1.7, R18.2
- new net MOSI: IM1.36, J1.3, R28.2, R29.2
- new net N$11: D1.C, MOTOR.2, Q3.5, Q3.6, Q3.7, Q3.8, Q3.9
- new net N$12: Q3.4, Q7.3, R1.1
- new net N$13: Q7.1, R10.1
- new net N$14: C77.1, D4.C, Q3.1, Q3.2, Q3.3, R1.2
- new net N$20: J1.1
- new net SS: IM1.29, J1.2
- new net SW: IM1.6, Q11.3, R24.1
- new net SW1: Q11.1, Q4.1, R26.1, U$62.P$5
- net +5V: now also C84.2, D3.A, D4.A, D5.A, U2.3; no longer D1.C, IM1.19, LED4.A, MOTOR.2, Q2.1, Q2.2, Q2.3, R6.1, R9.1
- net ENC-A: now also IM1.33; no longer IM1.29
- net GND: now also C77.2, C78.2, C79.2, C80.2, C81.-, C82.1, C83.2, C84.1, D1.A, J1.6, MOTOR.1, Q11.2, Q4.2, Q7.2, R18.1, R26.2, R27.1, R28.1, R29.1, U2.1; no longer JP2.11, JP2.5, JP2.7, JP2.9, Q3.1, Q3.2, Q3.3, Q4.3, Q8.4, R11.1, U$62.P$5
- net IO34: now also JP2.2; no longer JP2.6
- net N$2: now also C71.2, Q4.3, R11.2; no longer D1.A, MOTOR.1, Q3.5, Q3.6, Q3.7, Q3.8, Q3.9
- net N$4: now also J1.8; no longer Q8.5, Q8.6, Q8.7, Q8.8, Q8.9, X1.1, X2.1
- net N$5: now also C82.2, C83.1, J1.4, U2.2; no longer Q8.1, Q8.2, Q8.3, Q9.1, Q9.2, Q9.3, R15.2
- net N$6: now also R11.1; no longer R18.1
- net N$7: now also C78.1, D3.C, Q2.1, Q2.2, Q2.3, R6.1; no longer Q4.2, R26.1
- net QMC5883-INTERRUPT: now also IM1.7; no longer IM1.31
- net RX-GPS: now also IM1.26; no longer IM1.27
- net SCL: now also IM1.3; no longer IM1.36
- net SQW/INT: now also IM1.8; no longer IM1.33
- net SW0: now also Q9.1, Q9.2, Q9.3, R15.2, U$62.P$4, X1.1, X2.1; no longer IM1.30, R24.1, R26.2
- net TX-GPS: now also IM1.27; no longer IM1.26
- net VCC: now also R9.1
Routing:
- net SW0: track 3.57 -> 96.2 mm, vias 0 -> 3
- net N$4: track 35.9 -> 0.00 mm
- net !SW0: track 35.8 -> 0.00 mm, vias 2 -> 0
- net MOSI: track 0.00 -> 34.1 mm, vias 0 -> 1
- net N$5: track 0.00 -> 28.3 mm, vias 0 -> 2
- net SQW/INT: track 56.9 -> 84.9 mm
- net SW1: track 0.00 -> 26.8 mm
- net +3V3: track 241.1 -> 216.2 mm, vias 7 -> 8
- net MISO: track 0.00 -> 24.5 mm
- net SCL: track 99.3 -> 121.6 mm, vias 0 -> 4
- net CLK: track 0.00 -> 22.0 mm
- net N$7: track 21.8 -> 0.00 mm
- net N$2: track 0.00 -> 21.5 mm, vias 0 -> 2
- net SS: track 0.00 -> 21.0 mm, vias 0 -> 1
- net +5V: track 95.6 -> 75.9 mm, vias 3 -> 5
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- added copper zone on layer 1, net +5VA
- added copper zone on layer 1, net N$11
- added copper zone on layer 1, net N$14
- added copper zone on layer 1, net N$7
- added copper zone on layer 1, net SW0
- removed copper zone on layer 1, net N$2
- removed copper zone on layer 1, net N$4
- removed copper zone on layer 1, net N$5

Commit message: SD-karta_na_BlackBoxu
Parts:
- removed U2: V_REG_317SMD, SparkFun-IC-Power:SOT223
- added C85, C86, C87: 10uf, rcl_upravena:C0805
- R18, R27, R28, R29: value (none) -> 10k
- moved R29 115.7 mm to (73.7, 51.3)
- moved R27 114.8 mm to (69.8, 61.0)
- moved R28 113.8 mm to (73.7, 52.6)
- moved R18 113.2 mm to (77.5, 55.9), turned to 180 degrees
- moved C84 106.7 mm to (88.4, 40.6), turned to 180 degrees
- moved C83 105.1 mm to (88.4, 44.2), turned to 180 degrees
- moved C82 102.7 mm to (88.4, 46.0), turned to 180 degrees
- moved C74 1.14 mm to (70.0, 79.0)
- moved R2 0.25 mm to (69.8, 77.2)
- moved R3 0.13 mm to (69.8, 76.2)
Connections:
- removed net N$5: C82.2, C83.1, J1.4, U2.2
- net +3V3: now also C82.2, C83.2, C84.2, C85.2, C86.1, C87.1, J1.4
- net +5V: no longer C84.2, U2.3
- net GND: now also C83.1, C85.1, C86.2, C87.2; no longer C83.2, U2.1
- net MOSI: no longer R29.2
- net SS: now also R29.2
Routing:
- net +3V3: track 216.2 -> 245.0 mm, vias 8 -> 9
- net N$5: track 28.3 -> 0.00 mm, vias 2 -> 0
- net SW: track 13.8 -> 37.2 mm, vias 1 -> 3
- net QMC5883-INTERRUPT: track 57.4 -> 71.1 mm, vias 2 -> 1
- net INT_MPU5060: track 23.0 -> 29.5 mm
- net SS: track 21.0 -> 26.4 mm
- net RX-485-5V: track 59.2 -> 55.1 mm, vias 0 -> 2
- net SCL: track 121.6 -> 118.4 mm, vias 4 -> 5
- net CLK: track 22.0 -> 24.3 mm
- net +5V: track 75.9 -> 73.6 mm
- net MISO: track 24.5 -> 26.5 mm
- net MOSI: track 34.1 -> 36.1 mm
- net LED-SHUTDOWN: track 61.3 -> 62.5 mm
- net MOTOR: track 36.8 -> 38.1 mm

Commit message: dalsi_text_a_firstbot
Parts:
- removed C82, C83, C84, C85, C87: 10uf, rcl_upravena:C0805
- removed J1: (no value), SD-kart:693072010801
- removed R18, R27, R28, R29, R8: 10k, rcl:R0402
- JP2: device pinhead:2X02 -> pinhead:2X06
- moved JP2 5.08 mm to (97.2, 59.1), flipped to the bottom, turned to 270 degrees
- moved R9 4.58 mm to (99.1, 45.7)
- moved C86 3.43 mm to (70.0, 81.0), turned to 180 degrees
- moved R10 2.05 mm to (79.4, 32.1)
Connections:
- removed net CLK: IM1.30, J1.5, R27.2
- removed net IO11_NC2: J1.Z2
- removed net IO11_NC3: J1.Z4
- removed net IO11_NC4: J1.Z3
- removed net IO11_NC5: J1.Z1
- removed net MISO: IM1.31, J1.7, R18.2
- removed net MOSI: IM1.36, J1.3, R28.2
- removed net N$20: J1.1
- removed net N$4: J1.8
- removed net SS: IM1.29, J1.2, R29.2
- new net IO32: IM1.7, JP2.10
- new net IO33: IM1.8, JP2.12
- new net IO35: IM1.6, JP2.8
- new net SVP: IM1.3, JP2.2
- net +3V3: no longer C82.2, C83.2, C84.2, C85.2, C87.1, J1.4, R8.1
- net ENC-A: now also IM1.29; no longer IM1.33
- net GND: now also JP2.11, JP2.5, JP2.7, JP2.9; no longer C82.1, C83.1, C84.1, C85.1, C87.2, J1.6, R18.1, R27.1, R28.1, R29.1
- net IO34: now also JP2.6; no longer JP2.2
- net QMC5883-INTERRUPT: now also IM1.31; no longer IM1.7
- net SCL: now also IM1.36; no longer IM1.3
- net SQW/INT: now also IM1.33; no longer IM1.8
- net SW: now also IM1.30; no longer IM1.6
- net WS2812: no longer R8.2
Routing:
- net MOSI: track 36.1 -> 0.00 mm, vias 1 -> 0
- net QMC5883-INTERRUPT: track 71.1 -> 38.4 mm, vias 1 -> 2
- net +3V3: track 245.0 -> 213.4 mm, vias 9 -> 8
- net SW: track 37.2 -> 6.44 mm, vias 3 -> 0
- net SQW/INT: track 84.9 -> 57.8 mm, vias 2 -> 1
- net MISO: track 26.5 -> 0.00 mm
- net SS: track 26.4 -> 0.00 mm, vias 1 -> 0
- net CLK: track 24.3 -> 0.00 mm
- net SCL: track 118.4 -> 98.8 mm, vias 5 -> 4
- net ENC-A: track 21.3 -> 7.27 mm
- net SVP: track 0.00 -> 10.8 mm
- net IO35: track 0.00 -> 10.8 mm
- net IO33: track 0.00 -> 10.8 mm
- net IO32: track 0.00 -> 10.8 mm
- net INT_MPU5060: track 29.5 -> 24.3 mm
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
Commit message: trochu v tom delam bordel
proste to neumim delat poredne tak tet delam tenhle bordel commit bych mel vse na gitu a budu se snazit to dal delat poradne
Parts:
- moved C7 0.38 mm to (56.8, 96.1)
- moved C6 0.13 mm to (56.8, 97.4)
Connections:
- net +3V3: now also IC2.4, U1.9; no longer IC2.S1
- net GND: no longer U1.9
Routing:
- net +3V3: track 213.4 -> 220.8 mm
- net SDA: track 87.9 -> 89.8 mm
Other:
- board text added: "+3V3"
- board text added: "IO32 GND"
- board text added: "IO33 GND"
- board text added: "IO34 GND"
- board text added: "IO35 GND"
- board text added: "RX-GPS"
- board text added: "SCL"
- board text added: "SDA"
- board text added: "SVN GND"
- board text added: "SVP GND"
- board text added: "TX-GPS"
