File: ele/TableBot/main_board.brd (EAGLE design)
At the start: 140 x 140 mm, 124 parts, among them IC1 MCP602ST, K1 ARK550/2, X4 POWER_IN

Commit message: 2.KSK
Parts:
- removed R7: 100k, rcl_upravena:R0805
- added Q11: (no value), transistors:MLP3.3X3.3_HS
Connections:
- removed net N$35: Q7.4, Q9.1, R7.2
- new net N$37: Q11.5, Q11.6, Q11.7, Q11.8, Q9.1
- net GND: now also Q11.1, Q11.2, Q11.3
- net N$7: now also Q11.4, Q7.4; no longer R7.1
Changed lines of the file:
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@@
 <attribute name="VALUE" x="-84.455" y="-548.64" size="1.27" layer="27"/>
-</element>
-<element name="R7" library="rcl_upravena" package="R0805" value="100k" x="-83.82" y="-553.72" smashed="yes">
-<attribute name="NAME" x="-84.455" y="-552.45" size="1.27" layer="25"/>
-<attribute name="VALUE" x="-84.455" y="-556.26" size="1.27" layer="27"/>
 </element>
 <element name="K1" library="#PaJa_konektory" package="ARK550/2" value="ARK550/2" x="-93.98" y="-551.18" smashed="yes">
@@
 <attribute name="NAME" x="-94.615" y="-581.025" size="1.27" layer="25"/>
 <attribute name="VALUE" x="-94.615" y="-583.565" size="1.27" layer="27"/>
+</element>
+<element name="Q11" library="transistors" package="MLP3.3X3.3_HS" value="" x="-101.6" y="-576.58" smashed="yes">
+<attribute name="NAME" x="-104.7" y="-573.98" size="1.27" layer="25" font="vector" ratio="16"/>
+<attribute name="VALUE" x="-104.7" y="-580.48" size="1.27" layer="27" font="vector" ratio="16"/>
 </element>
 </elements>
@@
 <contactref element="JP3" pad="3"/>
 <contactref element="Q10" pad="2"/>
+<contactref element="Q11" pad="2"/>
+<contactref element="Q11" pad="3"/>
+<contactref element="Q11" pad="1"/>
 <wire x1="-60.2488" y1="-185.6994" x2="-66.7512" y2="-185.6994" width="0" layer="19" extent="1-1"/>
 <wire x1="-66.04" y1="-193.83" x2="-66.7512" y2="-185.6994" width="0" layer="19" extent="1-1"/>
@@
 <wire x1="-88.9" y1="-568.96" x2="-88.9" y2="-561.34" width="0" layer="19" extent="1-1"/>
 <wire x1="-93.03" y1="-577.68" x2="-88.9" y2="-568.96" width="0" layer="19" extent="1-1"/>
+<wire x1="-101.275" y1="-578.28" x2="-93.03" y2="-577.68" width="0" layer="19" extent="1-1"/>
+<wire x1="-101.925" y1="-578.28" x2="-101.275" y2="-578.28" width="0" layer="19" extent="1-1"/>
+<wire x1="-102.575" y1="-578.28" x2="-101.925" y2="-578.28" width="0" layer="19" extent="1-1"/>
 <wire x1="-41.91" y1="-49.53" x2="-63.5" y2="-106.68" width="0" layer="19" extent="1-1"/>
 <wire x1="-39.37" y1="-46.99" x2="-41.91" y2="-49.53" width="0" layer="19" extent="1-1"/>
@@
 <contactref element="Q2" pad="8"/>
 <contactref element="R3" pad="1"/>
-<contactref element="R7" pad="1"/>
 <contactref element="Q9" pad="3"/>
-<wire x1="-84.77" y1="-546.1" x2="-84.77" y2="-553.72" width="0" layer="19" extent="1-1"/>
+<contactref element="Q7" pad="4"/>
+<contactref element="Q11" pad="4"/>
+<wire x1="-84.77" y1="-546.1" x2="-100.625" y2="-578.28" width="0" layer="19" extent="1-1"/>
 <wire x1="-83.82" y1="-532.3" x2="-84.77" y2="-546.1" width="0" layer="19" extent="1-1"/>
-<wire x1="26.24" y1="-3.515" x2="-83.82" y2="-532.3" width="0" layer="19" extent="1-1"/>
+<wire x1="-82.845" y1="-524.94" x2="-83.82" y2="-532.3" width="0" layer="19" extent="1-1"/>
+<wire x1="26.24" y1="-3.515" x2="-82.845" y2="-524.94" width="0" layer="19" extent="1-1"/>
 <wire x1="26.24" y1="-2.865" x2="26.24" y2="-3.515" width="0" layer="19" extent="1-1"/>
 <wire x1="26.24" y1="-2.215" x2="26.24" y2="-2.865" width="0" layer="19" extent="1-1"/>
 <wire x1="26.24" y1="-1.565" x2="26.24" y2="-2.215" width="0" layer="19" extent="1-1"/>
-</signal>
-<signal name="N$35">
-<contactref element="Q7" pad="4"/>
-<contactref element="R7" pad="2"/>
-<contactref element="Q9" pad="1"/>
-<wire x1="-84.77" y1="-534.5" x2="-82.87" y2="-553.72" width="0" layer="19" extent="1-1"/>
-<wire x1="-82.845" y1="-524.94" x2="-84.77" y2="-534.5" width="0" layer="19" extent="1-1"/>
 </signal>
 <signal name="GPIO17">
@@
 <wire x1="-72.685" y1="-469.06" x2="-93.98" y2="-575.48" width="0" layer="19" extent="1-1"/>
 </signal>
+<signal name="N$37">
+<contactref element="Q9" pad="1"/>
+<contactref element="Q11" pad="7"/>
+<contactref element="Q11" pad="5"/>
+<contactref element="Q11" pad="6"/>
+<contactref element="Q11" pad="8"/>
+<wire x1="-102.575" y1="-574.88" x2="-101.925" y2="-574.88" width="0" layer="19" extent="1-1"/>
+<wire x1="-101.275" y1="-574.88" x2="-101.925" y2="-574.88" width="0" layer="19" extent="1-1"/>
+<wire x1="-100.625" y1="-574.88" x2="-101.275" y2="-574.88" width="0" layer="19" extent="1-1"/>
+<wire x1="-84.77" y1="-534.5" x2="-100.625" y2="-574.88" width="0" layer="19" extent="1-1"/>
+</signal>
 </signals>

Commit message: dalsi_text_a_firstbot
Parts:
- removed C2: 10u, rcl_upravena:C1206
- removed Q11: (no value), transistors:MLP3.3X3.3_HS
- removed R15, R3: 2M, rcl_upravena:R0805
- Q9: device transistors:SOT23 -> transistors:MLP3.3X3.3_HS
- moved Q7 63.7 mm to (-109.2, -581.7)
- moved Q9 53.8 mm to (-101.6, -584.2)
Connections:
- removed net N$37: Q11.5, Q11.6, Q11.7, Q11.8, Q9.1
- new net ESP_SHUTDOWN: Q6.1, R16.2, SW5.3, SW5.4
- net BAT_POL+: now also Q7.4
- net GND: no longer C2.2, Q11.1, Q11.2, Q11.3, R15.2, R3.2
- net N$7: now also Q9.5, Q9.6, Q9.7, Q9.8; no longer Q11.4, Q7.4, Q9.3, R3.1
- net N$9: now also Q7.1, Q7.2, Q7.3, Q9.1, Q9.2, Q9.3; no longer C2.1, Q6.1, R15.1, R16.2, SW5.3, SW5.4
- net START_GATE1: now also Q9.4
- net VCC: no longer Q7.1, Q7.2, Q7.3, Q9.2
