File: ele/Blackbox/main_board/main_board 1.0.0/board.sch (EAGLE design)
At the start: 205 parts, among them IC1 DS3231/SO, IC2 QMC5883L-TR, Q2 AO3401ASOP-8_EP_5.0X5.0X1.27P, Q3 AO3401ASOP-8_EP_5.0X5.0X1.27P, Q4 BSS84, Q8 AO3401ASOP-8_EP_5.0X5.0X1.27P, Q9 AO3401ASOP-8_EP_5.0X5.0X1.27P, U1 MPU-6050

Commit message: trochu v tom delam bordel
proste to neumim delat poredne tak tet delam tenhle bordel commit bych mel vse na gitu a budu se snazit to dal delat poradne
Changed lines of the file:
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@@
 <instance part="Q1" gate="G$1" x="38.1" y="38.1" smashed="yes" rot="R270">
 <attribute name="VALUE" x="38.1" y="49.53" size="1.778" layer="96" rot="R270"/>
-<attribute name="NAME" x="35.56" y="31.75" size="1.778" layer="95" rot="R270"/>
+<attribute name="NAME" x="36.576" y="39.37" size="1.778" layer="95"/>
 </instance>
 <instance part="R8" gate="G$1" x="27.94" y="43.18" smashed="yes" rot="R270">
