File: ele/Blackbox/motor_board/untitled.sch (EAGLE design)
At the start: 93 parts, among them IC1 ATXMEGA16A4U-AU, X1 SMKDSP_1,5/2, X2 SMKDSP_1,5/2, X4 POWER_IN

Commit message: 2.KSK
Parts:
- removed C1, C5: 0.022uf, rcl:C-EUC0603
- removed C2, C6: (no value), rcl:C-EUC0603
- removed C3, C7: (no value), rcl:CPOL-EUE5-10.5
- removed C4, C8: (no value), rcl:C-EUC1206
- removed U$1, U$2: DRV8876, texas_instrument:DRV8876
- removed U$3: LM1086TO263, v-reg-2:LM1086TO263
- removed X2: SMKDSP_1,5/2, con-phoenix-smkdsp:SMKDSP_1,5/2
- removed X4: POWER_IN, con-wago-508:W237-02P
- added C13: (no value), rcl:C-EUC0603
- added C14: (no value), rcl:CPOL-EUD
- added C15, C16: (no value), rcl:CPOL-EUE5-10.5
- added C17, C21: 47nf - 200v, rcl:C-EUC0603
- added C18, C22: 1uf - 200v, rcl:C-EUC1206
- added C19, C23: 1uf, rcl:C-EUC1206
- added C20, C24: 47nf, rcl:C-EUC1206
- added IC2: PQ20WZ, v-reg-2:PQ20WZ
- added JP3, JP4: (no value), pinhead:PINHD-1X2
- added L1: (no value), rcl:L-EUL3216C
- added Q1: (no value), transistors:N-MOSFET-SOT23-GSD
- added R36, R37, R38, R39, R42, R43, R44, R45, R46, R47: (no value), rcl:R-EU_R0603
- added R40: 130k, rcl_upravena:R-EU_R0805
- added R41: 100k, rcl_upravena:R-EU_R0805
- added U$4: MC33063/MC34063D, adafruit:MC33063/MC34063D
- added U$55, U$58: DER8873, texas_instrument:DER8873
- added X0: POWER_IN, con-wago-508:W237-02P
- added X3: SMKDSP_1,5/2, con-phoenix-smkdsp:SMKDSP_1,5/2
- Q2, Q5: device transistors:P-MOSFET-TO220V -> transistors:P-MOSFET-MLP_HS
Connections:
- removed net +3V3: C10.1, C11.1, C12.1, IC1.AVCC, IC1.VCC@1, IC1.VCC@2, IC1.VCC@3, ISL1.VCC, ISL10.VCC, ISL11.VCC, ISL12.VCC, ISL13.VCC, ISL14.VCC, ISL15.VCC, ISL16.VCC, ISL2.VCC, ISL3.VCC, ISL4.VCC, ISL5.VCC, ISL6.VCC, ISL7.VCC, ISL8.VCC, ISL9.VCC, JP1.2, JP2.1, R1.2, R10.2, R11.2, R12.2, R13.2, R14.2, R15.2, R16.2, R17.2, R18.2, R19.2, R20.2, R21.2, R22.2, R23.2, R24.2, R25.2, R26.2, R27.2, R28.2, R29.2, R30.2, R31.2, R32.2, R33.2, R34.2, R35.2, R5.2, R6.2, R7.2, R8.2, R9.2, U$1.VREF, U$2.VREF, U$3.OUT
- removed net 0-INA: U$1.PH/IN1
- removed net 0-INB: U$1.EN/IN2
- removed net 0-NFAULT: U$1.NFAULT
- removed net 0-NSLEEP: U$1.NSLEEP
- removed net 1-INA: U$2.PH/IN1
- removed net 1-INB: U$2.EN/IN2
- removed net 1-NFAULT: U$2.NFAULT
- removed net 1-NSLEEP: U$2.NSLEEP
- removed net 1-OUTA: U$2.OUT1, X2-1.KL
- removed net 1-OUTB: U$2.OUT2, X2-2.KL
- removed net N$1: C1.1, U$1.CPH
- removed net N$2: C1.2, U$1.CPL
- removed net N$3: C2.1, U$1.VCP
- removed net N$4: U$1.GND, U$1.IMODE, U$1.PGND, U$1.PMODE, U$2.GND, U$2.IMODE, U$2.PGND, U$2.PMODE
- removed net N$5: C5.1, U$2.CPH
- removed net N$6: C5.2, U$2.CPL
- removed net N$7: C6.1, U$2.VCP
- new net +2V8: C10.1, C11.1, C12.1, C16.+, C20.1, C24.1, IC1.AVCC, IC1.VCC@1, IC1.VCC@2, IC1.VCC@3, ISL1.VCC, ISL10.VCC, ISL11.VCC, ISL12.VCC, ISL13.VCC, ISL14.VCC, ISL15.VCC, ISL16.VCC, ISL2.VCC, ISL3.VCC, ISL4.VCC, ISL5.VCC, ISL6.VCC, ISL7.VCC, ISL8.VCC, ISL9.VCC, JP1.2, JP2.1, R1.2, R10.2, R11.2, R12.2, R13.2, R14.2, R15.2, R16.2, R17.2, R18.2, R19.2, R20.2, R21.2, R22.2, R23.2, R24.2, R25.2, R26.2, R27.2, R28.2, R29.2, R30.2, R31.2, R32.2, R33.2, R34.2, R35.2, R40.1, R44.2, R47.2, R5.2, R6.2, R7.2, R8.2, R9.2, U$55.DVDD, U$58.DVDD
- new net +5V: C14.+, C15.+, IC2.VC, IC2.VIN, L1.2, R39.1
- new net 0-OUTA1: U$58.OUT-B, X3-1.KL
- new net 0-OUTB1: U$58.OUT-A, X3-2.KL
- new net DISAMLE-0: U$55.DISABLE
- new net DISAMLE-1: U$58.DISABLE
- new net INA-0: U$55.IN-A
- new net INA-1: U$58.IN-A
- new net INB-0: U$55.IN-B
- new net INB-1: U$58.IN-B
- new net IPROBI-0A: R43.2, U$55.IPROPI-A
- new net IPROBI-1A: R46.2, U$58.IPROPI-A
- new net IPROPI-0B: R42.2, U$55.IPROPI-B
- new net IPROPI-1B: R45.2, U$58.IPROPI-B
- new net N$26: IC2.VADJ, R40.2, R41.1
- new net N$27: Q1.D, R37.2, U$4.DC, U$4.IPK, U$4.SWC
- new net N$28: IC2.VO, IC2.VO-3
- new net N$29: R38.2, R39.2, U$4.COMP
- new net N$30: C17.1, U$55.CPH
- new net N$31: C17.2, U$55.CPL
- new net N$32: C19.2, U$55.VCP
- new net N$33: C13.1, U$4.TC
- new net N$34: C21.1, U$58.CPH
- new net N$35: C21.2, U$58.CPL
- new net N$36: C23.2, U$58.VCP
- new net N$38: L1.1, Q1.S
- new net NFAUL-0: R44.1, U$55.FAOU
- new net NFAUL-1: R47.1, U$58.FAOU
- new net NSLEEP-0: U$55.NSLEEP
- new net NSLEEP-1: U$58.NSLEEP
- new net SCLK: IC1.EVOUT/SCK/TXD1/PC7, U$55.SCLK, U$58.SCLK
- new net SCS-0: IC1.~SS/OC1A/PC4, U$55.SCS
- new net SCS-1: IC1.TXD0/OC0D/PC3, U$58.SCS
- new net SDI: IC1.MOSI/XCK1/OC1B/PC5, U$55.SDI, U$58.SDI
- new net SDO: IC1.MISO/RXD1/PC6, U$55.SDO, U$58.SDO
- net 0-IPROPI: no longer U$1.IPROPI
- net 0-OUTA: now also U$55.OUT-B; no longer U$1.OUT1
- net 0-OUTB: now also U$55.OUT-A; no longer U$1.OUT2
- net 1-IPROPI: no longer U$2.IPROPI
- net BAT1: now also X0-2.KL; no longer X4-2.KL
- net GND: now also C13.2, C14.-, C15.-, C16.-, C18.2, C20.2, C22.2, C24.2, IC2.GND, JP3.2, JP4.2, R36.1, R38.1, R41.2, R42.1, R43.1, R45.1, R46.1, U$4.GND, U$55.GND, U$58.GND, X0-1.KL; no longer C3.-, C4.2, C7.-, C8.2, U$3.GND, X4-1.KL
- net N$9: now also Q1.G, R36.2, U$4.SWE; no longer U$3.IN
- net OFF: now also JP4.1
- net ON: now also JP3.1
- net VCC: now also C18.1, C19.1, C22.1, C23.1, R37.1, U$4.VCC, U$55.VM, U$58.VM; no longer C2.2, C3.+, C4.1, C6.2, C7.+, C8.1, U$1.VMOT, U$2.VMOT

Commit message: ladeni_drah
Parts:
- added C69, C70: 10uf, rcl:C-EUC0402K
- added JP5: (no value), pinhead:PINHD-1X4
- added MAX1: MAX485, maxim:MAX485
- added Q10: (no value), transistors:N-MOSFET-SOT23-GSD
- added R48: 120, rcl:R-EU_R0402
- added R49, R50: 20k, rcl:R-EU_R0402
- added R51: 10k, rcl:R-EU_R0402
- added R52: 100k, rcl:R-EU_R0402
- added SJ1: (no value), jumper:SJ
Connections:
- new net +3V3: Q10.G, R51.2
- new net A: JP5.2, MAX1.A, R48.2, R50.1
- new net B: JP5.3, MAX1.B, R49.1, SJ1.2
- new net MODE_485: MAX1.DE, MAX1.RE/, R52.1
- new net N$1: R48.1, SJ1.1
- new net RX-485-5V: MAX1.RO, Q10.D
- new net RX_485: Q10.S, R51.1
- new net TX_485: MAX1.DI
- net +5V: now also C69.1, C70.1, JP5.4, MAX1.VCC, R49.2
- net GND: now also C69.2, C70.2, JP5.1, MAX1.GND, R50.2, R52.2

Commit message: dokumentace ke SchoolBoardu
Connections:
- removed net 0-IPROPI: IC1.AREF/ADC0/AC0/PA0
- removed net 1-IPROPI: IC1.ADC1/AC1/PA1
- removed net IPROBI-0A: R43.2, U$55.IPROPI-A
- removed net IPROBI-1A: R46.2, U$58.IPROPI-A
- new net IPROPI-0A: IC1.AREF/ADC0/AC0/PA0, R43.2, U$55.IPROPI-A
- new net IPROPI-1A: IC1.ADC2/AC2/PA2, R46.2, U$58.IPROPI-A
- net IPROPI-0B: now also IC1.ADC1/AC1/PA1
- net IPROPI-1B: now also IC1.ADC3/AC3/PA3
Other:
- moved on the sheet: C17, C18, C19, C20, C21, C22, C23, R42, R43, R44, R45, R46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

Commit message: dalsi_text_a_firstbot
Parts:
- removed ISL1, ISL10, ISL11, ISL12, ISL13, ISL14, ISL15, ISL16, ISL2, ISL3, ISL4, ISL5, ISL6, ISL7, ISL8, ISL9: ISL29035, renesas:ISL29035
- removed LED1, LED10, LED11, LED12, LED13, LED14, LED15, LED16, LED2, LED3, LED4, LED5, LED6, LED7, LED8, LED9: (no value), led:LEDCHIP-LED0603
- removed R1, R10, R12, R14, R16, R18, R20, R22, R24, R26, R28, R30, R32, R34, R6, R8: 4k7, rcl:R-EU_R0402
- removed R11, R13, R15, R17, R19, R21, R23, R25, R27, R29, R31, R33, R35, R5, R7, R9: 180, rcl:R-EU_R0402
- added CH1: CH340C, ch340g:CH340C
- added X2: USB-MICRO-B-BOTTOM, usb:USB-MICRO-B-BOTTOM
Connections:
- removed net !INT: ISL1.!INT, ISL10.!INT, ISL11.!INT, ISL12.!INT, ISL13.!INT, ISL14.!INT, ISL15.!INT, ISL16.!INT, ISL2.!INT, ISL3.!INT, ISL4.!INT, ISL5.!INT, ISL6.!INT, ISL7.!INT, ISL8.!INT, ISL9.!INT, R1.1, R10.1, R12.1, R14.1, R16.1, R18.1, R20.1, R22.1, R24.1, R26.1, R28.1, R30.1, R32.1, R34.1, R6.1, R8.1
- removed net N$10: LED1.A, R5.1
- removed net N$11: LED2.A, R7.1
- removed net N$12: LED3.A, R9.1
- removed net N$13: LED4.A, R11.1
- removed net N$14: LED5.A, R13.1
- removed net N$15: LED6.A, R15.1
- removed net N$16: LED7.A, R17.1
- removed net N$17: LED8.A, R19.1
- removed net N$18: LED9.A, R21.1
- removed net N$19: LED10.A, R23.1
- removed net N$20: LED11.A, R25.1
- removed net N$21: LED12.A, R27.1
- removed net N$22: LED13.A, R29.1
- removed net N$23: LED14.A, R31.1
- removed net N$24: LED15.A, R33.1
- removed net N$25: LED16.A, R35.1
- removed net SCL: ISL1.SCL, ISL10.SCL, ISL11.SCL, ISL12.SCL, ISL13.SCL, ISL14.SCL, ISL15.SCL, ISL16.SCL, ISL2.SCL, ISL3.SCL, ISL4.SCL, ISL5.SCL, ISL6.SCL, ISL7.SCL, ISL8.SCL, ISL9.SCL
- removed net SDA: ISL1.SDA, ISL10.SDA, ISL11.SDA, ISL12.SDA, ISL13.SDA, ISL14.SDA, ISL15.SDA, ISL16.SDA, ISL2.SDA, ISL3.SDA, ISL4.SDA, ISL5.SDA, ISL6.SDA, ISL7.SDA, ISL8.SDA, ISL9.SDA
- new net D+: CH1.D+, X2.D+
- new net D-: CH1.D-, X2.D-
- new net RXD0: CH1.RX, IC1.RXD0/OC0C/PE2
- new net TXD0: CH1.TX, IC1.TXD0/OC0D/PE3
- new net VBUS: CH1.VCC, X2.VBUS
- net !RESET: now also CH1.RTS
- net +2V8: now also CH1.V3; no longer ISL1.VCC, ISL10.VCC, ISL11.VCC, ISL12.VCC, ISL13.VCC, ISL14.VCC, ISL15.VCC, ISL16.VCC, ISL2.VCC, ISL3.VCC, ISL4.VCC, ISL5.VCC, ISL6.VCC, ISL7.VCC, ISL8.VCC, ISL9.VCC, R1.2, R10.2, R11.2, R12.2, R13.2, R14.2, R15.2, R16.2, R17.2, R18.2, R19.2, R20.2, R21.2, R22.2, R23.2, R24.2, R25.2, R26.2, R27.2, R28.2, R29.2, R30.2, R31.2, R32.2, R33.2, R34.2, R35.2, R5.2, R6.2, R7.2, R8.2, R9.2
- net GND: now also CH1.GND, X2.GND; no longer ISL1.GND, ISL10.GND, ISL11.GND, ISL12.GND, ISL13.GND, ISL14.GND, ISL15.GND, ISL16.GND, ISL2.GND, ISL3.GND, ISL4.GND, ISL5.GND, ISL6.GND, ISL7.GND, ISL8.GND, ISL9.GND, LED1.C, LED10.C, LED11.C, LED12.C, LED13.C, LED14.C, LED15.C, LED16.C, LED2.C, LED3.C, LED4.C, LED5.C, LED6.C, LED7.C, LED8.C, LED9.C

Commit message: trochu v tom delam bordel
proste to neumim delat poredne tak tet delam tenhle bordel commit bych mel vse na gitu a budu se snazit to dal delat poradne
Parts:
- removed C18, C22: 1uf - 200v, rcl:C-EUC1206
- removed C19, C23: 1uf, rcl:C-EUC1206
- removed C21: 47nf - 200v, rcl:C-EUC0603
- removed C24: 47nf, rcl:C-EUC1206
- removed CH1: CH340C, ch340g:CH340C
- removed IC2: PQ20WZ, v-reg-2:PQ20WZ
- removed L1: (no value), rcl:L-EUL3216C
- removed Q1, Q6: (no value), transistors:N-MOSFET-SOT23-GSD
- removed Q2, Q5: (no value), transistors:P-MOSFET-MLP_HS
- removed R2: 10k, rcl_upravena:R-EU_R0805
- removed R3, R41: 100k, rcl_upravena:R-EU_R0805
- removed R36, R37, R38, R39, R42, R43, R44, R45, R46, R47: (no value), rcl:R-EU_R0603
- removed R4: 2M, rcl_upravena:R-EU_M0805
- removed R40: 130k, rcl_upravena:R-EU_R0805
- removed SW4, SW5: (no value), switch-omron:10-XX
- removed U$4: MC33063/MC34063D, adafruit:MC33063/MC34063D
- removed U$55, U$58: DER8873, texas_instrument:DER8873
- removed X0: POWER_IN, con-wago-508:W237-02P
- removed X1, X3: SMKDSP_1,5/2, con-phoenix-smkdsp:SMKDSP_1,5/2
- added C1, C2, C3, C4, C5, C6, C7, C8: (no value), rcl:C-EUC0402
- added C27, C31: 47nf - 200v, rcl:C-EUC0603
- added C28, C32: 1uf - 200v, rcl:C-EUC1206
- added C29, C33: 1uf, rcl:C-EUC1206
- added C30, C34: 47nf, rcl:C-EUC1206
- added C35, C36: 10uf, rcl:C-EUC0805
- added C37: 10u, rcl_upravena:C-EUC1206
- added C38, C39: (no value), rcl:CPOL-EUE5-10.5
- added CH2: CH340C, ch340g:CH340C
- added IC3: ATXMEGA128A1U-AU, xmega:ATXMEGA128A1U-AU
- added JP10, JP11, JP12, JP13, JP14, JP15, JP16, JP17: (no value), pinhead:PINHD-1X25
- added JP6: (no value), pinhead:PINHD-1X4
- added JP7, JP8: (no value), pinhead:PINHD-1X2
- added JP9: (no value), pinhead:PINHD-2X25
- added L2: (no value), rcl:L-EUL3216C
- added Q3, Q4: (no value), transistors:P-MOSFET-MLP_HS
- added Q7, Q8: (no value), transistors:N-MOSFET-SOT23-GSD
- added R1: 10k, rcl_upravena:R-EU_R0805
- added R10, R11, R12, R13, R14, R15, R16, R7, R8, R9: (no value), rcl:R-EU_R0603
- added R17, R6: 2M, rcl_upravena:R-EU_M0805
- added R5: 100k, rcl_upravena:R-EU_R0805
- added SW1, SW2: (no value), switch-omron:10-XX
- added U$1: MC33063/MC34063D, adafruit:MC33063/MC34063D
- added U$2, U$6: DER8873, texas_instrument:DER8873
- added U$3: TMC2224, TRINAMIC:TMC2224
- added X4: USB-MICRO-B-BOTTOM, usb:USB-MICRO-B-BOTTOM
- added X5, X6: SMKDSP_1,5/2, con-phoenix-smkdsp:SMKDSP_1,5/2
- C11: device rcl:C-EUC0402 -> rcl:C-EUC0603
- C12: value (none) -> 10u; device rcl:C-EUC0402 -> rcl_upravena:C-EUC1206
- C13: value (none) -> 100nf - 15v; device rcl:C-EUC0603 -> rcl:C-EUC1206
- C14: value (none) -> 1uf - 200v; device rcl:CPOL-EUD -> rcl:C-EUC1206
- C15: value (none) -> 22nf - 50v; device rcl:CPOL-EUE5-10.5 -> rcl:C-EUC1206
- C16: value (none) -> 1uf - 200v - T; device rcl:CPOL-EUE5-10.5 -> rcl:C-EUC1206
- C17: value 47nf - 200v -> 100uf - 200v; device rcl:C-EUC0603 -> rcl:CPOL-EUE5-10.5
- C20: value 47nf -> (none); device rcl:C-EUC1206 -> rcl:CPOL-EUD
- C9: value 10u -> (none); device rcl_upravena:C-EUC1206 -> rcl:C-EUC0402
- IC1: value ATXMEGA16A4U-AU -> (none); device xmega:ATXMEGA16A4U-AU -> v-reg-2:LM1117
- JP1: device pinhead:PINHD-1X4 -> jumper:JP2E
- JP2: device jumper:JP2E -> pinhead:PINHD-2X25
- JP3, JP4: device pinhead:PINHD-1X2 -> pinhead:PINHD-2X25
- X2: value USB-MICRO-B-BOTTOM -> POWER_IN; device usb:USB-MICRO-B-BOTTOM -> con-wago-508:W237-02P
Connections:
- removed net +2V8: C10.1, C11.1, C12.1, C16.+, C20.1, C24.1, CH1.V3, IC1.AVCC, IC1.VCC@1, IC1.VCC@2, IC1.VCC@3, JP1.2, JP2.1, R40.1, R44.2, R47.2, U$55.DVDD, U$58.DVDD
- removed net 0-OUTA: U$55.OUT-B, X1-1.KL
- removed net 0-OUTA1: U$58.OUT-B, X3-1.KL
- removed net 0-OUTB: U$55.OUT-A, X1-2.KL
- removed net 0-OUTB1: U$58.OUT-A, X3-2.KL
- removed net N$26: IC2.VADJ, R40.2, R41.1
- removed net N$27: Q1.D, R37.2, U$4.DC, U$4.IPK, U$4.SWC
- removed net N$28: IC2.VO, IC2.VO-3
- removed net N$29: R38.2, R39.2, U$4.COMP
- removed net N$30: C17.1, U$55.CPH
- removed net N$31: C17.2, U$55.CPL
- removed net N$32: C19.2, U$55.VCP
- removed net N$33: C13.1, U$4.TC
- removed net N$34: C21.1, U$58.CPH
- removed net N$35: C21.2, U$58.CPL
- removed net N$36: C23.2, U$58.VCP
- removed net N$38: L1.1, Q1.S
- removed net PDI: IC1.PDI, JP1.4
- removed net SCS-0: IC1.~SS/OC1A/PC4, U$55.SCS
- removed net SCS-1: IC1.TXD0/OC0D/PC3, U$58.SCS
- removed net SDI: IC1.MOSI/XCK1/OC1B/PC5, U$55.SDI, U$58.SDI
- removed net SDO: IC1.MISO/RXD1/PC6, U$55.SDO, U$58.SDO
- removed net VBUS: CH1.VCC, X2.VBUS
- new net 0-OUTA2: U$2.OUT-B, X5-1.KL
- new net 0-OUTA3: U$6.OUT-B, X6-1.KL
- new net 0-OUTB2: U$2.OUT-A, X5-2.KL
- new net 0-OUTB3: U$6.OUT-A, X6-2.KL
- new net LED0: IC3.PH0
- new net LED1: IC3.PH1
- new net LED2: IC3.PH2
- new net LED3: IC3.PH3
- new net MISO: IC3.PC6, JP10.21, JP14.21, U$2.SDO, U$6.SDO
- new net MOSI: IC3.PC5, JP10.20, JP14.20, U$2.SDI, U$6.SDI
- new net N$10: C27.1, U$2.CPH
- new net N$11: C27.2, U$2.CPL
- new net N$12: C29.2, U$2.VCP
- new net N$13: C31.1, U$6.CPH
- new net N$14: C31.2, U$6.CPL
- new net N$15: C33.2, U$6.VCP
- new net N$16: C15.1, U$3.CPO
- new net N$17: C15.2, U$3.CPI
- new net N$18: U$3.VCC_IN
- new net N$2: JP1.2, R1.1
- new net N$3: Q8.D, R8.2, U$1.DC, U$1.IPK, U$1.SWC
- new net N$4: R10.2, R9.2, U$1.COMP
- new net N$5: C11.1, U$1.TC
- new net N$6: L2.1, Q8.S
- new net N$7: Q8.G, R7.2, U$1.SWE
- new net PA2: IC3.PA2, JP13.22, JP17.22
- new net PA3: IC3.PA3, JP13.23, JP17.23
- new net PA4: IC3.PA4, JP13.24, JP17.24
- new net PA5: IC3.PA5, JP13.25, JP17.25
- new net PA6: IC3.PA6, JP10.1, JP14.1
- new net PA7: IC3.PA7, JP10.2, JP14.2
- new net PB2: IC3.PB2, JP10.7, JP14.7
- new net PB3: IC3.PB3, JP10.8, JP14.8
- new net PB4: IC3.PB4, JP10.9, JP14.9
- new net PB5: IC3.PB5, JP10.10, JP14.10
- new net PB6: IC3.PB6, JP10.11, JP14.11
- new net PB7: IC3.PB7, JP10.12, JP14.12
- new net PC0: IC3.PC0, JP10.15, JP14.15
- new net PC1: IC3.PC1, JP10.16, JP14.16
- new net PC2: IC3.PC2, JP10.17, JP14.17
- new net PDI_DATA: IC3.PDI_DATA, JP13.14, JP17.14, JP6.4
- new net PE0: IC3.PE0, JP11.10, JP15.10
- new net PE1: IC3.PE1, JP11.11, JP15.11
- new net PE2: IC3.PE2, JP11.12, JP15.12
- new net PE3: IC3.PE3, JP11.13, JP15.13
- new net PE4: IC3.PE4, JP11.14, JP15.14
- new net PE5: JP11.15, JP15.15
- new net PF0: IC3.PF0, JP11.20, JP15.20
- new net PF1: IC3.PF1, JP11.21, JP15.21
- new net PF2: IC3.PF2, JP11.22, JP15.22
- new net PF3: IC3.PF3, JP11.23, JP15.23
- new net PF4: IC3.PF4, JP11.24, JP15.24
- new net PF5: IC3.PF5, JP11.25, JP15.25
- new net PH0: JP12.5, JP16.5
- new net PH1: JP12.6, JP16.6
- new net PH2: JP12.7, JP16.7
- new net PH3: JP12.8, JP16.8
- new net PH4: JP12.9, JP16.9
- new net PH5: JP12.10, JP16.10
- new net PH6: JP12.11, JP16.11
- new net PH7: JP12.12, JP16.12
- new net PJ0: IC3.PJ0, JP12.15, JP16.15
- new net PJ1: IC3.PJ1, JP12.16, JP16.16
- new net PJ2: IC3.PJ2, JP12.17, JP16.17
- new net PJ3: IC3.PJ3, JP12.18, JP16.18
- new net PJ4: IC3.PJ4, JP12.19, JP16.19
- new net PJ5: IC3.PJ5, JP12.20, JP16.20
- new net PJ6: IC3.PJ6, JP12.21, JP16.21
- new net PJ7: JP12.22, JP16.22
- new net PK0: IC3.PK0, JP12.25, JP16.25
- new net PK1: IC3.PK1, JP13.1, JP17.1
- new net PK2: IC3.PK2, JP13.2, JP17.2
- new net PK3: IC3.PK3, JP13.3, JP17.3
- new net PK4: IC3.PK4, JP13.4, JP17.4
- new net PK5: IC3.PK5, JP13.5, JP17.5
- new net PK6: IC3.PK6, JP13.6, JP17.6
- new net PK7: IC3.PK7, JP13.7, JP17.7
- new net PQ0: IC3.PQ0, JP13.10, JP17.10
- new net PQ1: IC3.PQ1, JP13.11, JP17.11
- new net PQ2: IC3.PQ2, JP13.12, JP17.12
- new net PQ3: IC3.PQ3, JP13.13, JP17.13
- new net PR0: IC3.PR0, JP13.16, JP17.16
- new net PR1: IC3.PR1, JP13.17, JP17.17
- new net RESET: JP6.3
- new net RX: IC3.PF6, JP12.1, JP16.1
- new net SCK: IC3.PC7, JP10.22, JP14.22
- new net SS-0: IC3.PC3, JP10.18, JP14.18, U$2.SCS
- new net SS-1: IC3.PC4, JP10.19, JP14.19, U$6.SCS
- new net SW0: IC3.PH7
- new net SW1: IC3.PH6
- new net SW2: IC3.PH5
- new net SW3: IC3.PH4
- new net TX: IC3.PF7, JP12.2, JP16.2
- net !RESET: now also CH2.RTS, IC3.RESET, JP13.15, JP17.15; no longer CH1.RTS, IC1.!RESET, JP1.1
- net +3V3: now also C1.1, C10.1, C2.1, C3.1, C30.1, C34.1, C36.1, C4.1, C5.1, C6.1, C7.1, C8.1, C9.1, CH2.V3, IC1.OUT, IC3.AVCC, IC3.VCC, JP1.1, JP10.14, JP10.24, JP10.4, JP11.19, JP11.9, JP12.14, JP12.24, JP12.4, JP13.19, JP13.9, JP14.14, JP14.24, JP14.4, JP15.19, JP15.9, JP16.14, JP16.24, JP16.4, JP17.19, JP17.9, JP2.10, JP2.12, JP2.14, JP2.16, JP2.18, JP2.2, JP2.20, JP2.22, JP2.24, JP2.26, JP2.28, JP2.30, JP2.32, JP2.34, JP2.36, JP2.38, JP2.4, JP2.40, JP2.42, JP2.44, JP2.46, JP2.48, JP2.50, JP2.6, JP2.8, JP3.10, JP3.12, JP3.14, JP3.16, JP3.18, JP3.2, JP3.20, JP3.22, JP3.24, JP3.26, JP3.28, JP3.30, JP3.32, JP3.34, JP3.36, JP3.38, JP3.4, JP3.40, JP3.42, JP3.44, JP3.46, JP3.48, JP3.50, JP3.6, JP3.8, JP4.10, JP4.12, JP4.14, JP4.16, JP4.18, JP4.2, JP4.20, JP4.22, JP4.24, JP4.26, JP4.28, JP4.30, JP4.32, JP4.34, JP4.36, JP4.38, JP4.4, JP4.40, JP4.42, JP4.44, JP4.46, JP4.48, JP4.50, JP4.6, JP4.8, JP6.1, JP9.10, JP9.12, JP9.14, JP9.16, JP9.18, JP9.2, JP9.20, JP9.22, JP9.24, JP9.26, JP9.28, JP9.30, JP9.32, JP9.34, JP9.36, JP9.38, JP9.4, JP9.40, JP9.42, JP9.44, JP9.46, JP9.48, JP9.50, JP9.6, JP9.8, R13.2, R16.2, U$2.DVDD, U$6.DVDD
- net +5V: now also C20.+, C35.1, CH2.VCC, IC1.IN, L2.2, R10.1, X4.VBUS; no longer C14.+, C15.+, IC2.VC, IC2.VIN, L1.2, R39.1
- net BAT1: now also Q4.D, X2-2.KL; no longer Q5.D, X0-2.KL
- net BAT_POL+: now also Q3.S, Q4.S, R5.1; no longer Q2.S, Q5.S, R3.1
- net D+: now also CH2.D+, X4.D+; no longer CH1.D+, X2.D+
- net D-: now also CH2.D-, X4.D-; no longer CH1.D-, X2.D-
- net DISAMLE-0: now also U$2.DISABLE; no longer U$55.DISABLE
- net DISAMLE-1: now also U$6.DISABLE; no longer U$58.DISABLE
- net GND: now also C1.2, C14.2, C16.2, C17.-, C2.2, C20.-, C28.2, C3.2, C30.2, C32.2, C34.2, C35.2, C36.2, C37.1, C38.-, C39.-, C4.2, C5.2, C6.2, C7.2, C8.2, C9.2, CH2.GND, IC1.GND, IC3.AGND, IC3.GND, JP10.13, JP10.23, JP10.3, JP11.18, JP11.8, JP12.13, JP12.23, JP12.3, JP13.18, JP13.8, JP14.13, JP14.23, JP14.3, JP15.18, JP15.8, JP16.13, JP16.23, JP16.3, JP17.18, JP17.8, JP2.1, JP2.11, JP2.13, JP2.15, JP2.17, JP2.19, JP2.21, JP2.23, JP2.25, JP2.27, JP2.29, JP2.3, JP2.31, JP2.33, JP2.35, JP2.37, JP2.39, JP2.41, JP2.43, JP2.45, JP2.47, JP2.49, JP2.5, JP2.7, JP2.9, JP3.1, JP3.11, JP3.13, JP3.15, JP3.17, JP3.19, JP3.21, JP3.23, JP3.25, JP3.27, JP3.29, JP3.3, JP3.31, JP3.33, JP3.35, JP3.37, JP3.39, JP3.41, JP3.43, JP3.45, JP3.47, JP3.49, JP3.5, JP3.7, JP3.9, JP4.1, JP4.11, JP4.13, JP4.15, JP4.17, JP4.19, JP4.21, JP4.23, JP4.25, JP4.27, JP4.29, JP4.3, JP4.31, JP4.33, JP4.35, JP4.37, JP4.39, JP4.41, JP4.43, JP4.45, JP4.47, JP4.49, JP4.5, JP4.7, JP4.9, JP6.2, JP7.2, JP8.2, JP9.1, JP9.11, JP9.13, JP9.15, JP9.17, JP9.19, JP9.21, JP9.23, JP9.25, JP9.27, JP9.29, JP9.3, JP9.31, JP9.33, JP9.35, JP9.37, JP9.39, JP9.41, JP9.43, JP9.45, JP9.47, JP9.49, JP9.5, JP9.7, JP9.9, Q4.G, Q7.S, R11.1, R12.1, R14.1, R15.1, R17.2, R7.1, R9.1, SW1.S, SW1.S1, SW2.S, SW2.S1, U$1.GND, U$2.GND, U$3.GND, U$6.GND, X2-1.KL, X4.GND; no longer C12.2, C13.2, C14.-, C15.-, C16.-, C18.2, C20.2, C22.2, C24.2, CH1.GND, IC1.GND@1, IC1.GND@2, IC1.GND@3, IC1.GND@4, IC2.GND, JP1.3, JP3.2, JP4.2, Q5.G, Q6.S, R36.1, R38.1, R41.2, R42.1, R43.1, R45.1, R46.1, SW4.S, SW4.S1, SW5.S, SW5.S1, U$4.GND, U$55.GND, U$58.GND, X0-1.KL, X2.GND
- net INA-0: now also IC3.PD5, JP11.5, JP15.5, U$2.IN-A; no longer U$55.IN-A
- net INA-1: now also IC3.PD1, JP11.1, JP15.1, U$6.IN-A; no longer U$58.IN-A
- net INB-0: now also IC3.PD4, JP11.4, JP15.4, U$2.IN-B; no longer U$55.IN-B
- net INB-1: now also IC3.PD0, JP10.25, JP14.25, U$6.IN-B; no longer U$58.IN-B
- net IPROPI-0A: now also IC3.PA1, IC3.PB1, JP10.6, JP13.21, JP14.6, JP17.21, R12.2, U$2.IPROPI-A; no longer IC1.AREF/ADC0/AC0/PA0, R43.2, U$55.IPROPI-A
- net IPROPI-0B: now also IC3.PA0, IC3.PB0, JP10.5, JP13.20, JP14.5, JP17.20, R11.2, U$2.IPROPI-B; no longer IC1.ADC1/AC1/PA1, R42.2, U$55.IPROPI-B
- net IPROPI-1A: now also R15.2, U$6.IPROPI-A; no longer IC1.ADC2/AC2/PA2, R46.2, U$58.IPROPI-A
- net IPROPI-1B: now also R14.2, U$6.IPROPI-B; no longer IC1.ADC3/AC3/PA3, R45.2, U$58.IPROPI-B
- net MODE_485: now also IC3.PE5
- net N$8: now also C13.2, U$3.VCP; no longer JP2.2, R2.1
- net N$9: now also U$3.5VOUT; no longer Q1.G, R36.2, U$4.SWE
- net NFAUL-0: now also IC3.PD7, JP11.7, JP15.7, R13.1, U$2.FAOU; no longer R44.1, U$55.FAOU
- net NFAUL-1: now also IC3.PD3, JP11.3, JP15.3, R16.1, U$6.FAOU; no longer R47.1, U$58.FAOU
- net NSLEEP-0: now also IC3.PD6, JP11.6, JP15.6, U$2.NSLEEP; no longer U$55.NSLEEP
- net NSLEEP-1: now also IC3.PD2, JP11.2, JP15.2, U$6.NSLEEP; no longer U$58.NSLEEP
- net OFF: now also C37.2, IC3.PJ7, JP1.3, JP8.1, Q7.G, R1.2, R17.1, SW2.P, SW2.P1; no longer JP2.3, JP4.1, Q6.G, R2.2, SW5.P, SW5.P1
- net ON: now also C12.2, JP7.1, R6.2, SW1.P, SW1.P1; no longer C9.2, JP3.1, R4.2, SW4.P, SW4.P1
- net RXD0: now also CH2.TX; no longer CH1.RX, IC1.RXD0/OC0C/PE2
- net RX_485: now also IC3.PE6, JP11.16, JP15.16
- net SCLK: now also U$2.SCLK, U$6.SCLK; no longer IC1.EVOUT/SCK/TXD1/PC7, U$55.SCLK, U$58.SCLK
- net START_GATE1: now also C12.1, Q3.G, Q7.D, R5.2, R6.1; no longer C9.1, Q2.G, Q6.D, R3.2, R4.1
- net TXD0: now also CH2.RX; no longer CH1.TX, IC1.TXD0/OC0D/PE3
- net TX_485: now also IC3.PE7, JP11.17, JP15.17
- net VCC: now also C13.1, C14.1, C16.1, C17.+, C28.1, C29.1, C32.1, C33.1, C38.+, C39.+, Q3.D, R8.1, U$1.VCC, U$2.VM, U$3.VS, U$6.VM; no longer C18.1, C19.1, C22.1, C23.1, Q2.D, R37.1, U$4.VCC, U$55.VM, U$58.VM
Other:
- note added: "kondenzátory na vyhlazení napájení procesoru ke každému vstupu napájení jeden"
- note removed: "condenzátory k nohám procesoru ke každé napájecí noze jeden"
