File: ele/FirstBot/untitled.brd (EAGLE design)
At the start: 160 x 100 mm, 58 parts, among them T1 BC337, T2 BC337, U1 ESP-WROOM-32, X0 POWER_IN, X1 USB-MICRO-B-BOTTOM

Commit message: ESP32_wroom
CH340C
Parts:
- added C10: 1uf, rcl_upravena:C0402
- added C11, C12, C13: 1n 50V, rcl_upravena:C0402
- added R10, R9: 470, rcl_upravena:R0603
- added R6, R7: 5k, rcl_upravena:R0603
- added R8: 12k, rcl_upravena:R0603
- added SW7, SW8: TL3342F160QG/TR, Switch:TL3342F160QG/TR
- C2: value 100n -> 100nf
- CH1: value CH340G -> CH340C
Connections:
- net !DTR renamed DTR
- net !RTS renamed RTS
- removed net IO0_!RST: T2.3, U1.25
- new net CTS: CH1.9
- new net IO0: R10.1, R6.1, T2.3, U1.25
- new net N$7: C13.1, R10.2, SW7.1, SW7.2
- net +3V3: now also C10.2, R6.2, R8.2
- net EN: now also C11.2, R8.1, R9.1
- net GND: now also C10.1, C11.1, C12.2, C13.2, CH1.1, R7.1, SW7.3, SW7.4, SW8.3, SW8.4, X1.5
- net N$1: now also C12.1, R9.2, SW8.1, SW8.2; no longer CH1.1, X1.5
- net PWM_A1: now also R7.2

Commit message: dalsi_text_a_firstbot
Parts:
- removed LED5: BLUE, led:CHIPLED_1206
- removed SW5, SW6: (no value), switch-omron:B3F-10XX
- removed SW7, SW8: TL3342F160QG/TR, Switch:TL3342F160QG/TR
- added BOOT, EN, NO, OFF: TL3342F160QG/TR, Switch:TL3342F160QG/TR
- added C14: (no value), rcl:SANYO-OSCON_SMD_F8
- added D1: BAT60JDO-214-AB, diode:DO214BA
- added IC1: 7808DT, adafruit:TO252
- added JP5: (no value), pinhead:1X06
- added JP8, JP9: (no value), pinhead:1X03
- added LED0: BLUE, led:CHIPLED_1206
- added Q1: (no value), transistors:SOT23
- added R12: 4,7k, rcl:R0402
- C1, C3, C4, C5, C8, C9: device rcl_upravena:C1206 -> rcl_upravena:C0402K
- C10, C12, C2: device rcl_upravena:C0402 -> rcl_upravena:C0402K
- C23: device resistor:C0603 -> resistor:C0402K
- C7: device resistor:C0805 -> resistor:C0402K
- Q2, Q5: value (none) -> AO3401ASOP-8_EP_5.0X5.0X1.27P; device transistors:MLP3.3X3.3_HS -> transistor-fet:SOP-8_EP_5.0X5.0X1.27P
- R1, R5: value 10k -> 12k
- R10, R6, R7, R8, R9: device rcl_upravena:R0603 -> rcl_upravena:R0402
- R2: device rcl_upravena:R0805 -> rcl_upravena:R0603
- R23, R40, R43, R46, R49: value 10k -> 47k; device resistor:R0805 -> resistor:R0402
- R24, R38, R41, R44, R47: device resistor:R0805 -> resistor:R0402
- R29, R39, R42, R45, R48: value (none) -> 180; device resistor:R0805 -> resistor:R0402
- R3: device rcl_upravena:R0805 -> rcl_upravena:R0402
- R4: device rcl_upravena:M0805 -> rcl_upravena:R0402
- SW0, SW1, SW2, SW3, SW4: value (none) -> TL3342F160QG/TR; device switch-omron:B3F-10XX -> Switch:TL3342F160QG/TR
- moved R10 273.5 mm to (3.81, 38.1), turned to 180 degrees
- moved C13 261.5 mm to (3.81, 36.2)
- moved R6 239.1 mm to (17.8, 45.1)
- moved R9 238.2 mm to (3.81, 7.62), turned to 180 degrees
- moved X1 232.8 mm to (34.3, 47.0), turned to 270 degrees
- moved R7 230.2 mm to (22.9, 30.5), turned to 270 degrees
- moved C12 224.0 mm to (1.52, 3.81), turned to 270 degrees
- moved R8 223.8 mm to (4.32, 10.3), turned to 90 degrees
- moved C11 216.2 mm to (7.62, 7.62), turned to 180 degrees
- moved C10 213.6 mm to (3.17, 10.3), turned to 90 degrees
- moved R5 211.2 mm to (18.4, 37.3), turned to 90 degrees
- moved T2 209.6 mm to (15.9, 42.4)
- moved R1 208.0 mm to (18.4, 42.4), turned to 90 degrees
- moved T1 197.0 mm to (15.9, 37.3)
- moved CH1 192.2 mm to (24.1, 39.9), turned to 90 degrees
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Connections:
- net N$3 renamed D-
- net N$4 renamed D+
- net N$5 renamed VBUS
- removed net VCC: Q2.5, Q2.6, Q2.7, Q2.8
- new net N$11: D1.A, Q2.5, Q2.6, Q2.7, Q2.8, Q2.9
- new net N$2: JP5.1, U1.9
- new net N$3: JP5.2, U1.8
- new net N$4: JP5.3, U1.7
- new net N$5: JP5.4, U1.6
- new net N$6: JP5.5, U1.5
- new net N$9: JP5.6, U1.4
- new net SERVO: JP9.2, U1.37
- new net WS2812: Q1.2, U1.36
- new net WS2812-5V: JP8.2, Q1.3, R12.2
- net +3V3: now also CH1.4, IC1.2, Q1.1
- net +5V: now also C14.+, D1.C, IC1.1, JP8.1, JP9.1, R12.1
- net BAT1: now also Q5.9
- net ENC_A0: now also U1.10; no longer U1.12
- net ENC_A1: now also U1.13; no longer U1.10
- net ENC_B0: now also U1.11; no longer U1.13
- net ENC_B1: now also U1.12; no longer U1.11
- net GND: now also BOOT.3, BOOT.4, C14.-, EN.3, EN.4, IC1.3, JP8.3, JP9.3, LED0.C, NO.1, NO.2, OFF.1, OFF.2; no longer LED5.C, SW5.1, SW5.2, SW6.1, SW6.2, SW7.3, SW7.4, SW8.3, SW8.4
- net N$1: now also EN.1, EN.2; no longer SW8.1, SW8.2
- net N$10: now also LED0.A; no longer LED3.A
- net N$28: now also LED3.A; no longer LED5.A
- net N$7: now also BOOT.1, BOOT.2; no longer SW7.1, SW7.2
- net OFF: now also OFF.3, OFF.4; no longer SW5.3, SW5.4
- net ON: now also NO.3, NO.4; no longer SW4.3, SW4.4
- net PWM_B0: now also U1.27; no longer U1.26
- net PWM_B1: now also U1.26; no longer U1.27
- net SW3: now also SW3.3, SW3.4; no longer SW6.3, SW6.4
- net SW4: now also SW4.3, SW4.4; no longer SW3.3, SW3.4
Routing:
- net +3V3: track 0.00 -> 186.8 mm, vias 0 -> 8
- net +5V: track 0.00 -> 108.6 mm
- net ENC_B0: track 0.00 -> 101.9 mm, vias 0 -> 1
- net ENC_A0: track 0.00 -> 101.0 mm, vias 0 -> 1
- net FAUL: track 0.00 -> 85.5 mm, vias 0 -> 2
- net ENC_B1: track 0.00 -> 85.4 mm, vias 0 -> 1
- net WS2812: track 0.00 -> 84.5 mm, vias 0 -> 2
- net ENC_A1: track 0.00 -> 81.7 mm, vias 0 -> 1
- net PWM_A1: track 0.00 -> 76.3 mm, vias 0 -> 2
- net SERVO: track 0.00 -> 74.7 mm, vias 0 -> 1
- net SLEEP: track 0.00 -> 73.9 mm, vias 0 -> 2
- net PWM_A0: track 0.00 -> 73.7 mm, vias 0 -> 2
- net PWM_B1: track 0.00 -> 73.3 mm, vias 0 -> 2
- net PWM_B0: track 0.00 -> 72.8 mm, vias 0 -> 2
- net ON: track 0.00 -> 60.6 mm
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- added copper zone on layer 1, net BAT1
- added copper zone on layer 1, net BAT_POL+
- added copper zone on layer 1, net GND
- added copper zone on layer 16, net GND
- added copper zone on layer 1, net N$11
Other:
- board size 160 x 100 mm -> 94 x 47 mm

Commit message: trochu v tom delam bordel
proste to neumim delat poredne tak tet delam tenhle bordel commit bych mel vse na gitu a budu se snazit to dal delat poradne
Parts:
- removed Q5: AO3401ASOP-8_EP_5.0X5.0X1.27P, transistor-fet:SOP-8_EP_5.0X5.0X1.27P
- added C15, C17, C18: 10uf, rcl:C0603
- added C16: 0,1uf, rcl:C0402
- added C19: 10uf, resistor:C0402K
- added JP10, JP11, JP12: (no value), pinhead:1X06
- added R11: 4,7k, rcl:R0402
- added R13, R14, R15, R16, R17, R18: 180, resistor:R0402
- C10, C2: device rcl_upravena:C0402K -> rcl_upravena:C0402
- R2: device rcl_upravena:R0603 -> rcl_upravena:R0402
- U$9: value DRV8833HTSSOP -> DRV8833CPWPR; device texas-cc2541:HTSSOP -> DRV8833CPWPR:SOP65P640X120-17N
- moved JP5 51.8 mm to (54.6, 40.6)
- moved Q2 7.62 mm to (62.2, 21.6)
- moved R3 7.49 mm to (57.9, 18.4)
- moved D1 5.85 mm to (69.8, 21.6)
- moved R4 4.58 mm to (54.6, 15.2), turned to 270 degrees
- moved R2 4.16 mm to (57.1, 15.2), turned to 270 degrees
- moved C9 2.84 mm to (55.9, 15.2), turned to 270 degrees
- moved Q6 2.55 mm to (59.7, 15.9), turned to 0 degrees
- moved C7 1.52 mm to (79.9, 20.6), turned to 180 degrees
- moved C23 0.46 mm to (79.9, 22.6), turned to 180 degrees
Connections:
- removed net BAT_POL+: Q2.1, Q2.2, Q2.3, Q5.1, Q5.2, Q5.3, R3.1
- removed net N$25: C23.1, U$9.VCP
- new net N$12: C23.1, U$9.11
- new net N$13: JP10.6, JP5.6
- net +3V3: now also C16.1, C18.1, JP12.1, JP12.2, JP12.3, JP12.4, JP12.5, JP12.6, R11.1
- net +5V: now also C15.1, C17.1, U$9.12; no longer U$9.VM
- net BAT1: now also Q2.1, Q2.2, Q2.3, R3.1; no longer Q5.5, Q5.6, Q5.7, Q5.8, Q5.9
- net FAUL: now also R11.2, U$9.8, U1.4; no longer U$9.NFAULT, U1.16
- net GND: now also C15.2, C17.2, C18.2, C19.2, JP11.1, JP11.2, JP11.3, JP11.4, JP11.5, JP11.6, U$9.13, U$9.17, U$9.3, U$9.6; no longer Q5.4, U$9.AISEN, U$9.BISEN, U$9.GND
- net N$14: now also U$9.4; no longer U$9.AOUT2
- net N$15: now also U$9.7; no longer U$9.BOUT1
- net N$16: now also U$9.5; no longer U$9.BOUT2
- net N$2: now also JP10.1; no longer U1.9
- net N$23: now also U$9.14; no longer U$9.VINT
- net N$3: now also JP10.2; no longer U1.8
- net N$4: now also JP10.3; no longer U1.7
- net N$5: now also JP10.4; no longer U1.6
- net N$6: now also JP10.5; no longer U1.5
- net N$8: now also U$9.2; no longer U$9.AOUT1
- net N$9: now also U1.16; no longer JP5.6, U1.4
- net OFF: now also C19.1
- net PWM_A0: now also U$9.16; no longer U$9.AIN1
- net PWM_A1: now also U$9.15; no longer U$9.AIN2
- net PWM_B0: now also U$9.9; no longer U$9.BIN1
- net PWM_B1: now also U$9.10; no longer U$9.BIN2
- net RXD0: now also U1.35; no longer U1.34
- net SLEEP: now also U$9.1; no longer U$9.NSLEEP
- net TXD0: now also U1.34; no longer U1.35
- net VBUS: now also C16.2
Routing:
- net +3V3: track 186.8 -> 0.00 mm, vias 8 -> 0
- net +5V: track 108.6 -> 0.00 mm
- net ENC_B0: track 101.9 -> 0.00 mm, vias 1 -> 0
- net ENC_A0: track 101.0 -> 0.00 mm, vias 1 -> 0
- net FAUL: track 85.5 -> 0.00 mm, vias 2 -> 0
- net ENC_B1: track 85.4 -> 0.00 mm, vias 1 -> 0
- net WS2812: track 84.5 -> 0.00 mm, vias 2 -> 0
- net ENC_A1: track 81.7 -> 0.00 mm, vias 1 -> 0
- net PWM_A1: track 76.3 -> 0.00 mm, vias 2 -> 0
- net SERVO: track 74.7 -> 0.00 mm, vias 1 -> 0
- net SLEEP: track 73.9 -> 0.00 mm, vias 2 -> 0
- net PWM_A0: track 73.7 -> 0.00 mm, vias 2 -> 0
- net PWM_B1: track 73.3 -> 0.00 mm, vias 2 -> 0
- net PWM_B0: track 72.8 -> 0.00 mm, vias 2 -> 0
- net ON: track 60.6 -> 0.00 mm
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- removed copper zone on layer 1, net BAT_POL+
