File: ele/FirstBot/untitled.sch (EAGLE design)
At the start: 58 parts, among them T1 BC337, T2 BC337, U1 ESP-WROOM-32, X0 POWER_IN, X1 USB-MICRO-B-BOTTOM

Commit message: ESP32_wroom
CH340C
Parts:
- added C10: 1uf, rcl_upravena:C-EUC0402
- added C11, C12, C13: 1n 50V, rcl_upravena:C-EUC0402
- added R10, R9: 470, rcl_upravena:R-EU_R0603
- added R6, R7: 5k, rcl_upravena:R-EU_R0603
- added R8: 12k, rcl_upravena:R-EU_R0603
- added SW7, SW8: TL3342F160QG/TR, Switch:TL3342F160QG/TR
- C2: value 100n -> 100nf
- CH1: value CH340G -> CH340C; device ch340g:CH340G -> ch340g:CH340C
Connections:
- net !DTR renamed DTR
- net !RTS renamed RTS
- removed net IO0_!RST: T2.C, U1.IO0
- new net CTS: CH1.CTS
- new net IO0: R10.1, R6.1, T2.C, U1.IO0
- new net N$7: C13.1, R10.2, SW7.1, SW7.2
- net +3V3: now also C10.2, R6.2, R8.2
- net EN: now also C11.2, R8.1, R9.1
- net GND: now also C10.1, C11.1, C12.2, C13.2, CH1.GND, R7.1, SW7.3, SW7.4, SW8.3, SW8.4, X1.GND
- net N$1: now also C12.1, R9.2, SW8.1, SW8.2; no longer CH1.GND, X1.GND
- net PWM_A1: now also R7.2
Other:
- moved on the sheet: C1, C2, C3, C4, C5, C8, LED1, LED2, LED3, LED4, LED5, R1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

Commit message: dalsi_text_a_firstbot
Parts:
- removed LED5: BLUE, led:LEDCHIPLED_1206
- removed SW5, SW6: (no value), switch-omron:10-XX
- removed SW7, SW8: TL3342F160QG/TR, Switch:TL3342F160QG/TR
- added BOOT, EN, NO, OFF: TL3342F160QG/TR, Switch:TL3342F160QG/TR
- added C14: (no value), rcl:CPOL-EUSANYO_SMD_F8
- added D1: BAT60JDO-214-AB, diode:BAT60JDO-214-AB
- added IC1: 7808DT, adafruit:7808DT
- added JP5: (no value), pinhead:PINHD-1X6
- added JP8, JP9: (no value), pinhead:PINHD-1X3
- added LED0: BLUE, led:LEDCHIPLED_1206
- added NC1, NC2, NC3, NC4, NC5, NC6: NC, NC:NC
- added Q1: (no value), transistors:N-MOSFET-SOT23-GSD
- added R12: 4,7k, rcl:R-EU_R0402
- C1, C3, C4, C5, C8, C9: device rcl_upravena:C-EUC1206 -> rcl_upravena:C-EUC0402K
- C10, C12, C2: device rcl_upravena:C-EUC0402 -> rcl_upravena:C-EUC0402K
- C23: device resistor:C-EUC0603 -> resistor:C-EUC0402K
- C7: device resistor:C-EUC0805 -> resistor:C-EUC0402K
- Q2, Q5: value (none) -> AO3401ASOP-8_EP_5.0X5.0X1.27P; device transistors:P-MOSFET-MLP_HS -> transistor-fet:AO3401ASOP-8_EP_5.0X5.0X1.27P
- R1, R5: value 10k -> 12k
- R10, R6, R7, R8, R9: device rcl_upravena:R-EU_R0603 -> rcl_upravena:R-EU_R0402
- R2: device rcl_upravena:R-EU_R0805 -> rcl_upravena:R-EU_R0603
- R23, R40, R43, R46, R49: value 10k -> 47k; device resistor:R-EU_R0805 -> resistor:R-EU_R0402
- R24, R38, R41, R44, R47: device resistor:R-EU_R0805 -> resistor:R-EU_R0402
- R29, R39, R42, R45, R48: value (none) -> 180; device resistor:R-EU_R0805 -> resistor:R-EU_R0402
- R3: device rcl_upravena:R-EU_R0805 -> rcl_upravena:R-EU_R0402
- R4: device rcl_upravena:R-EU_M0805 -> rcl_upravena:R-EU_R0402
- SW0, SW1, SW2, SW3, SW4: value (none) -> TL3342F160QG/TR; device switch-omron:10-XX -> Switch:TL3342F160QG/TR
Connections:
- net N$3 renamed D-
- net N$4 renamed D+
- net N$5 renamed VBUS
- removed net VCC: Q2.D
- new net N$11: D1.A, Q2.D
- new net N$2: JP5.1, U1.IO33
- new net N$3: JP5.2, U1.IO32
- new net N$4: JP5.3, U1.IO35
- new net N$5: JP5.4, U1.IO34
- new net N$6: JP5.5, U1.SENSOR_VN
- new net N$9: JP5.6, U1.SENSOR_VP
- new net SERVO: JP9.2, U1.IO23
- new net WS2812: Q1.S, U1.IO22
- new net WS2812-5V: JP8.2, Q1.D, R12.2
- net +3V3: now also CH1.V3, IC1.VO, Q1.G
- net +5V: now also C14.+, D1.C, IC1.VI, JP8.1, JP9.1, R12.1
- net ENC_A0: now also U1.IO25; no longer U1.IO27
- net ENC_A1: now also U1.IO14; no longer U1.IO25
- net ENC_B0: now also U1.IO26; no longer U1.IO14
- net ENC_B1: now also U1.IO27; no longer U1.IO26
- net GND: now also BOOT.3, BOOT.4, C14.-, EN.3, EN.4, IC1.GND, JP8.3, JP9.3, LED0.C, NO.1, NO.2, OFF.1, OFF.2, SW0.1, SW0.2, SW1.1, SW1.2, SW2.1, SW2.2, SW3.1, SW3.2, SW4.1, SW4.2; no longer LED5.C, SW0.S, SW0.S1, SW1.S, SW1.S1, SW2.S, SW2.S1, SW3.S, SW3.S1, SW4.S, SW4.S1, SW5.S, SW5.S1, SW6.S, SW6.S1, SW7.3, SW7.4, SW8.3, SW8.4
- net N$1: now also EN.1, EN.2; no longer SW8.1, SW8.2
- net N$10: now also LED0.A; no longer LED3.A
- net N$28: now also LED3.A; no longer LED5.A
- net N$7: now also BOOT.1, BOOT.2; no longer SW7.1, SW7.2
- net NC-CS: now also NC3.NC
- net NC-HOLD: now also NC1.NC
- net NC-MISO: now also NC6.NC
- net NC-MOSI: now also NC5.NC
- net NC-SCK: now also NC4.NC
- net NC-WP: now also NC2.NC
- net OFF: now also OFF.3, OFF.4; no longer SW5.P, SW5.P1
- net ON: now also NO.3, NO.4; no longer SW4.P, SW4.P1
- net PWM_B0: now also U1.IO16; no longer U1.IO4
- net PWM_B1: now also U1.IO4; no longer U1.IO16
- net SW0: now also SW0.3, SW0.4; no longer SW0.P, SW0.P1
- net SW1: now also SW1.3, SW1.4; no longer SW1.P, SW1.P1
- net SW2: now also SW2.3, SW2.4; no longer SW2.P, SW2.P1
- net SW3: now also SW3.3, SW3.4; no longer SW6.P, SW6.P1
- net SW4: now also SW4.3, SW4.4; no longer SW3.P, SW3.P1
Other:
- moved on the sheet: C10, C12, C13, C2, C9, JP1, JP2, JP6, JP7, LED3, Q6, R1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

Commit message: trochu v tom delam bordel
proste to neumim delat poredne tak tet delam tenhle bordel commit bych mel vse na gitu a budu se snazit to dal delat poradne
Parts:
- removed Q5: AO3401ASOP-8_EP_5.0X5.0X1.27P, transistor-fet:AO3401ASOP-8_EP_5.0X5.0X1.27P
- added C15, C17, C18: 10uf, rcl:C-EUC0603
- added C16: 0,1uf, rcl:C-EUC0402
- added C19: 10uf, resistor:C-EUC0402K
- added JP10, JP11, JP12: (no value), pinhead:PINHD-1X6
- added R11: 4,7k, rcl:R-EU_R0402
- added R13, R14, R15, R16, R17, R18: 180, resistor:R-EU_R0402
- C10, C2: device rcl_upravena:C-EUC0402K -> rcl_upravena:C-EUC0402
- R2: device rcl_upravena:R-EU_R0603 -> rcl_upravena:R-EU_R0402
- U$9: value DRV8833HTSSOP -> DRV8833CPWPR; device texas-cc2541:DRV8833HTSSOP -> DRV8833CPWPR:DRV8833CPWPR
Connections:
- removed net BAT_POL+: Q2.S, Q5.S, R3.1
- new net N$13: JP10.6, JP5.6
- net +3V3: now also C16.1, C18.1, JP12.1, JP12.2, JP12.3, JP12.4, JP12.5, JP12.6, R11.1
- net +5V: now also C15.1, C17.1, U$9.VM; no longer U$9.VM_2.7-10.8V
- net BAT1: now also Q2.S, R3.1; no longer Q5.D
- net FAUL: now also R11.2, U1.SENSOR_VP; no longer U1.IO13
- net GND: now also C15.2, C17.2, C18.2, C19.2, JP11.1, JP11.2, JP11.3, JP11.4, JP11.5, JP11.6, U$9.EXP; no longer Q5.G
- net N$14: now also U$9.AOUT2; no longer U$9.AUOT2
- net N$2: now also JP10.1; no longer U1.IO33
- net N$3: now also JP10.2; no longer U1.IO32
- net N$4: now also JP10.3; no longer U1.IO35
- net N$5: now also JP10.4; no longer U1.IO34
- net N$6: now also JP10.5; no longer U1.SENSOR_VN
- net N$9: now also U1.IO13; no longer JP5.6, U1.SENSOR_VP
- net OFF: now also C19.1
- net RXD0: now also U1.TXD0; no longer U1.RXD0
- net TXD0: now also U1.RXD0; no longer U1.TXD0
- net VBUS: now also C16.2
Other:
- moved on the sheet: C14, C23, C6, C7, JP1, JP2, JP3, JP4, JP5, JP7, OFF, R1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
